File: MotorController/BMC1.sch (EAGLE design)
At the start: 58 parts, among them IC2 LP2950, IC3 MEGA8-AI, Q1 20MHz, U1 BTN8982TA, U2 BTN8982TA, U3 BTN8982TA, U4 TC77-5.0MCTTR, U5 MCP2561-E/SN

Commit message: Finished version 1.
Parts:
- removed IC3: MEGA8-AI, atmel:MEGA8-AI
- removed L1: 10uH, resistor:R-EU_R0805
- removed R27, R29: 10k, resistor:R-EU_R0805
- added IC1: LP2950, linear:LP2950
- added R24, R26: 1k, resistor:R-EU_R0805
- added R25: 30k, resistor:R-EU_R0805
- C1, C4: value 0.1uf 40v -> 0.1uf
- C10: value 0.1uf -> 0.1uf 40v; MF WALSIN -> KEMET; MPN 0805B104K500CT -> C0805C104J5RACTU; OC_FARNELL 2496944 -> 1414663
- C11: value (none) -> 0.1uf 40v; device resistor:CPOL-EUE5-10.5 -> rcl:C-EUC0805; MF (none) -> KEMET; MPN (none) -> C0805C104J5RACTU; OC_FARNELL (none) -> 1414663
- C12: value 0.1uf -> 0.1uf 40v
- C13: value 0.1uf -> 1000uF 50V; device rcl:C-EUC0805 -> rcl:CPOL-EUUD-10X10; MPN C0805C104J5RACTU -> T491A105K016AT; OC_FARNELL 1414663 -> 1457406
- C14: value 0.1uf -> 1000uf 50V; device rcl:C-EUC0805 -> resistor:CPOL-EUE5-10.5; MF WALSIN -> (none); MPN 0805B104K500CT -> (none); OC_FARNELL 2496944 -> (none)
- C2: value 0.1uf -> 10uf 35V; MF KEMET -> MURATA; MPN C0805C104J5RACTU -> GRM32ER7YA106KA12L; OC_FARNELL 1414663 -> 1735537
- C3: value 1000uF 40V -> 0.1uf; device rcl:CPOL-EUUD-10X10 -> rcl:C-EUC0805; MF KEMET -> WALSIN; MPN T491A105K016AT -> 0805B104K500CT; OC_FARNELL 1457406 -> 2496944
- C5: value 0.1uf 40v -> 0.1uf; MF KEMET -> WALSIN; MPN C0805C104J5RACTU -> 0805B104K500CT; OC_FARNELL 1414663 -> 2496944
- C6: value 10uf 35V -> 2.2uf 10V; MF MURATA -> KEMET; MPN GRM32ER7YA106KA12L -> C0805C225K8RACAUTO; OC_FARNELL 1735537 -> 2478259
- C7: value 2.2uf 10V -> 18pf; MF KEMET -> WALSIN; MPN C0805C225K8RACAUTO -> 0805N180J500CT; OC_FARNELL 2478259 -> 2497020
- C9: value 18pf -> 0.1uf; MF WALSIN -> KEMET; MPN 0805N180J500CT -> C0805C104J5RACTU; OC_FARNELL 2497020 -> 1414663
- IC2: value LP2950 -> MEGA8-AI; device linear:LP2950 -> atmel:MEGA8-AI; MF ON SEMICONDUCTOR -> ATMEL; MPN LP2950CDT-5.0G -> (none); OC_FARNELL 1468707 -> (none)
- R10, R3: value 750R -> 10k; MF VISHAY -> WELWYN; MPN CRCW0805750RFKEA -> WCR0805-10KFI; OC_FARNELL 1469956 -> 1099807
- R11, R5: value 100R -> 10k; MPN WCR0805-100RFI -> WCR0805-10KFI; OC_FARNELL 1099793 -> 1099807
- R12, R6: value 30k -> 10k; MF VISHAY -> WELWYN; MPN CRCW080530K0FKEA -> WCR0805-10KFI; OC_FARNELL 1469914 -> 1099807
- R13, R7: value 1k -> 10k; MF VISHAY -> WELWYN; MPN CRCW08051K00FKEA -> WCR0805-10KFI; OC_FARNELL 1469847 -> 1099807
- R14, R15: value 10k -> 750R; MF WELWYN -> VISHAY; MPN WCR0805-10KFI -> CRCW0805750RFKEA; OC_FARNELL 1099807 -> 1469956
- R18: value 30k -> 100R; MF VISHAY -> WELWYN; MPN CRCW080530K0FKEA -> WCR0805-100RFI; OC_FARNELL 1469914 -> 1099793
- R19: value 1k -> 100R; MF VISHAY -> WELWYN; MPN CRCW08051K00FKEA -> WCR0805-100RFI; OC_FARNELL 1469847 -> 1099793
- R2: value 10k -> 10uH; MF WELWYN -> TAIYO YUDEN; MPN WCR0805-10KFI -> LB2012T100KR; OC_FARNELL 1099807 -> 1463501
- R20, R23: value 10k -> 30k; MF WELWYN -> VISHAY; MPN WCR0805-10KFI -> CRCW080530K0FKEA; OC_FARNELL 1099807 -> 1469914
- R21: value 10k -> 1k; MF WELWYN -> VISHAY; MPN WCR0805-10KFI -> CRCW08051K00FKEA; OC_FARNELL 1099807 -> 1469847
- R22: value 120R -> 10k; MF VISHAY -> WELWYN; MPN CRCW0805750RFKEA -> WCR0805-10KFI; OC_FARNELL 1469956 -> 1099807
- R4: value 10k -> 120R; MF WELWYN -> VISHAY; MPN WCR0805-10KFI -> CRCW0805750RFKEA; OC_FARNELL 1099807 -> 1469956
- SV1: device con-lstb:MA06-1 -> con-lstb:MA04-1
- SV2: device con-lstb:MA04-1 -> con-lstb:MA03-2
- SV3: device con-lstb:MA03-2 -> con-lstb:MA06-1
- U1: value BTN8982TA -> TC77-5.0MCTTR; device BTN8982TA:BTN8982TA -> temp-tc77-5v:TC77-5.0MCTTR; MF INFINEON -> MICROCHIP; MPN BTN8982TA -> (none); OC_FARNELL 2470127 -> (none)
- U2: value BTN8982TA -> MCP2561-E/SN; device BTN8982TA:BTN8982TA -> Microchip-MCP2561-E_SN:MCP2561-E/SN; MF INFINEON -> (none); MPN BTN8982TA -> (none); OC_FARNELL 2470127 -> (none)
- U4: value TC77-5.0MCTTR -> BTN8982TA; device temp-tc77-5v:TC77-5.0MCTTR -> BTN8982TA:BTN8982TA; MF MICROCHIP -> INFINEON; MPN (none) -> BTN8982TA; OC_FARNELL (none) -> 2470127
- U5: value MCP2561-E/SN -> BTN8982TA; device Microchip-MCP2561-E_SN:MCP2561-E/SN -> BTN8982TA:BTN8982TA; MF (none) -> INFINEON; MPN (none) -> BTN8982TA; OC_FARNELL (none) -> 2470127
Connections:
- removed net N$1 (its old number): R5.2, U1.SR
- new net N$14: R19.2, U5.SR
- net +7V: now also SV1.2; no longer SV2.2
- net 18V: now also C10.1, C11.1, C12.1, C13.+, C14.+, PAD1.P, R22.2, U4.VS, U5.VS; no longer C1.1, C11.+, C3.+, C4.1, C5.1, PAD4.P, R29.2, U1.VS, U2.VS
- net GND: now also C11.2, C13.-, C14.-, C3.2, C7.1, C9.2, IC1.GND, IC2.GND@1, IC2.GND@2, PAD2.P, R14.1, R15.1, R18.1, R21.1, R24.1, R26.1, SV1.1, SV2.6, SV3.2, U1.VSS, U2.VSS, U4.GND, U5.GND; no longer C11.-, C13.2, C14.2, C3.-, C7.2, C9.1, IC3.GND, IC3.GND@1, IC3.GND@2, PAD5.P, R10.1, R11.1, R13.1, R3.1, R5.1, R7.1, SV1.2, SV2.1, SV3.6, U1.GND, U2.GND, U4.VSS, U5.VSS
- net N$10: now also R8.2, U4.IN; no longer R9.2, U2.IN
- net N$11: now also IC2.PC2(ADC2), R5.1; no longer IC3.PC2(ADC2), R20.1
- net N$12: now also IC2.PD4(XCK/T0), R8.1; no longer IC3.PD4(XCK/T0), R9.1
- net N$13: now also PAD5.P, R25.2, U5.OUT2; no longer PAD3.P, R18.2, U3.OUT2
- net N$15: now also R12.2, U5.INH; no longer R14.2, U3.INH
- net N$16: now also R11.2, U5.IN; no longer R15.2, U3.IN
- net N$17: now also IC2.ADC6, R10.1; no longer IC3.ADC6, R23.1
- net N$18: now also IC2.ADC7, R25.1, R26.2; no longer IC3.ADC7, R18.1, R19.2
- net N$19: now also R4.1, SV1.4, U2.CANL; no longer R22.1, SV2.4, U5.CANL
- net N$2: now also PAD3.P, R20.2, U3.OUT2; no longer PAD1.P, R6.2, U1.OUT2
- net N$21: now also IC2.PD5(T1), R9.1; no longer IC3.PD5(T1), R8.1
- net N$22: now also IC2.PC3(ADC3), R23.1, R24.2; no longer IC3.PC3(ADC3), R12.1, R13.2
- net N$23: now also R4.2, SV1.3, U2.CANH; no longer R22.2, SV2.3, U5.CANH
- net N$25: now also IC2.PB1(OC1A), U2.STBY; no longer IC3.PB1(OC1A), U5.STBY
- net N$26: now also C2.1, IC1.I; no longer C6.1, IC2.I
- net N$27: now also C7.2, IC2.PB6(XTAL1/TOSC1); no longer C8.2, IC3.PB6(XTAL1/TOSC1)
- net N$3: now also R7.2, U3.INH; no longer R1.2, U1.INH
- net N$31: now also C8.2, IC2.PB7(XTAL2/TOSC2); no longer C9.2, IC3.PB7(XTAL2/TOSC2)
- net N$32: now also IC2.PB3(MOSI/OC2), SV2.4, SV3.6; no longer IC3.PB3(MOSI/OC2), SV1.6, SV3.4
- net N$33: now also IC2.PD2(INT0), R6.1; no longer IC3.PD2(INT0), R2.1
- net N$34: now also IC2.PB5(SCK), SV2.3, U1.SCK; no longer IC3.PB5(SCK), SV3.3, U4.SCK
- net N$36: now also R15.2, R5.2, U4.IS; no longer R10.2, R20.2, U2.IS
- net N$37: now also IC2.PC4(ADC4/SDA), SV3.3; no longer IC3.PC4(ADC4/SDA), SV1.3
- net N$38: now also R13.2, R14.2, U3.IS; no longer R3.2, R4.2, U1.IS
- net N$39: now also R10.2, U5.IS; no longer R23.2, U3.IS
- net N$4: now also R6.2, U3.IN; no longer R2.2, U1.IN
- net N$40: now also C3.1, IC2.AVCC, R2.1; no longer C10.1, IC3.AVCC, L1.1
- net N$41: now also IC2.PC5(ADC5/SCL), SV3.4; no longer IC3.PC5(ADC5/SCL), SV1.4
- net N$42: now also IC2.PD0(RXD), U2.RXD; no longer IC3.PD0(RXD), U5.RXD
- net N$43: now also IC2.PD1(TXD), U2.TXD; no longer IC3.PD1(TXD), U5.TXD
- net N$44: now also IC2.PD7(AIN1), R12.1; no longer IC3.PD7(AIN1), R14.1
- net N$45: now also IC2.PD6(AIN0), R11.1; no longer IC3.PD6(AIN0), R15.1
- net N$46: now also IC2.PD3(INT1), R7.1; no longer IC3.PD3(INT1), R1.1
- net N$49: now also IC2.PB2(SS/OC1B), SV3.5; no longer IC3.PB2(SS/OC1B), SV1.5
- net N$5: now also IC2.PC1(ADC1), R20.1, R21.2; no longer IC3.PC1(ADC1), R6.1, R7.2
- net N$50: now also IC2.PB0(ICP), R1.1, U1.CS*; no longer IC3.PB0(ICP), R27.1, U4.CS*
- net N$52: now also IC2.PC6(/RESET), R3.2, SV2.5; no longer IC3.PC6(/RESET), R21.2, SV3.5
- net N$54: now also C5.1, IC2.AREF; no longer C14.1, IC3.AREF
- net N$55: now also IC2.PC0(ADC0), R13.1; no longer IC3.PC0(ADC0), R4.1
- net N$6: now also IC2.PB4(MISO), SV2.1, U1.SI/O; no longer IC3.PB4(MISO), SV3.1, U4.SI/O
- net N$7: now also PAD4.P, R22.1, R23.2, U4.OUT2; no longer PAD2.P, R12.2, R29.1, U2.OUT2
- net N$8: now also R18.2, U4.SR; no longer R11.2, U2.SR
- net N$9: now also R9.2, U4.INH; no longer R8.2, U2.INH
- net VCC: now also C1.1, C4.1, C6.1, C9.1, IC1.O, IC2.VCC@1, IC2.VCC@2, R1.2, R2.2, R3.1, SV2.2, SV3.1, U1.VDD, U2.VDD; no longer C12.1, C13.1, C2.1, C7.1, IC2.O, IC3.VCC@1, IC3.VCC@2, L1.2, R21.1, R27.2, SV1.1, SV3.2, U4.VDD, U5.VDD
Other:
- moved on the sheet: C1, C10, C12, C2, C4, C5, C6, C7, C8, C9, PAD1, PAD2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
