File: MotorController2/BMC2.sch (KiCad schematic (older format))
At the start: 0 parts

Commit message: Most of new motor controller schematic, and leg V2.
Parts:
- added C?: 0.1uf (6V min), symbol C
- added C?: C, symbol C
- added D?: D_Schottky, symbol D_Schottky
- added P?: CONN_01X04, symbol CONN_01X04
- added P?: USB_OTG, symbol USB_OTG
- added P?: CONN_01X10, symbol CONN_01X10
- added R? (x2): 22R, symbol R
- added R? (x7): 1k, symbol R
- added R?: 10k, symbol R
- added U?: TJA1042T/3, Housings_SOIC:SOIC-8_3.9x4.9mm_Pitch1.27mm, symbol TJA1042T/3
Connections:
- net labels added: +3V3, +5V, +8V, GND
- wire segments 63 -> 152
- no-connect marks 0 -> 1

Commit message: Initial schematic complete.
Parts:
- added P?: CONN_01X05, symbol CONN_01X05
- added P? (x3): CONN_01X01, symbol CONN_01X01
- added W? (x2): TEST_1P, symbol TEST_1P
Connections:
- wire segments 152 -> 179
Changed lines of the file:
@@
 F37 "PWRGD" I R 4850 3750 60
 F38 "CAN_STBY" O L 3350 4200 60
+F39 "NRST" I L 3350 2300 60
+F40 "TempDrv" I R 4850 5050 60
 $EndSheet
 $Sheet
@@
 F24 "INLC" I L 6700 4750 60
 F25 "VSupplySense" O L 6700 2850 60
+F26 "TempDrv" I L 6700 5000 60
 $EndSheet
 $Sheet
@@
 $EndComp
 $Comp
-L +5V #PWR?
+L +5V #PWR01
 U 1 1 58654E2C
 P 1900 3450
-F 0 "#PWR?" H 1900 3300 50  0001 C CNN
+F 0 "#PWR01" H 1900 3300 50  0001 C CNN
 F 1 "+5V" H 1900 3590 50  0000 C CNN
 F 2 "" H 1900 3450 50  0000 C CNN
@@
 $EndComp
 $Comp
-L GND #PWR?
+L GND #PWR02
 U 1 1 5865537A
 P 1900 4500
-F 0 "#PWR?" H 1900 4250 50  0001 C CNN
+F 0 "#PWR02" H 1900 4250 50  0001 C CNN
 F 1 "GND" H 1900 4350 50  0000 C CNN
 F 2 "" H 1900 4500 50  0000 C CNN
@@
 $EndComp
 $Comp
-L +3V3 #PWR?
+L +3V3 #PWR03
 U 1 1 586556AA
 P 2550 4100
-F 0 "#PWR?" H 2550 3950 50  0001 C CNN
+F 0 "#PWR03" H 2550 3950 50  0001 C CNN
 F 1 "+3V3" H 2550 4240 50  0000 C CNN
 F 2 "" H 2550 4100 50  0000 C CNN
@@
 $EndComp
 $Comp
-L GND #PWR?
+L GND #PWR04
 U 1 1 58657281
 P 1100 3600
-F 0 "#PWR?" H 1100 3350 50  0001 C CNN
+F 0 "#PWR04" H 1100 3350 50  0001 C CNN
 F 1 "GND" H 1100 3450 50  0000 C CNN
 F 2 "" H 1100 3600 50  0000 C CNN
@@
 $EndComp
 $Comp
-L +8V #PWR?
+L +8V #PWR05
 U 1 1 5865817E
 P 1300 3650
-F 0 "#PWR?" H 1300 3500 50  0001 C CNN
+F 0 "#PWR05" H 1300 3500 50  0001 C CNN
 F 1 "+8V" H 1300 3790 50  0000 C CNN
 F 2 "" H 1300 3650 50  0000 C CNN
@@
 $EndComp
 $Comp
-L +5V #PWR?
+L +5V #PWR06
 U 1 1 5865BDDB
 P 1200 4450
-F 0 "#PWR?" H 1200 4300 50  0001 C CNN
+F 0 "#PWR06" H 1200 4300 50  0001 C CNN
 F 1 "+5V" H 1200 4590 50  0000 C CNN
 F 2 "" H 1200 4450 50  0000 C CNN
@@
 $EndComp
 $Comp
-L GND #PWR?
+L GND #PWR07
 U 1 1 5865BF5D
 P 1200 4900
-F 0 "#PWR?" H 1200 4650 50  0001 C CNN
+F 0 "#PWR07" H 1200 4650 50  0001 C CNN
 F 1 "GND" H 1200 4750 50  0000 C CNN
 F 2 "" H 1200 4900 50  0000 C CNN
@@
 $EndComp
 $Comp
-L GND #PWR?
+L GND #PWR08
 U 1 1 5865E9C4
 P 2350 5900
-F 0 "#PWR?" H 2350 5650 50  0001 C CNN
+F 0 "#PWR08" H 2350 5650 50  0001 C CNN
 F 1 "GND" H 2350 5750 50  0000 C CNN
 F 2 "" H 2350 5900 50  0000 C CNN
@@
 	2300 5150 2300 4750
 $Comp
-L +5V #PWR?
+L +5V #PWR09
 U 1 1 58660AEB
 P 2850 4650
-F 0 "#PWR?" H 2850 4500 50  0001 C CNN
+F 0 "#PWR09" H 2850 4500 50  0001 C CNN
 F 1 "+5V" H 2850 4790 50  0000 C CNN
 F 2 "" H 2850 4650 50  0000 C CNN
@@
 $EndComp
 $Comp
-L GND #PWR?
+L GND #PWR010
 U 1 1 58665413
 P 1050 2950
-F 0 "#PWR?" H 1050 2700 50  0001 C CNN
+F 0 "#PWR010" H 1050 2700 50  0001 C CNN
 F 1 "GND" H 1050 2800 50  0000 C CNN
 F 2 "" H 1050 2950 50  0000 C CNN
@@
 	1050 2850 950  2850
 $Comp
-L +3V3 #PWR?
+L +3V3 #PWR011
 U 1 1 58665925
 P 1200 2900
-F 0 "#PWR?" H 1200 2750 50  0001 C CNN
+F 0 "#PWR011" H 1200 2750 50  0001 C CNN
 F 1 "+3V3" H 1200 3040 50  0000 C CNN
 F 2 "" H 1200 2900 50  0000 C CNN
@@
 	2100 3150 2350 3150
 $Comp
-L GND #PWR?
+L GND #PWR012
 U 1 1 586688E0
 P 2200 3250
-F 0 "#PWR?" H 2200 3000 50  0001 C CNN
+F 0 "#PWR012" H 2200 3000 50  0001 C CNN
 F 1 "GND" H 2200 3100 50  0000 C CNN
 F 2 "" H 2200 3250 50  0000 C CNN
@@
 Wire Wire Line
 	1450 1950 1800 1950
+$Comp
+L CONN_01X05 P?
+U 1 1 586CDC2C
+P 850 1250
+F 0 "P?" H 850 1550 50  0000 C CNN
+F 1 "CONN_01X05" V 950 1250 50  0000 C CNN
+F 2 "" H 850 1250 50  0000 C CNN
+F 3 "" H 850 1250 50  0000 C CNN
+	1    850  1250
+	-1   0    0    -1
+$EndComp
+$Comp
+L GND #PWR013
+U 1 1 586CE0C4
+P 1150 1600
+F 0 "#PWR013" H 1150 1350 50  0001 C CNN
+F 1 "GND" H 1150 1450 50  0000 C CNN
+F 2 "" H 1150 1600 50  0000 C CNN
+F 3 "" H 1150 1600 50  0000 C CNN
+	1    1150 1600
+	1    0    0    -1
+$EndComp
+$Comp
+L +5V #PWR014
+U 1 1 586CE33C
+P 1450 1450
+F 0 "#PWR014" H 1450 1300 50  0001 C CNN
+F 1 "+5V" H 1450 1590 50  0000 C CNN
+F 2 "" H 1450 1450 50  0000 C CNN
+F 3 "" H 1450 1450 50  0000 C CNN
+	1    1450 1450
+	1    0    0    -1
+$EndComp
+Wire Wire Line
+	1050 1450 1150 1450
+Wire Wire Line
+	1150 1450 1150 1600
+Wire Wire Line
+	1050 1350 1250 1350
+Wire Wire Line
+	1250 1350 1250 1550
+Wire Wire Line
+	1250 1550 1450 1550
+Wire Wire Line
+	1450 1550 1450 1450
+Wire Wire Line
+	3350 2500 2950 2500
+Wire Wire Line
+	2950 2500 2950 1250
+Wire Wire Line
+	2950 1250 1050 1250
+Wire Wire Line
+	3350 2400 3050 2400
+Wire Wire Line
+	3050 2400 3050 1150
+Wire Wire Line
+	3050 1150 1050 1150
+Wire Wire Line
+	3350 2300 3150 2300
+Wire Wire Line
+	3150 2300 3150 1050
+Wire Wire Line
+	3150 1050 1050 1050
+$Comp
+L CONN_01X01 P?
+U 1 1 586D399A
+P 8750 2400
+F 0 "P?" H 8750 2500 50  0000 C CNN
+F 1 "CONN_01X01" V 8850 2400 50  0000 C CNN
+F 2 "" H 8750 2400 50  0000 C CNN
+F 3 "" H 8750 2400 50  0000 C CNN
+	1    8750 2400
+	1    0    0    -1
+$EndComp
+Wire Wire Line
+	8100 2400 8550 2400
+$Comp
+L CONN_01X01 P?
+U 1 1 586D4187
+P 8750 2650
+F 0 "P?" H 8750 2750 50  0000 C CNN
+F 1 "CONN_01X01" V 8850 2650 50  0000 C CNN
+F 2 "" H 8750 2650 50  0000 C CNN
+F 3 "" H 8750 2650 50  0000 C CNN
+	1    8750 2650
+	1    0    0    -1
+$EndComp
+$Comp
+L CONN_01X01 P?
+U 1 1 586D4351
+P 8750 2900
+F 0 "P?" H 8750 3000 50  0000 C CNN
+F 1 "CONN_01X01" V 8850 2900 50  0000 C CNN
+F 2 "" H 8750 2900 50  0000 C CNN
+F 3 "" H 8750 2900 50  0000 C CNN
+	1    8750 2900
+	1    0    0    -1
+$EndComp
+Wire Wire Line
+	8550 2650 8450 2650
+Wire Wire Line
+	8450 2650 8450 2550
+Wire Wire Line
+	8450 2550 8100 2550
+Wire Wire Line
+	8100 2700 8300 2700
+Wire Wire Line
+	8300 2700 8300 2900
+Wire Wire Line
+	8300 2900 8550 2900
+$Comp
+L TEST_1P W?
+U 1 1 586E727E
+P 2850 3850
+F 0 "W?" H 2850 4120 50  0000 C CNN
+F 1 "TEST_1P" H 2850 4050 50  0000 C CNN
+F 2 "" H 3050 3850 50  0000 C CNN
+F 3 "" H 3050 3850 50  0000 C CNN
+	1    2850 3850
+	1    0    0    -1
+$EndComp
+Wire Wire Line
+	2850 3850 2850 3950
+Connection ~ 2850 3950
+$Comp
+L TEST_1P W?
+U 1 1 586E75E8
+P 3150 3850
+F 0 "W?" H 3150 4120 50  0000 C CNN
+F 1 "TEST_1P" H 3150 4050 50  0000 C CNN
+F 2 "" H 3350 3850 50  0000 C CNN
+F 3 "" H 3350 3850 50  0000 C CNN
+	1    3150 3850
+	1    0    0    -1
+$EndComp
+Wire Wire Line
+	3150 3850 3150 4050
+Connection ~ 3150 4050
+Wire Wire Line
+	4850 5050 5900 5050
+Wire Wire Line
+	5900 5050 5900 5000
+Wire Wire Line
+	5900 5000 6700 5000
 $EndSCHEMATC

Commit message: Component footprints.
Parts:
- removed P?: CONN_01X10, symbol CONN_01X10
- added P1: Sensor, Socket_Strips:Socket_Strip_Angled_1x09, symbol CONN_01X09
- added P10: GND, Connect:Banana_Jack_1Pin, symbol CONN_01X01
- added P9: VSUPPLY, Connect:Banana_Jack_1Pin, symbol CONN_01X01
- C1: renamed from C?; footprint (none) -> Capacitors_SMD:C_0805_HandSoldering
- C2: renamed from C?; value C -> 0.1uF; footprint (none) -> Capacitors_SMD:C_0805_HandSoldering
- D1: renamed from D?; value D_Schottky -> 10V; footprint (none) -> Diodes_SMD:DO-214AB_Handsoldering
- P2: renamed from P?; value CONN_01X04 -> CAN; footprint (none) -> Sockets_MOLEX_KK-System:Socket_MOLEX-KK-RM2-54mm_Lock_4pin_straight
- P3: renamed from P?; value CONN_01X05 -> DATA; footprint (none) -> Sockets_MOLEX_KK-System:Socket_MOLEX-KK-RM2-54mm_Lock_5pin_straight
- P4: renamed from P?; footprint (none) -> Connect:USB_Mini-B; Order (none) -> http://uk.farnell.com/molex/67503-1020/mini-usb-2-0-otg-typ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
- P5: renamed from P?; value CONN_01X01 -> PhaseA; footprint (none) -> Connect:Banana_Jack_1Pin
- P6: renamed from P?; value CONN_01X01 -> PhaseB; footprint (none) -> Connect:Banana_Jack_1Pin
- P7: renamed from P?; value CONN_01X01 -> PhaseC; footprint (none) -> Connect:Banana_Jack_1Pin
- R1, R10, R2, R3, R4, R5, R6, R7, R8, R9: renamed from R?; footprint (none) -> Resistors_SMD:R_0805_HandSoldering
- W1: renamed from W?; value TEST_1P -> CAN_TX; footprint (none) -> Measurement_Points:Measurement_Point_Round-SMD-Pad_Big
- W2: renamed from W?; value TEST_1P -> CAN_RX; footprint (none) -> Measurement_Points:Measurement_Point_Round-SMD-Pad_Big
- gave numbers to parts that had none: 1
Connections:
- net labels added: +36V
- wire segments 179 -> 183
- no-connect marks 1 -> 4
Other:
- moved on the sheet: D1

Commit message: Add local library.
Parts:
- added P11: I2C, Sockets_MOLEX_KK-System:Socket_MOLEX-KK-RM2-54mm_Lock_4pin_straight, symbol CONN_01X04
Connections:
- wire segments 183 -> 195
- no-connect marks 4 -> 2
Changed lines of the file:
@@
 Wire Wire Line
 	1050 3050 1050 2850
-NoConn ~ 3350 4800
-NoConn ~ 3350 4900
 NoConn ~ 4050 1350
 $Comp
@@
 $EndComp
 Wire Wire Line
-	8200 1650 7800 1650
+	7800 1650 8200 1650
 Wire Wire Line
 	8200 1350 7750 1350
@@
 	7950 1950 7950 1650
 Connection ~ 7950 1650
+$Comp
+L CONN_01X04 P11
+U 1 1 586E38C6
+P 2650 4650
+F 0 "P11" H 2650 4900 50  0000 C CNN
+F 1 "I2C" V 2750 4650 50  0000 C CNN
+F 2 "Sockets_MOLEX_KK-System:Socket_MOLEX-KK-RM2-54mm_Lock_4pin_straight" H 2650 4650 50  0001 C CNN
+F 3 "" H 2650 4650 50  0000 C CNN
+F 4 "http://uk.farnell.com/molex/171856-0004/connector-header-tht-2-54mm-4way/dp/2366182" H 2650 4650 60  0001 C CNN "Order"
+	1    2650 4650
+	-1   0    0    -1
+$EndComp
+$Comp
+L GND #PWR018
+U 1 1 586E3AFE
+P 3150 4300
+F 0 "#PWR018" H 3150 4050 50  0001 C CNN
+F 1 "GND" H 3150 4150 50  0000 C CNN
+F 2 "" H 3150 4300 50  0000 C CNN
+F 3 "" H 3150 4300 50  0000 C CNN
+	1    3150 4300
+	1    0    0    -1
+$EndComp
+$Comp
+L +3V3 #PWR019
+U 1 1 586E3CD7
+P 3200 4650
+F 0 "#PWR019" H 3200 4500 50  0001 C CNN
+F 1 "+3V3" H 3200 4790 50  0000 C CNN
+F 2 "" H 3200 4650 50  0000 C CNN
+F 3 "" H 3200 4650 50  0000 C CNN
+	1    3200 4650
+	1    0    0    -1
+$EndComp
+Wire Wire Line
+	2850 4500 2900 4500
+Wire Wire Line
+	2900 4500 2900 4300
+Wire Wire Line
+	2900 4300 3150 4300
+Wire Wire Line
+	2850 4600 3050 4600
+Wire Wire Line
+	3050 4600 3050 4650
+Wire Wire Line
+	3050 4650 3200 4650
+Wire Wire Line
+	3350 4800 3000 4800
+Wire Wire Line
+	3000 4800 3000 4700
+Wire Wire Line
+	3000 4700 2850 4700
+Wire Wire Line
+	2850 4800 2950 4800
+Wire Wire Line
+	2950 4800 2950 4900
+Wire Wire Line
+	2950 4900 3350 4900
 $EndSCHEMATC

Commit message: Work on PCB layout.
Parts:
- added P12: CAN, Pin_Headers:Pin_Header_Angled_1x04, symbol CONN_01X04
- D1: footprint Diodes_SMD:DO-214AB_Handsoldering -> Diodes_SMD:SOD-123
- P1: footprint Socket_Strips:Socket_Strip_Angled_1x09 -> Pin_Headers:Pin_Header_Angled_1x09
- P10, P5, P6, P7, P9: footprint Connect:Banana_Jack_1Pin -> Connect:1pin
- P11: footprint Sockets_MOLEX_KK-System:Socket_MOLEX-KK-RM2-54mm_Lock_4pin_straight -> Pin_Headers:Pin_Header_Straight_1x04
- P2: footprint Sockets_MOLEX_KK-System:Socket_MOLEX-KK-RM2-54mm_Lock_4pin_straight -> Pin_Headers:Pin_Header_Angled_1x04
- P3: footprint Sockets_MOLEX_KK-System:Socket_MOLEX-KK-RM2-54mm_Lock_5pin_straight -> Pin_Headers:Pin_Header_Angled_1x05
Connections:
- wire segments 195 -> 200
Other:
- moved on the sheet: C1, P2
Changed lines of the file:
@@
 L CONN_01X04 P2
 U 1 1 58656D5A
-P 800 4000
-F 0 "P2" H 800 4250 50  0000 C CNN
-F 1 "CAN" V 900 4000 50  0000 C CNN
-F 2 "Sockets_MOLEX_KK-System:Socket_MOLEX-KK-RM2-54mm_Lock_4pin_straight" H 800 4000 50  0001 C CNN
-F 3 "" H 800 4000 50  0000 C CNN
-	1    800  4000
+P 750 4000
+F 0 "P2" H 750 4250 50  0000 C CNN
+F 1 "CAN" V 850 4000 50  0000 C CNN
+F 2 "Pin_Headers:Pin_Header_Angled_1x04" H 750 4000 50  0001 C CNN
+F 3 "" H 750 4000 50  0000 C CNN
+	1    750  4000
 	-1   0    0    -1
 $EndComp
@@
 L C C1
 U 1 1 5865BC3F
-P 1200 4650
-F 0 "C1" H 1225 4750 50  0000 L CNN
-F 1 "0.1uf (6V min)" H 1225 4550 50  0000 L CNN
-F 2 "Capacitors_SMD:C_0805_HandSoldering" H 1238 4500 50  0001 C CNN
-F 3 "" H 1200 4650 50  0000 C CNN
-	1    1200 4650
+P 1150 5250
+F 0 "C1" H 1175 5350 50  0000 L CNN
+F 1 "0.1uf (6V min)" H 1175 5150 50  0000 L CNN
+F 2 "Capacitors_SMD:C_0805_HandSoldering" H 1188 5100 50  0001 C CNN
+F 3 "" H 1150 5250 50  0000 C CNN
+	1    1150 5250
 	1    0    0    -1
 $EndComp
@@
 L +5V #PWR06
 U 1 1 5865BDDB
-P 1200 4450
-F 0 "#PWR06" H 1200 4300 50  0001 C CNN
-F 1 "+5V" H 1200 4590 50  0000 C CNN
-F 2 "" H 1200 4450 50  0000 C CNN
-F 3 "" H 1200 4450 50  0000 C CNN
-	1    1200 4450
+P 1150 5050
+F 0 "#PWR06" H 1150 4900 50  0001 C CNN
+F 1 "+5V" H 1150 5190 50  0000 C CNN
+F 2 "" H 1150 5050 50  0000 C CNN
+F 3 "" H 1150 5050 50  0000 C CNN
+	1    1150 5050
 	1    0    0    -1
 $EndComp
@@
 L GND #PWR07
 U 1 1 5865BF5D
-P 1200 4900
-F 0 "#PWR07" H 1200 4650 50  0001 C CNN
-F 1 "GND" H 1200 4750 50  0000 C CNN
-F 2 "" H 1200 4900 50  0000 C CNN
-F 3 "" H 1200 4900 50  0000 C CNN
-	1    1200 4900
+P 1150 5500
+F 0 "#PWR07" H 1150 5250 50  0001 C CNN
+F 1 "GND" H 1150 5350 50  0000 C CNN
+F 2 "" H 1150 5500 50  0000 C CNN
+F 3 "" H 1150 5500 50  0000 C CNN
+	1    1150 5500
 	1    0    0    -1
 $EndComp
@@
 	3350 4200 2400 4200
 Wire Wire Line
-	1400 4100 1250 4100
-Wire Wire Line
-	1250 4100 1250 4150
-Wire Wire Line
-	1250 4150 1000 4150
-Wire Wire Line
-	1000 4050 1200 4050
-Wire Wire Line
-	1200 4050 1200 3900
+	1400 4100 1300 4100
+Wire Wire Line
+	1300 4100 1300 4700
+Wire Wire Line
+	1300 4150 950  4150
+Wire Wire Line
+	950  4050 1200 4050
+Wire Wire Line
+	1200 3900 1200 4600
 Wire Wire Line
 	1200 3900 1400 3900
 Wire Wire Line
-	1000 3850 1000 3600
-Wire Wire Line
-	1000 3600 1100 3600
-Wire Wire Line
-	1000 3950 1100 3950
-Wire Wire Line
-	1100 3950 1100 3800
+	950  3950 1100 3950
+Wire Wire Line
+	1100 3800 1100 4500
 Wire Wire Line
 	1100 3800 1300 3800
@@
 	1300 3800 1300 3650
 Wire Wire Line
-	1200 4900 1200 4800
-Wire Wire Line
-	1200 4500 1200 4450
+	1150 5500 1150 5400
+Wire Wire Line
+	1150 5100 1150 5050
 Wire Wire Line
 	2950 5150 3150 5150
@@
 F 0 "D1" H 2350 5000 50  0000 C CNN
 F 1 "10V" H 2350 4800 50  0000 C CNN
-F 2 "Diodes_SMD:DO-214AB_Handsoldering" H 2350 4900 50  0001 C CNN
+F 2 "Diodes_SMD:SOD-123" H 2350 4900 50  0001 C CNN
 F 3 "" H 2350 4900 50  0000 C CNN
 	1    2350 4900
@@
 F 0 "P3" H 850 1550 50  0000 C CNN
 F 1 "DATA" V 950 1250 50  0000 C CNN
-F 2 "Sockets_MOLEX_KK-System:Socket_MOLEX-KK-RM2-54mm_Lock_5pin_straight" H 850 1250 50  0001 C CNN
+F 2 "Pin_Headers:Pin_Header_Angled_1x05" H 850 1250 50  0001 C CNN
 F 3 "" H 850 1250 50  0000 C CNN
 	1    850  1250
@@
 F 0 "P5" H 8750 2500 50  0000 C CNN
 F 1 "PhaseA" H 8850 2400 50  0000 C CNN
-F 2 "Connect:Banana_Jack_1Pin" H 8750 2400 50  0001 C CNN
+F 2 "Connect:1pin" H 8750 2400 50  0001 C CNN
 F 3 "" H 8750 2400 50  0000 C CNN
 	1    8750 2400
@@
 F 0 "P6" H 8750 2750 50  0000 C CNN
 F 1 "PhaseB" H 8850 2650 50  0000 C CNN
-F 2 "Connect:Banana_Jack_1Pin" H 8750 2650 50  0001 C CNN
+F 2 "Connect:1pin" H 8750 2650 50  0001 C CNN
 F 3 "" H 8750 2650 50  0000 C CNN
 	1    8750 2650
@@
 F 0 "P7" H 8750 3000 50  0000 C CNN
 F 1 "PhaseC" H 8850 2900 50  0000 C CNN
-F 2 "Connect:Banana_Jack_1Pin" H 8750 2900 50  0001 C CNN
+F 2 "Connect:1pin" H 8750 2900 50  0001 C CNN
 F 3 "" H 8750 2900 50  0000 C CNN
 	1    8750 2900
@@
 F 0 "P1" H 750 2950 50  0000 C CNN
 F 1 "Sensor" V 850 2450 50  0000 C CNN
-F 2 "Socket_Strips:Socket_Strip_Angled_1x09" H 750 2450 50  0001 C CNN
+F 2 "Pin_Headers:Pin_Header_Angled_1x09" H 750 2450 50  0001 C CNN
 F 3 "" H 750 2450 50  0000 C CNN
 	1    750  2450
@@
 F 0 "P9" H 8400 1450 50  0000 C CNN
 F 1 "VSUPPLY" H 8500 1350 50  0000 C CNN
-F 2 "Connect:Banana_Jack_1Pin" H 8400 1350 50  0001 C CNN
+F 2 "Connect:1pin" H 8400 1350 50  0001 C CNN
 F 3 "" H 8400 1350 50  0000 C CNN
 	1    8400 1350
@@
 F 0 "P10" H 8400 1750 50  0000 C CNN
 F 1 "GND" H 8500 1650 50  0000 C CNN
-F 2 "Connect:Banana_Jack_1Pin" H 8400 1650 50  0001 C CNN
+F 2 "Connect:1pin" H 8400 1650 50  0001 C CNN
 F 3 "" H 8400 1650 50  0000 C CNN
 	1    8400 1650
@@
 F 0 "P11" H 2650 4900 50  0000 C CNN
 F 1 "I2C" V 2750 4650 50  0000 C CNN
-F 2 "Sockets_MOLEX_KK-System:Socket_MOLEX-KK-RM2-54mm_Lock_4pin_straight" H 2650 4650 50  0001 C CNN
+F 2 "Pin_Headers:Pin_Header_Straight_1x04" H 2650 4650 50  0001 C CNN
 F 3 "" H 2650 4650 50  0000 C CNN
 F 4 "http://uk.farnell.com/molex/171856-0004/connector-header-tht-2-54mm-4way/dp/2366182" H 2650 4650 60  0001 C CNN "Order"
@@
 Wire Wire Line
 	2950 4900 3350 4900
+$Comp
+L CONN_01X04 P12
+U 1 1 58700494
+P 750 4550
+F 0 "P12" H 750 4800 50  0000 C CNN
+F 1 "CAN" V 850 4550 50  0000 C CNN
+F 2 "Pin_Headers:Pin_Header_Angled_1x04" H 750 4550 50  0001 C CNN
+F 3 "" H 750 4550 50  0000 C CNN
+	1    750  4550
+	-1   0    0    -1
+$EndComp
+Wire Wire Line
+	1200 4600 950  4600
+Connection ~ 1200 4050
+Wire Wire Line
+	1300 4700 950  4700
+Connection ~ 1300 4150
+Wire Wire Line
+	1100 4500 950  4500
+Connection ~ 1100 3950
+Wire Wire Line
+	950  3850 1000 3850
+Wire Wire Line
+	1000 3600 1000 4400
+Wire Wire Line
+	1000 4400 950  4400
+Wire Wire Line
+	1000 3600 1100 3600
+Connection ~ 1000 3850
 $EndSCHEMATC

Commit message: Laying out power section.
Parts:
- P4: symbol USB_OTG -> USB_OTG-RESCUE-BMC2
- W1, W2: footprint Measurement_Points:Measurement_Point_Round-SMD-Pad_Big -> Measurement_Points:Measurement_Point_Round-SMD-Pad_Small
Connections:
- no-connect marks 2 -> 1
Changed lines of the file:
@@
 EESchema Schematic File Version 2
+LIBS:BMC2-rescue
 LIBS:power
 LIBS:device
@@
 LIBS:IFX91041EJV33
 LIBS:BMC2-cache
-EELAYER 25 0
+EELAYER 26 0
 EELAYER END
 $Descr A4 11693 8268
@@
 $EndComp
 $Comp
-L USB_OTG P4
+L USB_OTG-RESCUE-BMC2 P4
 U 1 1 5865C76F
 P 2000 5350
@@
 F 0 "W1" H 2850 4120 50  0000 C CNN
 F 1 "CAN_TX" H 2850 4050 50  0000 C CNN
-F 2 "Measurement_Points:Measurement_Point_Round-SMD-Pad_Big" H 3050 3850 50  0001 C CNN
+F 2 "Measurement_Points:Measurement_Point_Round-SMD-Pad_Small" H 3050 3850 50  0001 C CNN
 F 3 "" H 3050 3850 50  0000 C CNN
 	1    2850 3850
@@
 F 0 "W2" H 3150 4120 50  0000 C CNN
 F 1 "CAN_RX" H 3150 4050 50  0000 C CNN
-F 2 "Measurement_Points:Measurement_Point_Round-SMD-Pad_Big" H 3350 3850 50  0001 C CNN
+F 2 "Measurement_Points:Measurement_Point_Round-SMD-Pad_Small" H 3350 3850 50  0001 C CNN
 F 3 "" H 3350 3850 50  0000 C CNN
 	1    3150 3850
@@
 Wire Wire Line
 	1050 3050 1050 2850
-NoConn ~ 4050 1350
 $Comp
 L +36V #PWR015

Commit message: More of the layout done.
Connections:
- net Controller/EndStop1: now also R3.1; no longer R1.1
- net Controller/Index: now also R1.1; no longer R3.1
- net at R1.2: now also P1.7 (P7); no longer P1.1 (P1)
- net at R2.2: now also P1.6 (P6); no longer P1.2 (P2)
- net at R3.2: now also P1.5 (P5); no longer P1.3 (P3)
- net at R5.2: now also P1.3 (P3); no longer P1.5 (P5)
- net at C2.1, R7.1, R8.2: now also P1.1 (P1); no longer P1.7 (P7)
- net at R6.2: now also P1.2 (P2); no longer P1.6 (P6)
Other:
- moved on the sheet: P1
Changed lines of the file:
@@
 F22 "UART_TX" O L 3350 2400 60
 F23 "UART_RX" I L 3350 2500 60
-F24 "EndStop1" I L 3350 2750 60
+F24 "EndStop1" I L 3350 2950 60
 F25 "EndStop2" I L 3350 2850 60
-F26 "Index" I L 3350 2950 60
+F26 "Index" I L 3350 2750 60
 F27 "MOSI" O R 4850 3400 60
 F28 "MISO" I R 4850 3300 60
@@
 L GND #PWR010
 U 1 1 58665413
-P 1050 3050
-F 0 "#PWR010" H 1050 2800 50  0001 C CNN
-F 1 "GND" H 1050 2900 50  0000 C CNN
-F 2 "" H 1050 3050 50  0000 C CNN
-F 3 "" H 1050 3050 50  0000 C CNN
-	1    1050 3050
-	1    0    0    -1
-$EndComp
-Wire Wire Line
-	1050 2850 950  2850
+P 1100 1650
+F 0 "#PWR010" H 1100 1400 50  0001 C CNN
+F 1 "GND" H 1100 1500 50  0000 C CNN
+F 2 "" H 1100 1650 50  0000 C CNN
+F 3 "" H 1100 1650 50  0000 C CNN
+	1    1100 1650
+	1    0    0    -1
+$EndComp
 $Comp
 L +3V3 #PWR011
 U 1 1 58665925
-P 1250 3050
-F 0 "#PWR011" H 1250 2900 50  0001 C CNN
-F 1 "+3V3" H 1250 3190 50  0000 C CNN
-F 2 "" H 1250 3050 50  0000 C CNN
-F 3 "" H 1250 3050 50  0000 C CNN
-	1    1250 3050
+P 1250 1900
+F 0 "#PWR011" H 1250 1750 50  0001 C CNN
+F 1 "+3V3" H 1250 2040 50  0000 C CNN
+F 2 "" H 1250 1900 50  0000 C CNN
+F 3 "" H 1250 1900 50  0000 C CNN
+	1    1250 1900
 	1    0    0    -1
 $EndComp
@@
 $EndComp
 Wire Wire Line
-	950  2750 1150 2750
-Wire Wire Line
 	2100 2700 2650 2700
 Wire Wire Line
@@
 	2750 2400 2100 2400
 Wire Wire Line
-	3350 2950 2800 2950
-Wire Wire Line
 	2800 2950 2800 2250
 Wire Wire Line
 	2800 2250 2100 2250
 Wire Wire Line
-	3350 2850 2850 2850
-Wire Wire Line
 	2850 2850 2850 2100
 Wire Wire Line
@@
 Wire Wire Line
 	2900 1950 2900 2750
-Wire Wire Line
-	2900 2750 3350 2750
 Wire Wire Line
 	1800 2700 1450 2700
@@
 L GND #PWR013
 U 1 1 586CE0C4
-P 1150 1600
-F 0 "#PWR013" H 1150 1350 50  0001 C CNN
-F 1 "GND" H 1150 1450 50  0000 C CNN
-F 2 "" H 1150 1600 50  0000 C CNN
-F 3 "" H 1150 1600 50  0000 C CNN
-	1    1150 1600
+P 1350 1600
+F 0 "#PWR013" H 1350 1350 50  0001 C CNN
+F 1 "GND" H 1350 1450 50  0000 C CNN
+F 2 "" H 1350 1600 50  0000 C CNN
+F 3 "" H 1350 1600 50  0000 C CNN
+	1    1350 1600
 	1    0    0    -1
 $EndComp
@@
 L +5V #PWR014
 U 1 1 586CE33C
-P 1450 1450
-F 0 "#PWR014" H 1450 1300 50  0001 C CNN
-F 1 "+5V" H 1450 1590 50  0000 C CNN
-F 2 "" H 1450 1450 50  0000 C CNN
-F 3 "" H 1450 1450 50  0000 C CNN
-	1    1450 1450
-	1    0    0    -1
-$EndComp
-Wire Wire Line
-	1050 1450 1150 1450
-Wire Wire Line
-	1150 1450 1150 1600
-Wire Wire Line
-	1050 1350 1250 1350
-Wire Wire Line
-	1250 1350 1250 1550
-Wire Wire Line
-	1250 1550 1450 1550
-Wire Wire Line
-	1450 1550 1450 1450
+P 1600 1450
+F 0 "#PWR014" H 1600 1300 50  0001 C CNN
+F 1 "+5V" H 1600 1590 50  0000 C CNN
+F 2 "" H 1600 1450 50  0000 C CNN
+F 3 "" H 1600 1450 50  0000 C CNN
+	1    1600 1450
+	1    0    0    -1
+$EndComp
+Wire Wire Line
+	1050 1450 1350 1450
+Wire Wire Line
+	1350 1450 1350 1600
+Wire Wire Line
+	1050 1350 1450 1350
+Wire Wire Line
+	1450 1350 1450 1550
+Wire Wire Line
+	1450 1550 1600 1550
+Wire Wire Line
+	1600 1550 1600 1450
 Wire Wire Line
 	3350 2500 2950 2500
@@
 L CONN_01X09 P1
 U 1 1 58736653
-P 750 2450
-F 0 "P1" H 750 2950 50  0000 C CNN
-F 1 "Sensor" V 850 2450 50  0000 C CNN
-F 2 "Pin_Headers:Pin_Header_Angled_1x09" H 750 2450 50  0001 C CNN
-F 3 "" H 750 2450 50  0000 C CNN
-	1    750  2450
-	-1   0    0    -1
-$EndComp
-Wire Wire Line
-	1250 3050 1150 3050
-Wire Wire Line
-	1150 3050 1150 2750
-Wire Wire Line
-	1050 3050 1050 2850
+P 750 2250
+F 0 "P1" H 750 2750 50  0000 C CNN
+F 1 "Sensor" V 850 2250 50  0000 C CNN
+F 2 "Pin_Headers:Pin_Header_Angled_1x09" H 750 2250 50  0001 C CNN
+F 3 "" H 750 2250 50  0000 C CNN
+	1    750  2250
+	-1   0    0    1
+$EndComp
 $Comp
 L +36V #PWR015
@@
 	1000 3600 1100 3600
 Connection ~ 1000 3850
+Wire Wire Line
+	950  1950 1250 1950
+Wire Wire Line
+	1000 1650 1000 1850
+Wire Wire Line
+	1000 1850 950  1850
+Wire Wire Line
+	1250 1950 1250 1900
+Wire Wire Line
+	1000 1650 1100 1650
+Wire Wire Line
+	2900 2750 3350 2750
+Wire Wire Line
+	2850 2850 3350 2850
+Wire Wire Line
+	2800 2950 3350 2950
 $EndSCHEMATC
