File: MotorController2/BMC2.sch (KiCad schematic (older format))
At the start: 28 parts, among them P1 Sensor, P10 GND, P11 I2C, P12 CAN, P2 CAN, P3 DATA, P4 USB_OTG, P5 PhaseA, P6 PhaseB, P7 PhaseC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

Commit message: Work on BOM.
Parts:
- added C45, C46, C47: 1nF 50V, Capacitors_SMD:C_0805_HandSoldering, symbol C
- C1: value 0.1uf (6V min) -> 0.1uF 50V; Farnell (none) -> 1759265
- C2: value 0.1uF -> 0.1uF 50V
- C44: value 0.1uf (6V min) -> 0.1uF 50V
- D1: value 10V -> 60V 2A; Farnell (none) -> 2284958
- P1: Farnell (none) -> 2468365; Plug Farnell (none) -> 1098695
- P12: Farnell (none) -> 588738
- P2: Farnell (none) -> 588738; Farnell Related (none) -> 1098455
- P3: Farnell (none) -> 588740
- R1: Order (none) -> http://uk.farnell.com/multicomp/mcwr08x1001ftl/res-thick-fi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
- R7: value 10k -> 10K
- U1: Order (none) -> http://uk.farnell.com/nxp/tja1042t-3-1j/can-transceiver-aec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
Connections:
- net Controller/HallA: now also C47.1
- net Controller/HallB: now also C46.1
- net Controller/HallC: now also C45.1
- net GND: now also C45.2, C46.2, C47.2
Other:
- moved on the sheet: C2, R1, R2, R3, R4, R5, R6, R7, R8

Commit message: BMCV2.1 updates.
Parts:
- removed P11: I2C, Pin_Headers:Pin_Header_Straight_1x04, symbol CONN_01X04
- removed R3, R8: 1k, Resistors_SMD:R_0805_HandSoldering, symbol R
- added U6, U7: MIC2009A-1YM6TR, TO_SOT_Packages_SMD:SOT-23-6, symbol MIC2009A-1YM6TR
- R1: Order http://uk.farnell.com/multicomp/mcwr08x1001ftl/res-thick-fi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 -> (none)
- R2: value 1k -> 300R
Connections:
- net +3V3: now also U6.1 (VIN); no longer P1.8 (P8)
- net +5V: now also U7.1 (VIN); no longer P3.4 (P4)
- net Controller/EndStop1: now also P1.5 (P5)
- net Controller/EndStop2: now also P1.6 (P6); no longer R2.1
- net Controller/Index: now also P1.7 (P7); no longer R1.1
- net Controller/Temp: now also C2.1, P1.1 (P1), R7.1
- net GND: now also R1.1, R2.1, U6.2 (GND), U7.2 (GND)
- net at R1.2: now also U6.5 (ILIMIT); no longer P1.7 (P7)
- net at R2.2: now also U7.5 (ILIMIT); no longer P1.6 (P6)
- new net: P3.4 (P4), U7.6 (VOUT)
- new net: P1.8 (P8), U6.6 (VOUT)
- new net Controller/FAN_FAULT: U7.4 (FAULT/)
- new net Controller/FanCtrl: U7.3 (ENABLE)
- new net Controller/SENSOR_PWR_FAULT: U6.4 (FAULT/)
- new net Controller/SensorPwrCtrl: U6.3 (ENABLE)
Other:
- note added: "Current limit to 700mA\n"
- note added: "Output limited to 200ma\n"
- moved on the sheet: P3

Commit message: Updates for parts list.
Parts:
- C1: Price (none) -> 0.0224
- C45: Price (none) -> 0.0182
- D1: Price (none) -> 0.425
- P1: MF (none) -> TE Connectivity; MP (none) -> 640457-9; Mouser (none) -> 571-6404579; Price (none) -> 0.266; Supplier (none) -> Mouser
- P10, P5, P6, P7, P9: Supplier (none) -> None
- P2: Price (none) -> 0.101
- P3: Price (none) -> 0.199
- P4: Farnell (none) -> 1125348; MF (none) -> Molex; MP (none) -> 67503-1020; Price (none) -> 0.555
- R2: Farnell (none) -> 2447633; Price (none) -> 0.005
- R4: Farnell (none) -> 2447587; Price (none) -> 0.0062
- R7: Farnell (none) -> 2447553; Price (none) -> 0.0062
- R9: Farnell (none) -> 2447609; Price (none) -> 0.0057
- U1: Farnell (none) -> 2574957; Price (none) -> 0.838
- U6: Availability Good -> (none); Farnell (none) -> 2509888; Price 0.37 USD -> 0.33
Changed lines of the file:
@@
-EESchema Schematic File Version 2
+EESchema Schematic File Version 3
 LIBS:BMC2-rescue
 LIBS:power
 LIBS:device
-LIBS:transistors
-LIBS:conn
 LIBS:linear
 LIBS:regul
-LIBS:74xx
-LIBS:cmos4000
 LIBS:adc-dac
 LIBS:memory
@@
 LIBS:digital-audio
 LIBS:philips
-LIBS:display
 LIBS:cypress
 LIBS:siliconi
@@
 LIBS:atmel
 LIBS:contrib
-LIBS:valves
-LIBS:stm32
 LIBS:Power_Management
 LIBS:motor_drivers
@@
 LIBS:MIC2009A-1YM6TR
 LIBS:BMC2-cache
-EELAYER 25 0
+EELAYER 26 0
 EELAYER END
 $Descr A4 11693 8268
@@
 F 3 "" H 1900 4000 50  0000 C CNN
 F 4 "http://uk.farnell.com/nxp/tja1042t-3-1j/can-transceiver-aec-q100-2mbps/dp/2574957" H 1900 4000 60  0001 C CNN "Order"
+F 5 "2574957" H 1900 4000 60  0001 C CNN "Farnell"
+F 6 "0.838" H 1900 4000 60  0001 C CNN "Price"
 	1    1900 4000
 	-1   0    0    -1
@@
 F 4 "588738" H 750 4000 60  0001 C CNN "Farnell"
 F 5 "1098455" H 750 4000 60  0001 C CNN "Farnell Related"
+F 6 "0.101" H 750 4000 60  0001 C CNN "Price"
 	1    750  4000
 	-1   0    0    -1
@@
 F 3 "" H 1150 5250 50  0000 C CNN
 F 4 "1759265" H 1150 5250 60  0001 C CNN "Farnell"
+F 5 "0.0224" H 1150 5250 60  0001 C CNN "Price"
 	1    1150 5250
 	1    0    0    -1
@@
 F 3 "" V 1950 5250 50  0000 C CNN
 F 4 "http://uk.farnell.com/molex/67503-1020/mini-usb-2-0-otg-type-b-rcpt-smt/dp/1125348" H 2000 5350 60  0001 C CNN "Order"
+F 5 "1125348" H 2000 5350 60  0001 C CNN "Farnell"
+F 6 " 67503-1020" H 2000 5350 60  0001 C CNN "MP"
+F 7 "Molex" H 2000 5350 60  0001 C CNN "MF"
+F 8 "0.555" H 2000 5350 60  0001 C CNN "Price"
 	1    2000 5350
 	0    -1   1    0
@@
 F 2 "Resistors_SMD:R_0805_HandSoldering" V 2730 5150 50  0001 C CNN
 F 3 "" H 2800 5150 50  0000 C CNN
+F 4 "2447609" V 2800 5150 60  0001 C CNN "Farnell"
+F 5 "0.0057" V 2800 5150 60  0001 C CNN "Price"
 	1    2800 5150
 	0    1    1    0
@@
 F 3 "" H 2350 4900 50  0000 C CNN
 F 4 "2284958" H 2350 4900 60  0001 C CNN "Farnell"
+F 5 "0.425" H 2350 4900 60  0001 C CNN "Price"
 	1    2350 4900
 	0    1    1    0
@@
 F 2 "Resistors_SMD:R_0805_HandSoldering" V 1730 2400 50  0001 C CNN
 F 3 "" H 1800 2400 50  0000 C CNN
+F 4 "2447587" V 1800 2400 60  0001 C CNN "Farnell"
+F 5 "0.0062" V 1800 2400 60  0001 C CNN "Price"
 	1    1800 2400
 	0    1    1    0
@@
 F 2 "Resistors_SMD:R_0805_HandSoldering" V 1330 3000 50  0001 C CNN
 F 3 "" H 1400 3000 50  0000 C CNN
+F 4 "2447553" V 1400 3000 60  0001 C CNN "Farnell"
+F 5 "0.0062" V 1400 3000 60  0001 C CNN "Price"
 	1    1400 3000
 	1    0    0    -1
@@
 F 3 "" H 850 900 50  0000 C CNN
 F 4 "588740" H 850 900 60  0001 C CNN "Farnell"
+F 5 "0.199" H 850 900 60  0001 C CNN "Price"
 	1    850  900
 	-1   0    0    -1
@@
 F 2 "Connect:1pin" H 8750 2400 50  0001 C CNN
 F 3 "" H 8750 2400 50  0000 C CNN
+F 4 "None" H 8750 2400 60  0001 C CNN "Supplier"
 	1    8750 2400
 	1    0    0    -1
@@
 F 2 "Connect:1pin" H 8750 2650 50  0001 C CNN
 F 3 "" H 8750 2650 50  0000 C CNN
+F 4 "None" H 8750 2650 60  0001 C CNN "Supplier"
 	1    8750 2650
 	1    0    0    -1
@@
 F 2 "Connect:1pin" H 8750 2900 50  0001 C CNN
 F 3 "" H 8750 2900 50  0000 C CNN
+F 4 "None" H 8750 2900 60  0001 C CNN "Supplier"
 	1    8750 2900
 	1    0    0    -1
@@
 F 4 "2468365" H 750 2250 60  0001 C CNN "Farnell"
 F 5 "1098695" H 750 2250 60  0001 C CNN "Plug Farnell"
+F 6 "Mouser" H 750 2250 60  0001 C CNN "Supplier"
+F 7 "571-6404579" H 750 2250 60  0001 C CNN "Mouser"
+F 8 "TE Connectivity" H 750 2250 60  0001 C CNN "MF"
+F 9 "640457-9" H 750 2250 60  0001 C CNN "MP"
+F 10 "0.266" H 750 2250 60  0001 C CNN "Price"
 	1    750  2250
 	-1   0    0    1
@@
 F 2 "Connect:1pin" H 8400 1350 50  0001 C CNN
 F 3 "" H 8400 1350 50  0000 C CNN
+F 4 "None" H 8400 1350 60  0001 C CNN "Supplier"
 	1    8400 1350
 	1    0    0    -1
@@
 F 2 "Connect:1pin" H 8400 1650 50  0001 C CNN
 F 3 "" H 8400 1650 50  0000 C CNN
+F 4 "None" H 8400 1650 60  0001 C CNN "Supplier"
 	1    8400 1650
 	1    0    0    -1
@@
 F 3 "" H 1950 3050 50  0000 C CNN
 F 4 "9406344" H 1950 3050 60  0001 C CNN "Farnell"
+F 5 "0.0182" H 1950 3050 60  0001 C CNN "Price"
 	1    1950 3050
 	1    0    0    -1
@@
 F 3 "SOT-23-6 Microchip" H 2950 1350 50  0001 L BNN
 F 4 "MIC2009A-1YM6-TR" H 2900 1400 50  0001 L BNN "MP"
-F 5 "Good" H 3000 1700 50  0001 L BNN "Availability"
-F 6 "0.37 USD" H 3050 1600 50  0001 L BNN "Price"
-F 7 "Microchip" H 3100 1500 50  0001 L BNN "MF"
-F 8 "MIC2009 Series 1 Channel 5.5 V Adj. High Side Power Distribution Switch SOT-23-6" H 2700 1100 50  0001 L BNN "Description"
+F 5 "0.33" H 3050 1600 50  0001 L BNN "Price"
+F 6 "Microchip" H 3100 1500 50  0001 L BNN "MF"
+F 7 "MIC2009 Series 1 Channel 5.5 V Adj. High Side Power Distribution Switch SOT-23-6" H 2700 1100 50  0001 L BNN "Description"
+F 8 "2509888" H 2150 1450 60  0001 C CNN "Farnell"
 	1    2150 1450
 	-1   0    0    -1
@@
 F 2 "Resistors_SMD:R_0805_HandSoldering" V 4930 1600 50  0001 C CNN
 F 3 "" H 5000 1600 50  0000 C CNN
+F 4 "2447633" V 5000 1600 60  0001 C CNN "Farnell"
+F 5 "0.005" V 5000 1600 60  0001 C CNN "Price"
 	1    5000 1600
 	-1   0    0    1

Commit message: Add some annotations.
Other:
- note added: "Power to external sensors or fan"
- note added: "The 'Data' connector and be used to interface to \nexternal sensors, and/or power a cooling fan. \n"
- note added: "The CAN bus connections also provide an external supply \nto the board for powering the controller when the main \nmotor supply is disconnected."
Changed lines of the file:
@@
-EESchema Schematic File Version 3
+EESchema Schematic File Version 2
 LIBS:BMC2-rescue
 LIBS:power
 LIBS:device
+LIBS:transistors
+LIBS:conn
 LIBS:linear
 LIBS:regul
+LIBS:74xx
+LIBS:cmos4000
 LIBS:adc-dac
 LIBS:memory
@@
 LIBS:digital-audio
 LIBS:philips
+LIBS:display
 LIBS:cypress
 LIBS:siliconi
@@
 LIBS:atmel
 LIBS:contrib
+LIBS:valves
+LIBS:stm32
 LIBS:Power_Management
 LIBS:motor_drivers
@@
 LIBS:MIC2009A-1YM6TR
 LIBS:BMC2-cache
-EELAYER 26 0
+EELAYER 25 0
 EELAYER END
 $Descr A4 11693 8268
@@
 Text Notes 4700 1750 2    60   ~ 0
 Current limit to 700mA\n
+Text Notes 3550 800  0    60   ~ 0
+Power to external sensors or fan
+Text Notes 700  6400 0    60   ~ 0
+The CAN bus connections also provide an external supply \nto the board for powering the controller when the main \nmotor supply is disconnected.
+Text Notes 1100 700  0    60   ~ 0
+The 'Data' connector and be used to interface to \nexternal sensors, and/or power a cooling fan. \n
 $EndSCHEMATC
