File: MotorController2/power.sch (KiCad schematic (older format))
At the start: 39 parts

Commit message: Most of new motor controller schematic, and leg V2.
Connections:
- net +3V3: no longer C?.1, U?.48 (VREF)
- new net +3.3VADC: C?.1, U?.48 (VREF)
Changed lines of the file:
@@
 LIBS:drv8305
 LIBS:bsc016n06ns
+LIBS:dc-dc
+LIBS:IFX91041EJV33
 LIBS:BMC2-cache
 EELAYER 25 0
@@
 $Descr A4 11693 8268
 encoding utf-8
-Sheet 3 3
+Sheet 3 4
 Title ""
 Date ""
@@
 	1550 2050 1550 1900
 Wire Wire Line
-	1550 1900 2200 1900
-Wire Wire Line
 	3850 1900 3850 1950
 Wire Wire Line
@@
 $EndComp
 Wire Wire Line
-	2000 1950 2000 1900
+	2000 1750 2000 1950
 Connection ~ 2000 1900
 $Comp
@@
 	5450 4150 5450 4050
 Connection ~ 5450 4050
+Wire Wire Line
+	1550 1900 1750 1900
+Wire Wire Line
+	2000 1900 2200 1900
+$Comp
+L +3.3VADC #PWR?
+U 1 1 585F8E91
+P 2000 1750
+F 0 "#PWR?" H 2150 1700 50  0001 C CNN
+F 1 "+3.3VADC" H 2000 1850 50  0000 C CNN
+F 2 "" H 2000 1750 50  0000 C CNN
+F 3 "" H 2000 1750 50  0000 C CNN
+	1    2000 1750
+	1    0    0    -1
+$EndComp
 $EndSCHEMATC

Commit message: Initial schematic complete.
Parts:
- added C?: 0.1uF 5V, symbol C
- added R?: 10K, symbol R
- added TH?: THERMISTOR, symbol THERMISTOR
- added W? (x3): TEST_1P, symbol TEST_1P
- added W?: GHA, symbol TEST_1P
- added W?: GLA, symbol TEST_1P
- added W?: SLA, symbol TEST_1P
- added W?: SHA, symbol TEST_1P
- C?: value 0.1uf 50V -> 0.1uf 50V min
- C? (x2): value 0.1uf 50V -> 0.1uf (Min 50V)
- C? (x2): value 1000pf -> 1nF 5V
- C?: value 1000pf -> 1nf 5V
Connections:
- net +3V3: now also TH?.1
- net GND: now also C?.2, R?.2
- net ISenseA: now also W?.1
- net ISenseB: now also W?.1
- net ISenseC: now also W?.1
- net PhaseA: now also W?.1
- net at C?.1, Q?.1 (S), Q?.2 (S)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: now also W?.1
- net at Q?.4 (G), U?.33 (GLA): now also W?.1
- net at Q?.4 (G), U?.36 (GHA): now also W?.1
- new net TempDrv: C?.1, R?.1, TH?.2

Commit message: Component footprints.
Parts:
- C17, C19, C20, C21, C24, C25, C26, C29, C33, C34, C35: renamed from C?; footprint (none) -> Capacitors_SMD:C_0805_HandSoldering
- C18, C22, C23, C27, C28, C30, C31, C32: renamed from C?; footprint (none) -> Capacitors_SMD:C_1206_HandSoldering
- Q1, Q2, Q3, Q4, Q5, Q6: renamed from Q?; footprint (none) -> SON127P532X615X110-8N:SON127P532X615X110-8N
- R18, R19, R20, R21, R22, R23, R27, R28, R29, R30, R31, R32: renamed from R?; footprint (none) -> Resistors_SMD:R_0805_HandSoldering
- R24: renamed from R?; Order (none) -> http://www.mouser.co.uk/ProductDetail/ROHM-Semiconductor/PS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
- TH1: renamed from TH?; footprint (none) -> Resistors_SMD:R_0805_HandSoldering; Order (none) -> http://uk.farnell.com/epcos/b57620c103j62/thermistor-ntc-10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
- U3: renamed from U?; footprint (none) -> QFP50P900X900X120-49N:QFP50P900X900X120-49N
- W3: renamed from W?; value TEST_1P -> ISenseA; footprint (none) -> Measurement_Points:Measurement_Point_Round-SMD-Pad_Big
- W4: renamed from W?; value TEST_1P -> ISenseB; footprint (none) -> Measurement_Points:Measurement_Point_Round-SMD-Pad_Big
- W5: renamed from W?; value TEST_1P -> ISenseC; footprint (none) -> Measurement_Points:Measurement_Point_Round-SMD-Pad_Big
- W6, W7, W8, W9: renamed from W?; footprint (none) -> Measurement_Points:Measurement_Point_Round-SMD-Pad_Big
- gave numbers to parts that had none: 2
Connections:
- net +3V3: now also R23.1; no longer TH1.1
- net GND: now also TH1.2; no longer R23.2
- net TempDrv: now also R23.2, TH1.1; no longer R23.1, TH1.2
Other:
- moved on the sheet: R23, TH1

Commit message: Add local library.
Parts:
- Q2: Order (none) -> http://www.mouser.co.uk/ProductDetail/Infineon-Technologies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
- R24, R26: footprint (none) -> Local:R_PSR400
- R25: footprint (none) -> Local:R_PSR400; Order (none) -> http://www.mouser.co.uk/ProductDetail/ROHM-Semiconductor/PS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; Order2 (none) -> https://www.digikey.co.uk/product-detail/en/rohm-semiconduc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
Changed lines of the file:
@@
 $EndComp
 $Comp
-L GND #PWR046
+L GND #PWR048
 U 1 1 58539F8F
 P 3350 5250
-F 0 "#PWR046" H 3350 5000 50  0001 C CNN
+F 0 "#PWR048" H 3350 5000 50  0001 C CNN
 F 1 "GND" H 3350 5100 50  0000 C CNN
 F 2 "" H 3350 5250 50  0000 C CNN
@@
 $EndComp
 $Comp
-L +3V3 #PWR047
+L +3V3 #PWR049
 U 1 1 5853A0E8
 P 1750 1900
-F 0 "#PWR047" H 1750 1750 50  0001 C CNN
+F 0 "#PWR049" H 1750 1750 50  0001 C CNN
 F 1 "+3V3" H 1750 2040 50  0000 C CNN
 F 2 "" H 1750 1900 50  0000 C CNN
@@
 $EndComp
 $Comp
-L GND #PWR048
+L GND #PWR050
 U 1 1 58544FF0
 P 2350 1850
-F 0 "#PWR048" H 2350 1600 50  0001 C CNN
+F 0 "#PWR050" H 2350 1600 50  0001 C CNN
 F 1 "GND" H 2350 1700 50  0000 C CNN
 F 2 "" H 2350 1850 50  0000 C CNN
@@
 $EndComp
 $Comp
-L GND #PWR049
+L GND #PWR051
 U 1 1 585451CE
 P 5250 2250
-F 0 "#PWR049" H 5250 2000 50  0001 C CNN
+F 0 "#PWR051" H 5250 2000 50  0001 C CNN
 F 1 "GND" H 5250 2100 50  0000 C CNN
 F 2 "" H 5250 2250 50  0000 C CNN
@@
 $EndComp
 $Comp
-L +36V #PWR050
+L +36V #PWR052
 U 1 1 58545328
 P 5950 1600
-F 0 "#PWR050" H 5950 1450 50  0001 C CNN
+F 0 "#PWR052" H 5950 1450 50  0001 C CNN
 F 1 "+36V" H 5950 1740 50  0000 C CNN
 F 2 "" H 5950 1600 50  0000 C CNN
@@
 F 0 "R26" V 8780 5200 50  0000 C CNN
 F 1 "R001" V 8700 5200 50  0000 C CNN
-F 2 "" V 8630 5200 50  0001 C CNN
+F 2 "Local:R_PSR400" V 8630 5200 50  0001 C CNN
 F 3 "http://uk.farnell.com/welwyn/oars-xp-0r001/resistor-open-air-0r001-3-5w/dp/1292583" H 8700 5200 50  0001 C CNN
 	1    8700 5200
@@
 F 0 "R25" V 8030 5650 50  0000 C CNN
 F 1 "R001" V 7950 5650 50  0000 C CNN
-F 2 "" V 7880 5650 50  0001 C CNN
+F 2 "Local:R_PSR400" V 7880 5650 50  0001 C CNN
 F 3 "" H 7950 5650 50  0000 C CNN
+F 4 "http://www.mouser.co.uk/ProductDetail/ROHM-Semiconductor/PSR400ITQFH1L00/?qs=sGAEpiMZZMtlubZbdhIBICz%2ftfrlArmdMl%252b8hR2qw6A%3d" V 7950 5650 60  0001 C CNN "Order"
+F 5 "https://www.digikey.co.uk/product-detail/en/rohm-semiconductor/PSR400ITQFH1L00/RHM1676-DKR-ND/4864209" V 7950 5650 60  0001 C CNN "Order2"
 	1    7950 5650
 	1    0    0    -1
@@
 F 0 "R24" V 7030 6050 50  0000 C CNN
 F 1 "R001" V 6950 6050 50  0000 C CNN
-F 2 "" V 6880 6050 50  0001 C CNN
+F 2 "Local:R_PSR400" V 6880 6050 50  0001 C CNN
 F 3 "http://www.mouser.com/ds/2/348/psr-951869.pdf" H 6950 6050 50  0001 C CNN
 F 4 "http://www.mouser.co.uk/ProductDetail/ROHM-Semiconductor/PSR400ITQFH1L00/?qs=sGAEpiMZZMtlubZbdhIBICz%2ftfrlArmdMl%252b8hR2qw6A%3d" V 6950 6050 60  0001 C CNN "Order"
@@
 $EndComp
 $Comp
-L GND #PWR051
+L GND #PWR053
 U 1 1 585465EE
 P 7950 6000
-F 0 "#PWR051" H 7950 5750 50  0001 C CNN
+F 0 "#PWR053" H 7950 5750 50  0001 C CNN
 F 1 "GND" H 7950 5850 50  0000 C CNN
 F 2 "" H 7950 6000 50  0000 C CNN
@@
 F 2 "SON127P532X615X110-8N:SON127P532X615X110-8N" H 6850 5100 50  0001 C CIN
 F 3 "" V 6850 4900 50  0000 L CNN
+F 4 "http://www.mouser.co.uk/ProductDetail/Infineon-Technologies/BSC016N06NS/?qs=sGAEpiMZZMshyDBzk1%2fWi6ODfQGXJyDAz3qJRaaNuYk%3d" H 6850 4900 60  0001 C CNN "Order"
 	1    6850 4900
 	1    0    0    -1
 $EndComp
 $Comp
-L +36V #PWR052
+L +36V #PWR054
 U 1 1 58554223
 P 8950 700
-F 0 "#PWR052" H 8950 550 50  0001 C CNN
+F 0 "#PWR054" H 8950 550 50  0001 C CNN
 F 1 "+36V" H 8950 840 50  0000 C CNN
 F 2 "" H 8950 700 50  0000 C CNN
@@
 $EndComp
 $Comp
-L +36V #PWR053
+L +36V #PWR055
 U 1 1 5855565E
 P 8100 2350
-F 0 "#PWR053" H 8100 2200 50  0001 C CNN
+F 0 "#PWR055" H 8100 2200 50  0001 C CNN
 F 1 "+36V" H 8100 2490 50  0000 C CNN
 F 2 "" H 8100 2350 50  0000 C CNN
@@
 $EndComp
 $Comp
-L +36V #PWR054
+L +36V #PWR056
 U 1 1 585563B7
 P 7150 3950
-F 0 "#PWR054" H 7150 3800 50  0001 C CNN
+F 0 "#PWR056" H 7150 3800 50  0001 C CNN
 F 1 "+36V" H 7150 4090 50  0000 C CNN
 F 2 "" H 7150 3950 50  0000 C CNN
@@
 $EndComp
 $Comp
-L GND #PWR055
+L GND #PWR057
 U 1 1 5855C999
 P 9350 2350
-F 0 "#PWR055" H 9350 2100 50  0001 C CNN
+F 0 "#PWR057" H 9350 2100 50  0001 C CNN
 F 1 "GND" H 9350 2200 50  0000 C CNN
 F 2 "" H 9350 2350 50  0000 C CNN
@@
 $EndComp
 $Comp
-L GND #PWR056
+L GND #PWR058
 U 1 1 5855E51E
 P 9350 4100
-F 0 "#PWR056" H 9350 3850 50  0001 C CNN
+F 0 "#PWR058" H 9350 3850 50  0001 C CNN
 F 1 "GND" H 9350 3950 50  0000 C CNN
 F 2 "" H 9350 4100 50  0000 C CNN
@@
 VSenseC
 $Comp
-L GND #PWR057
+L GND #PWR059
 U 1 1 5855F833
 P 9250 5650
-F 0 "#PWR057" H 9250 5400 50  0001 C CNN
+F 0 "#PWR059" H 9250 5400 50  0001 C CNN
 F 1 "GND" H 9250 5500 50  0000 C CNN
 F 2 "" H 9250 5650 50  0000 C CNN
@@
 $EndComp
 $Comp
-L GND #PWR058
+L GND #PWR060
 U 1 1 585560F6
 P 8700 5500
-F 0 "#PWR058" H 8700 5250 50  0001 C CNN
+F 0 "#PWR060" H 8700 5250 50  0001 C CNN
 F 1 "GND" H 8700 5350 50  0000 C CNN
 F 2 "" H 8700 5500 50  0000 C CNN
@@
 $EndComp
 $Comp
-L GND #PWR059
+L GND #PWR061
 U 1 1 58556274
 P 6950 6300
-F 0 "#PWR059" H 6950 6050 50  0001 C CNN
+F 0 "#PWR061" H 6950 6050 50  0001 C CNN
 F 1 "GND" H 6950 6150 50  0000 C CNN
 F 2 "" H 6950 6300 50  0000 C CNN
@@
 $EndComp
 $Comp
-L GND #PWR060
+L GND #PWR062
 U 1 1 58556BEB
 P 7500 4400
-F 0 "#PWR060" H 7500 4150 50  0001 C CNN
+F 0 "#PWR062" H 7500 4150 50  0001 C CNN
 F 1 "GND" H 7500 4250 50  0000 C CNN
 F 2 "" H 7500 4400 50  0000 C CNN
@@
 $EndComp
 $Comp
-L GND #PWR061
+L GND #PWR063
 U 1 1 5855728A
 P 8350 2900
-F 0 "#PWR061" H 8350 2650 50  0001 C CNN
+F 0 "#PWR063" H 8350 2650 50  0001 C CNN
 F 1 "GND" H 8350 2750 50  0000 C CNN
 F 2 "" H 8350 2900 50  0000 C CNN
@@
 $EndComp
 $Comp
-L GND #PWR062
+L GND #PWR064
 U 1 1 5855769F
 P 9300 1250
-F 0 "#PWR062" H 9300 1000 50  0001 C CNN
+F 0 "#PWR064" H 9300 1000 50  0001 C CNN
 F 1 "GND" H 9300 1100 50  0000 C CNN
 F 2 "" H 9300 1250 50  0000 C CNN
@@
 $EndComp
 $Comp
-L GND #PWR063
+L GND #PWR065
 U 1 1 5855A877
 P 3350 6750
-F 0 "#PWR063" H 3350 6500 50  0001 C CNN
+F 0 "#PWR065" H 3350 6500 50  0001 C CNN
 F 1 "GND" H 3350 6600 50  0000 C CNN
 F 2 "" H 3350 6750 50  0000 C CNN
@@
 $EndComp
 $Comp
-L +36V #PWR064
+L +36V #PWR066
 U 1 1 5855A8E8
 P 3350 5800
-F 0 "#PWR064" H 3350 5650 50  0001 C CNN
+F 0 "#PWR066" H 3350 5650 50  0001 C CNN
 F 1 "+36V" H 3350 5940 50  0000 C CNN
 F 2 "" H 3350 5800 50  0000 C CNN
@@
 Connection ~ 2000 1900
 $Comp
-L GND #PWR065
+L GND #PWR067
 U 1 1 5855C539
 P 2000 2300
-F 0 "#PWR065" H 2000 2050 50  0001 C CNN
+F 0 "#PWR067" H 2000 2050 50  0001 C CNN
 F 1 "GND" H 2000 2150 50  0000 C CNN
 F 2 "" H 2000 2300 50  0000 C CNN
@@
 	2200 1900 2000 1900
 $Comp
-L +3.3VADC #PWR066
+L +3.3VADC #PWR068
 U 1 1 585F8E91
 P 2000 1750
-F 0 "#PWR066" H 2150 1700 50  0001 C CNN
+F 0 "#PWR068" H 2150 1700 50  0001 C CNN
 F 1 "+3.3VADC" H 2000 1850 50  0000 C CNN
 F 2 "" H 2000 1750 50  0000 C CNN
@@
 $EndComp
 $Comp
-L GND #PWR067
+L GND #PWR069
 U 1 1 587114E5
 P 5450 7600
-F 0 "#PWR067" H 5450 7350 50  0001 C CNN
+F 0 "#PWR069" H 5450 7350 50  0001 C CNN
 F 1 "GND" H 5450 7450 50  0000 C CNN
 F 2 "" H 5450 7600 50  0000 C CNN
@@
 	4650 7050 5000 7050
 $Comp
-L +3V3 #PWR068
+L +3V3 #PWR070
 U 1 1 58712CAE
 P 5450 6450
-F 0 "#PWR068" H 5450 6300 50  0001 C CNN
+F 0 "#PWR070" H 5450 6300 50  0001 C CNN
 F 1 "+3V3" H 5450 6590 50  0000 C CNN
 F 2 "" H 5450 6450 50  0000 C CNN
@@
 	5450 6550 5450 6450
 $Comp
-L PWR_FLAG #FLG069
+L PWR_FLAG #FLG071
 U 1 1 58764F41
 P 2900 1450
-F 0 "#FLG069" H 2900 1545 50  0001 C CNN
+F 0 "#FLG071" H 2900 1545 50  0001 C CNN
 F 1 "PWR_FLAG" H 2900 1630 50  0000 C CNN
 F 2 "" H 2900 1450 50  0000 C CNN
@@
 Connection ~ 2900 1500
 $Comp
-L PWR_FLAG #FLG070
+L PWR_FLAG #FLG072
 U 1 1 58765140
 P 2900 1750
-F 0 "#FLG070" H 2900 1845 50  0001 C CNN
+F 0 "#FLG072" H 2900 1845 50  0001 C CNN
 F 1 "PWR_FLAG" H 2900 1930 50  0000 C CNN
 F 2 "" H 2900 1750 50  0000 C CNN
@@
 Connection ~ 2850 1750
 $Comp
-L PWR_FLAG #FLG071
+L PWR_FLAG #FLG073
 U 1 1 587653A1
 P 5000 2450
-F 0 "#FLG071" H 5000 2545 50  0001 C CNN
+F 0 "#FLG073" H 5000 2545 50  0001 C CNN
 F 1 "PWR_FLAG" H 5000 2630 50  0000 C CNN
 F 2 "" H 5000 2450 50  0000 C CNN

Commit message: Work on PCB layout.
Parts:
- C30: value 0.1uf 50V min -> 1uF 50V
- C31, C32: value 0.1uf (Min 50V) -> 1uF 50V
Other:
- moved on the sheet: C18, C19
Changed lines of the file:
@@
 U 1 1 58544790
 P 2600 1750
-F 0 "C20" H 2625 1850 50  0000 L CNN
+F 0 "C20" V 2650 1850 50  0000 L CNN
 F 1 "1uf 6.3V" V 2750 1600 50  0000 L CNN
 F 2 "Capacitors_SMD:C_0805_HandSoldering" H 2638 1600 50  0001 C CNN
@@
 L C C19
 U 1 1 585447EA
-P 2600 1500
-F 0 "C19" H 2625 1600 50  0000 L CNN
-F 1 "1uf 6.3V" V 2750 1400 50  0000 L CNN
-F 2 "Capacitors_SMD:C_0805_HandSoldering" H 2638 1350 50  0001 C CNN
-F 3 "" H 2600 1500 50  0000 C CNN
-	1    2600 1500
+P 2600 1400
+F 0 "C19" V 2650 1500 50  0000 L CNN
+F 1 "1uf 6.3V" V 2750 1250 50  0000 L CNN
+F 2 "Capacitors_SMD:C_0805_HandSoldering" H 2638 1250 50  0001 C CNN
+F 3 "" H 2600 1400 50  0000 C CNN
+	1    2600 1400
 	0    1    1    0
 $EndComp
@@
 L C C18
 U 1 1 58544849
-P 2600 1200
-F 0 "C18" H 2625 1300 50  0000 L CNN
-F 1 "1uf 16V" V 2750 1050 50  0000 L CNN
-F 2 "Capacitors_SMD:C_1206_HandSoldering" H 2638 1050 50  0001 C CNN
-F 3 "" H 2600 1200 50  0000 C CNN
-	1    2600 1200
+P 2600 1050
+F 0 "C18" V 2625 1150 50  0000 L CNN
+F 1 "1uf 16V" V 2750 900 50  0000 L CNN
+F 2 "Capacitors_SMD:C_1206_HandSoldering" H 2638 900 50  0001 C CNN
+F 3 "" H 2600 1050 50  0000 C CNN
+	1    2600 1050
 	0    1    1    0
 $EndComp
@@
 P 7500 4200
 F 0 "C30" H 7525 4300 50  0000 L CNN
-F 1 "0.1uf 50V min" H 7525 4100 50  0000 L CNN
+F 1 "1uF 50V" H 7525 4100 50  0000 L CNN
 F 2 "Capacitors_SMD:C_1206_HandSoldering" H 7538 4050 50  0001 C CNN
 F 3 "" H 7500 4200 50  0000 C CNN
@@
 P 8350 2650
 F 0 "C31" H 8375 2750 50  0000 L CNN
-F 1 "0.1uf (Min 50V)" H 8375 2550 50  0000 L CNN
+F 1 "1uF 50V" H 8375 2550 50  0000 L CNN
 F 2 "Capacitors_SMD:C_1206_HandSoldering" H 8388 2500 50  0001 C CNN
 F 3 "" H 8350 2650 50  0000 C CNN
@@
 P 9300 1000
 F 0 "C32" H 9325 1100 50  0000 L CNN
-F 1 "0.1uf (Min 50V)" H 9325 900 50  0000 L CNN
+F 1 "1uF 50V" H 9325 900 50  0000 L CNN
 F 2 "Capacitors_SMD:C_1206_HandSoldering" H 9338 850 50  0001 C CNN
 F 3 "" H 9300 1000 50  0000 C CNN
@@
 	3400 1350 3400 1900
 Wire Wire Line
-	3000 1500 3000 1900
-Wire Wire Line
-	2850 1900 2850 1750
-Wire Wire Line
-	2750 1750 2900 1750
-Wire Wire Line
-	2750 1500 3000 1500
-Wire Wire Line
-	2750 1200 3150 1200
-Wire Wire Line
-	3150 1200 3150 1900
-Wire Wire Line
-	2450 1200 2350 1200
-Wire Wire Line
-	2350 1200 2350 1850
-Wire Wire Line
-	2350 1500 2450 1500
+	3000 1400 3000 1900
+Wire Wire Line
+	2850 1750 2850 1900
+Wire Wire Line
+	2850 1750 2750 1750
+Wire Wire Line
+	2750 1400 3000 1400
+Wire Wire Line
+	2750 1050 3150 1050
+Wire Wire Line
+	3150 1050 3150 1900
+Wire Wire Line
+	2450 1050 2350 1050
+Wire Wire Line
+	2350 1050 2350 1850
+Wire Wire Line
+	2350 1400 2450 1400
 Wire Wire Line
 	2350 1750 2450 1750
-Connection ~ 2350 1500
+Connection ~ 2350 1400
 Connection ~ 2350 1750
 Wire Wire Line
@@
 L PWR_FLAG #FLG071
 U 1 1 58764F41
-P 2900 1450
-F 0 "#FLG071" H 2900 1545 50  0001 C CNN
-F 1 "PWR_FLAG" H 2900 1630 50  0000 C CNN
-F 2 "" H 2900 1450 50  0000 C CNN
-F 3 "" H 2900 1450 50  0000 C CNN
-	1    2900 1450
-	1    0    0    -1
-$EndComp
-Wire Wire Line
-	2900 1450 2900 1500
-Connection ~ 2900 1500
+P 2950 1350
+F 0 "#FLG071" H 2950 1445 50  0001 C CNN
+F 1 "PWR_FLAG" H 3150 1350 50  0000 C CNN
+F 2 "" H 2950 1350 50  0000 C CNN
+F 3 "" H 2950 1350 50  0000 C CNN
+	1    2950 1350
+	1    0    0    -1
+$EndComp
+Wire Wire Line
+	2950 1350 2950 1400
+Connection ~ 2950 1400
 $Comp
 L PWR_FLAG #FLG072
 U 1 1 58765140
-P 2900 1750
-F 0 "#FLG072" H 2900 1845 50  0001 C CNN
-F 1 "PWR_FLAG" H 2900 1930 50  0000 C CNN
-F 2 "" H 2900 1750 50  0000 C CNN
-F 3 "" H 2900 1750 50  0000 C CNN
-	1    2900 1750
-	1    0    0    -1
-$EndComp
+P 2850 1750
+F 0 "#FLG072" H 2850 1845 50  0001 C CNN
+F 1 "PWR_FLAG" H 3150 1850 50  0000 C CNN
+F 2 "" H 2850 1750 50  0000 C CNN
+F 3 "" H 2850 1750 50  0000 C CNN
+	1    2850 1750
+	1    0    0    -1
+$EndComp

Commit message: Laying out power section.
Parts:
- Q1, Q2, Q3, Q4, Q5, Q6: footprint SON127P532X615X110-8N:SON127P532X615X110-8N -> Local:SON127P532X615X110-8N
- W3, W4, W5, W6, W7, W8, W9: footprint Measurement_Points:Measurement_Point_Round-SMD-Pad_Big -> Measurement_Points:Measurement_Point_Round-SMD-Pad_Small
Changed lines of the file:
@@
 EESchema Schematic File Version 2
+LIBS:BMC2-rescue
 LIBS:power
 LIBS:device
@@
 LIBS:IFX91041EJV33
 LIBS:BMC2-cache
-EELAYER 25 0
+EELAYER 26 0
 EELAYER END
 $Descr A4 11693 8268
@@
 F 0 "Q3" H 7600 3100 50  0000 L CNN
 F 1 "BSC016N06NS" H 7600 2550 50  0000 L CNN
-F 2 "SON127P532X615X110-8N:SON127P532X615X110-8N" H 7800 3000 50  0001 C CIN
+F 2 "Local:SON127P532X615X110-8N" H 7800 3000 50  0001 C CIN
 F 3 "" V 7800 2800 50  0000 L CNN
 	1    7800 2800
@@
 F 0 "Q4" H 7600 3750 50  0000 L CNN
 F 1 "BSC016N06NS" H 7600 3200 50  0000 L CNN
-F 2 "SON127P532X615X110-8N:SON127P532X615X110-8N" H 7800 3650 50  0001 C CIN
+F 2 "Local:SON127P532X615X110-8N" H 7800 3650 50  0001 C CIN
 F 3 "http://uk.farnell.com/infineon/bsc016n06ns/mosfet-n-ch-60v-100a-tdson-8/dp/2432702" V 7800 3450 50  0001 L CNN
 	1    7800 3450
@@
 F 0 "Q6" H 8450 2150 50  0000 L CNN
 F 1 "BSC016N06NS" H 8450 1600 50  0000 L CNN
-F 2 "SON127P532X615X110-8N:SON127P532X615X110-8N" H 8650 2050 50  0001 C CIN
+F 2 "Local:SON127P532X615X110-8N" H 8650 2050 50  0001 C CIN
 F 3 "" V 8650 1850 50  0000 L CNN
 	1    8650 1850
@@
 F 0 "Q5" H 8450 1450 50  0000 L CNN
 F 1 "BSC016N06NS" H 8450 900 50  0000 L CNN
-F 2 "SON127P532X615X110-8N:SON127P532X615X110-8N" H 8650 1350 50  0001 C CIN
+F 2 "Local:SON127P532X615X110-8N" H 8650 1350 50  0001 C CIN
 F 3 "" V 8650 1150 50  0000 L CNN
 	1    8650 1150
@@
 F 0 "Q1" H 6650 4550 50  0000 L CNN
 F 1 "BSC016N06NS" H 6650 4000 50  0000 L CNN
-F 2 "SON127P532X615X110-8N:SON127P532X615X110-8N" H 6850 4450 50  0001 C CIN
+F 2 "Local:SON127P532X615X110-8N" H 6850 4450 50  0001 C CIN
 F 3 "" V 6850 4250 50  0000 L CNN
 	1    6850 4250
@@
 F 0 "Q2" H 6650 5200 50  0000 L CNN
 F 1 "BSC016N06NS" H 6650 4650 50  0000 L CNN
-F 2 "SON127P532X615X110-8N:SON127P532X615X110-8N" H 6850 5100 50  0001 C CIN
+F 2 "Local:SON127P532X615X110-8N" H 6850 5100 50  0001 C CIN
 F 3 "" V 6850 4900 50  0000 L CNN
 F 4 "http://www.mouser.co.uk/ProductDetail/Infineon-Technologies/BSC016N06NS/?qs=sGAEpiMZZMshyDBzk1%2fWi6ODfQGXJyDAz3qJRaaNuYk%3d" H 6850 4900 60  0001 C CNN "Order"
@@
 F 0 "W5" H 2250 5320 50  0000 C CNN
 F 1 "ISenseC" H 2250 5250 50  0000 C CNN
-F 2 "Measurement_Points:Measurement_Point_Round-SMD-Pad_Big" H 2450 5050 50  0001 C CNN
+F 2 "Measurement_Points:Measurement_Point_Round-SMD-Pad_Small" H 2450 5050 50  0001 C CNN
 F 3 "" H 2450 5050 50  0000 C CNN
 	1    2250 5050
@@
 F 0 "W4" H 1850 5320 50  0000 C CNN
 F 1 "ISenseB" H 1850 5250 50  0000 C CNN
-F 2 "Measurement_Points:Measurement_Point_Round-SMD-Pad_Big" H 2050 5050 50  0001 C CNN
+F 2 "Measurement_Points:Measurement_Point_Round-SMD-Pad_Small" H 2050 5050 50  0001 C CNN
 F 3 "" H 2050 5050 50  0000 C CNN
 	1    1850 5050
@@
 F 0 "W3" H 1500 5320 50  0000 C CNN
 F 1 "ISenseA" H 1500 5250 50  0000 C CNN
-F 2 "Measurement_Points:Measurement_Point_Round-SMD-Pad_Big" H 1700 5050 50  0001 C CNN
+F 2 "Measurement_Points:Measurement_Point_Round-SMD-Pad_Small" H 1700 5050 50  0001 C CNN
 F 3 "" H 1700 5050 50  0000 C CNN
 	1    1500 5050
@@
 F 0 "W7" H 7600 1420 50  0000 C CNN
 F 1 "GHA" H 7600 1350 50  0000 C CNN
-F 2 "Measurement_Points:Measurement_Point_Round-SMD-Pad_Big" H 7800 1150 50  0001 C CNN
+F 2 "Measurement_Points:Measurement_Point_Round-SMD-Pad_Small" H 7800 1150 50  0001 C CNN
 F 3 "" H 7800 1150 50  0000 C CNN
 	1    7600 1150
@@
 F 0 "W8" H 7650 2070 50  0000 C CNN
 F 1 "GLA" H 7650 2000 50  0000 C CNN
-F 2 "Measurement_Points:Measurement_Point_Round-SMD-Pad_Big" H 7850 1800 50  0001 C CNN
+F 2 "Measurement_Points:Measurement_Point_Round-SMD-Pad_Small" H 7850 1800 50  0001 C CNN
 F 3 "" H 7850 1800 50  0000 C CNN
 	1    7650 1800
@@
 F 0 "W9" H 8850 2820 50  0000 C CNN
 F 1 "SLA" H 8850 2750 50  0000 C CNN
-F 2 "Measurement_Points:Measurement_Point_Round-SMD-Pad_Big" H 9050 2550 50  0001 C CNN
+F 2 "Measurement_Points:Measurement_Point_Round-SMD-Pad_Small" H 9050 2550 50  0001 C CNN
 F 3 "" H 9050 2550 50  0000 C CNN
 	1    8850 2550
@@
 F 0 "W6" H 7100 2070 50  0000 C CNN
 F 1 "SHA" H 7100 2000 50  0000 C CNN
-F 2 "Measurement_Points:Measurement_Point_Round-SMD-Pad_Big" H 7300 1800 50  0001 C CNN
+F 2 "Measurement_Points:Measurement_Point_Round-SMD-Pad_Small" H 7300 1800 50  0001 C CNN
 F 3 "" H 7300 1800 50  0000 C CNN
 	1    7100 1800

Commit message: More of the layout done.
Parts:
- removed R24, R25, R26: R001, Local:R_PSR400, symbol R
- removed W6: SHA, Measurement_Points:Measurement_Point_Round-SMD-Pad_Small, symbol TEST_1P
- removed W9: SLA, Measurement_Points:Measurement_Point_Round-SMD-Pad_Small, symbol TEST_1P
- added R24, R25, R26: R001, Local:R_PSR400_SENSE, symbol R_Shunt
Connections:
- net GND: now also R24.4, R25.4, R26.4; no longer C24.2, C26.2, C29.2, U3.19 (SN3), U3.21 (SN2), U3.23 (SN1)
- net at Q2.1 (S), Q2.2 (S), Q2.3 (S)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: now also R24.1; no longer C24.1, U3.20 (SP3)
- net at Q4.1 (S), Q4.2 (S), Q4.3 (S)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: now also R25.1; no longer C26.1, U3.22 (SP2)
- net at Q6.1 (S), Q6.2 (S), Q6.3 (S)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: now also R26.1; no longer C29.1, U3.24 (SP1)
- new net: C24.2, R24.3, U3.19 (SN3)
- new net: C24.1, R24.2, U3.20 (SP3)
- new net: C26.2, R25.3, U3.21 (SN2)
- new net: C26.1, R25.2, U3.22 (SP2)
- new net: C29.2, R26.3, U3.23 (SN1)
- new net: C29.1, R26.2, U3.24 (SP1)
