File: MotorController2/power.sch (KiCad schematic (older format))
At the start: 47 parts, among them Q1 BSC016N06NS, Q2 BSC016N06NS, Q3 BSC016N06NS, Q4 BSC016N06NS, Q5 BSC016N06NS, Q6 BSC016N06NS, U3 DRV8305

Commit message: Work on BOM.
Parts:
- C17: value 1uF 4V -> 1uF 50V; Notes (none) -> 4V required
- C18: value 1uf 16V -> 1uF 100V; Farnell (none) -> 2320876; Notes (none) -> 16V
- C19, C20: value 1uf 6.3V -> 1uF 50V; Notes (none) -> 6.3V
- C21, C25: value 0.1uF 5V -> 0.1uF 50V
- C22: value 0.047uf 90V -> 47nF 200V; Farnell (none) -> 1855874
- C23: value 0.047uf 45v -> 47nF 200V; Farnell (none) -> 1855874; Notes (none) -> 45V
- C24, C26: value 1nF 5V -> 1nF 50V; Farnell (none) -> 9406344
- C27: value 2.2uf 16V -> 2.2uF 50V; Farnell (none) -> 1797017; Notes (none) -> 16V
- C28: value 4.7uF 45V -> 4.7uF 100V; Farnell (none) -> 1797017; Notes (none) -> 45V
- C29: value 1nf 5V -> 1nF 50V; Farnell (none) -> 9406344
- C30, C31, C32: value 1uF 50V -> 1uF 100V; Farnell (none) -> 2320876
- C33, C34, C35: Farnell (none) -> 2581093
- TH1: value THERMISTOR -> NTC 10K; Farnell (none) -> 2103179; Order http://uk.farnell.com/epcos/b57620c103j62/thermistor-ntc-10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 -> http://uk.farnell.com/vishay/ntcs0805e3103jlt/thermistor-10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

Commit message: BMCV2.1 updates.
Parts:
- removed R18, R19: 10K, Resistors_SMD:R_0805_HandSoldering, symbol R
- added C48, C49, C50: 100pF 50V, Capacitors_SMD:C_0805_HandSoldering, symbol C
- added R14, R3, R8: 1K, Resistors_SMD:R_0805_HandSoldering, symbol R
- added W11: GLB, Measurement_Points:Measurement_Point_Round-SMD-Pad_Small, symbol TEST_1P
- added W14: GHB, Measurement_Points:Measurement_Point_Round-SMD-Pad_Small, symbol TEST_1P
- added W6: GLC, Measurement_Points:Measurement_Point_Round-SMD-Pad_Small, symbol TEST_1P
- added W9: GHC, Measurement_Points:Measurement_Point_Round-SMD-Pad_Small, symbol TEST_1P
- C21: value 0.1uF 50V -> 10nF 50V
Connections:
- net GND: now also C48.2, C49.2, C50.2
- net ISenseA: now also C48.1, R3.2; no longer U3.16 (SO1), W3.1
- net ISenseB: now also C49.1, R8.2; no longer U3.17 (SO2), W4.1
- net ISenseC: now also C50.1, R14.2; no longer U3.18 (SO3), W5.1
- net at Q2.4 (G), U3.25 (GLC): now also W6.1
- net at Q1.4 (G), U3.28 (GHC): now also W9.1
- net at Q3.4 (G), U3.29 (GHB): now also W14.1
- net at Q4.4 (G), U3.32 (GLB): now also W11.1
- new net: R3.1, U3.16 (SO1), W3.1
- new net: R8.1, U3.17 (SO2), W4.1
- new net: R14.1, U3.18 (SO3), W5.1
Other:
- moved on the sheet: W3, W4, W5

Commit message: Updates for parts list.
Parts:
- C18: Price (none) -> 0.259
- C20: Price (none) -> 0.0617
- C21: Farnell (none) -> 1414662; Price (none) -> 0.0186
- C23: Price (none) -> 0.112
- C27: Farnell 1797017 -> 1288208; Price (none) -> 0.253
- C28: Farnell 1797017 -> 2310265; MF (none) -> AVX; MP (none) -> 12061Z475KAT2A; Price (none) -> 1.19
- C35: Price (none) -> 0.102
- C48: Farnell 9406344 -> 499687; Price (none) -> 0.0184
- C49, C50: Farnell 9406344 -> 499687
- Q5: Farnell2 (none) -> 2432702; Mouser (none) -> 726-BSC016N06NS; Price (none) -> 1.49; Supplier (none) -> Mouser
- R22: Farnell (none) -> 2447552; Price (none) -> 0.0062
- R26: Farnell (none) -> 2475107; MF (none) -> ROHM; MP (none) -> PSR400ITQFH1L00; Price (none) -> 1.20
- R29: Farnell (none) -> 2447646; Price (none) -> 0.0061
- R30: Farnell (none) -> 2073731; Price (none) -> 0.0178
- TH1: Price (none) -> 0.307
- U3: Farnell (none) -> 2611246; Price (none) -> 4.06
Changed lines of the file:
@@
-EESchema Schematic File Version 2
+EESchema Schematic File Version 3
 LIBS:BMC2-rescue
 LIBS:power
 LIBS:device
-LIBS:transistors
-LIBS:conn
 LIBS:linear
 LIBS:regul
-LIBS:74xx
-LIBS:cmos4000
 LIBS:adc-dac
 LIBS:memory
@@
 LIBS:digital-audio
 LIBS:philips
-LIBS:display
 LIBS:cypress
 LIBS:siliconi
@@
 LIBS:atmel
 LIBS:contrib
-LIBS:valves
-LIBS:stm32
 LIBS:Power_Management
 LIBS:motor_drivers
@@
 LIBS:MIC2009A-1YM6TR
 LIBS:BMC2-cache
-EELAYER 25 0
+EELAYER 26 0
 EELAYER END
 $Descr A4 11693 8268
@@
 F 2 "QFP50P900X900X120-49N:QFP50P900X900X120-49N" H 3300 2850 60  0001 C CNN
 F 3 "" H 3300 2850 60  0001 C CNN
+F 4 "2611246" H 3200 3350 60  0001 C CNN "Farnell"
+F 5 "4.06" H 3200 3350 60  0001 C CNN "Price"
 	1    3200 3350
 	1    0    0    -1
@@
 F 4 "45V" H 3850 1800 60  0001 C CNN "Notes"
 F 5 "1855874" H 3850 1800 60  0001 C CNN "Farnell"
+F 6 "0.112" H 3850 1800 60  0001 C CNN "Price"
 	1    3850 1800
 	1    0    0    -1
@@
 F 3 "" H 2600 1750 50  0000 C CNN
 F 4 "6.3V" V 2600 1750 60  0001 C CNN "Notes"
+F 5 "0.0617" V 2600 1750 60  0001 C CNN "Price"
 	1    2600 1750
 	0    1    1    0
@@
 F 4 "16V" V 2600 1050 60  0001 C CNN "Notes"
 F 5 "2320876" V 2600 1050 60  0001 C CNN "Farnell"
+F 6 "0.259" V 2600 1050 60  0001 C CNN "Price"
 	1    2600 1050
 	0    1    1    0
@@
 F 3 "" H 5250 1600 50  0000 C CNN
 F 4 "16V" H 5250 1600 60  0001 C CNN "Notes"
-F 5 "1797017" H 5250 1600 60  0001 C CNN "Farnell"
+F 5 "1288208" H 5250 1600 60  0001 C CNN "Farnell"
+F 6 "0.253" H 5250 1600 60  0001 C CNN "Price"
 	1    5250 1600
 	1    0    0    -1
@@
 F 3 "" H 5250 2050 50  0000 C CNN
 F 4 "45V" H 5250 2050 60  0001 C CNN "Notes"
-F 5 "1797017" H 5250 2050 60  0001 C CNN "Farnell"
+F 5 "2310265" H 5250 2050 60  0001 C CNN "Farnell"
+F 6 "12061Z475KAT2A" H 5250 2050 60  0001 C CNN "MP"
+F 7 "AVX" H 5250 2050 60  0001 C CNN "MF"
+F 8 "1.19" H 5250 2050 60  0001 C CNN "Price"
 	1    5250 2050
 	1    0    0    -1
@@
 F 2 "Resistors_SMD:R_0805_HandSoldering" V 5180 2550 50  0001 C CNN
 F 3 "" H 5250 2550 50  0000 C CNN
+F 4 "2447552" V 5250 2550 60  0001 C CNN "Farnell"
+F 5 "0.0062" V 5250 2550 60  0001 C CNN "Price"
 	1    5250 2550
 	0    1    1    0
@@
 F 2 "Local:SON127P532X615X110-8N" H 8650 1350 50  0001 C CIN
 F 3 "" V 8650 1150 50  0000 L CNN
+F 4 "2432702" H 8650 1150 60  0001 C CNN "Farnell2"
+F 5 "Mouser" H 8650 1150 60  0001 C CNN "Supplier"
+F 6 "726-BSC016N06NS" H 8650 1150 60  0001 C CNN "Mouser"
+F 7 "1.49" H 8650 1150 60  0001 C CNN "Price"
 	1    8650 1150
 	1    0    0    -1
@@
 F 2 "Resistors_SMD:R_0805_HandSoldering" V 9280 1700 50  0001 C CNN
 F 3 "" H 9350 1700 50  0000 C CNN
+F 4 "2447646" V 9350 1700 60  0001 C CNN "Farnell"
+F 5 "0.0061" V 9350 1700 60  0001 C CNN "Price"
 	1    9350 1700
 	1    0    0    -1
@@
 F 2 "Resistors_SMD:R_0805_HandSoldering" V 9280 2100 50  0001 C CNN
 F 3 "" H 9350 2100 50  0000 C CNN
+F 4 "2073731" V 9350 2100 60  0001 C CNN "Farnell"
+F 5 "0.0178" V 9350 2100 60  0001 C CNN "Price"
 	1    9350 2100
 	1    0    0    -1
@@
 F 3 "" H 9600 3850 50  0000 C CNN
 F 4 "2581093" H 9600 3850 60  0001 C CNN "Farnell"
+F 5 "0.102" H 9600 3850 60  0001 C CNN "Price"
 	1    9600 3850
 	1    0    0    -1
@@
 F 2 "Capacitors_SMD:C_0805_HandSoldering" H 3138 6350 50  0001 C CNN
 F 3 "" H 3100 6500 50  0000 C CNN
+F 4 "1414662 " H 3100 6500 60  0001 C CNN "Farnell"
+F 5 "0.0186" H 3100 6500 60  0001 C CNN "Price"
 	1    3100 6500
 	1    0    0    -1
@@
 F 4 "http://uk.farnell.com/vishay/ntcs0805e3103jlt/thermistor-10k-5-smd-ntc/dp/2103179" V 5450 7200 60  0001 C CNN "Order"
 F 5 "2103179" V 5450 7200 60  0001 C CNN "Farnell"
+F 6 "0.307" V 5450 7200 60  0001 C CNN "Price"
 	1    5450 7200
 	1    0    0    -1
@@
 F 2 "Local:R_PSR400_SENSE" H 8612 5059 50  0001 R CNN
 F 3 "" H 8700 5150 50  0000 C CNN
+F 4 "2475107" H 8700 5150 60  0001 C CNN "Farnell"
+F 5 "PSR400ITQFH1L00" H 8700 5150 60  0001 C CNN "MP"
+F 6 "ROHM" H 8700 5150 60  0001 C CNN "MF"
+F 7 "1.20" H 8700 5150 60  0001 C CNN "Price"
 	1    8700 5150
 	-1   0    0    -1
@@
 F 2 "Capacitors_SMD:C_0805_HandSoldering" H 1188 4250 50  0001 C CNN
 F 3 "" H 1150 4400 50  0000 C CNN
-F 4 "9406344" H 1150 4400 60  0001 C CNN "Farnell"
+F 4 "499687" H 1150 4400 60  0001 C CNN "Farnell"
+F 5 "0.0184" H 1150 4400 60  0001 C CNN "Price"
 	1    1150 4400
 	1    0    0    -1
@@
 F 2 "Capacitors_SMD:C_0805_HandSoldering" H 1188 4850 50  0001 C CNN
 F 3 "" H 1150 5000 50  0000 C CNN
-F 4 "9406344" H 1150 5000 60  0001 C CNN "Farnell"
+F 4 "499687" H 1150 5000 60  0001 C CNN "Farnell"
 	1    1150 5000
 	1    0    0    -1
@@
 F 2 "Capacitors_SMD:C_0805_HandSoldering" H 1188 5600 50  0001 C CNN
 F 3 "" H 1150 5750 50  0000 C CNN
-F 4 "9406344" H 1150 5750 60  0001 C CNN "Farnell"
+F 4 "499687" H 1150 5750 60  0001 C CNN "Farnell"
 	1    1150 5750
 	1    0    0    -1

Commit message: Update part number.
Parts:
- C48: Farnell 499687 -> 1759203; Notes (none) -> +/- 5%
- C49, C50: Farnell 499687 -> (none)
Changed lines of the file:
@@
 F 2 "Capacitors_SMD:C_0805_HandSoldering" H 1188 4250 50  0001 C CNN
 F 3 "" H 1150 4400 50  0000 C CNN
-F 4 "499687" H 1150 4400 60  0001 C CNN "Farnell"
+F 4 "1759203 " H 1150 4400 60  0001 C CNN "Farnell"
 F 5 "0.0184" H 1150 4400 60  0001 C CNN "Price"
+F 6 "+/- 5%" H 1150 4400 60  0001 C CNN "Notes"
 	1    1150 4400
 	1    0    0    -1
@@
 F 2 "Capacitors_SMD:C_0805_HandSoldering" H 1188 4850 50  0001 C CNN
 F 3 "" H 1150 5000 50  0000 C CNN
-F 4 "499687" H 1150 5000 60  0001 C CNN "Farnell"
 	1    1150 5000
 	1    0    0    -1
@@
 F 2 "Capacitors_SMD:C_0805_HandSoldering" H 1188 5600 50  0001 C CNN
 F 3 "" H 1150 5750 50  0000 C CNN
-F 4 "499687" H 1150 5750 60  0001 C CNN "Farnell"
 	1    1150 5750
 	1    0    0    -1

Commit message: Add some annotations.
Other:
- note added: "TH1 is placed near the drive transistors."
- note added: "The filters on the current sense lines \nwere added in a hope to reduce noise \nin the current readings, but have had \nlittle impact."
Changed lines of the file:
@@
-EESchema Schematic File Version 3
+EESchema Schematic File Version 2
 LIBS:BMC2-rescue
 LIBS:power
 LIBS:device
+LIBS:transistors
+LIBS:conn
 LIBS:linear
 LIBS:regul
+LIBS:74xx
+LIBS:cmos4000
 LIBS:adc-dac
 LIBS:memory
@@
 LIBS:digital-audio
 LIBS:philips
+LIBS:display
 LIBS:cypress
 LIBS:siliconi
@@
 LIBS:atmel
 LIBS:contrib
+LIBS:valves
+LIBS:stm32
 LIBS:Power_Management
 LIBS:motor_drivers
@@
 LIBS:MIC2009A-1YM6TR
 LIBS:BMC2-cache
-EELAYER 26 0
+EELAYER 25 0
 EELAYER END
 $Descr A4 11693 8268
@@
 	6300 4900 6300 5000
 Connection ~ 6300 5000
+Text Notes 3350 7650 0    60   ~ 0
+TH1 is placed near the drive transistors.
+Text Notes 1350 6050 0    60   ~ 0
+The filters on the current sense lines \nwere added in a hope to reduce noise \nin the current readings, but have had \nlittle impact.
 $EndSCHEMATC
