File: MotorController2/BMC2.kicad_pcb (KiCad board)
At the start: 2 copper layers, 96 x 56 mm, 131 parts, among them P1 Sensor, P10 GND, P11 I2C, P12 CAN, P2 CAN, P3 DATA, P4 USB_OTG, P5 PhaseA, P6 PhaseB, P7 PhaseC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

Commit message: Add some vias
Parts:
- moved W7 0.50 mm to (193.0, 69.8)
Routing:
- net GND: track 723.1 -> 731.7 mm, vias 86 -> 99
Changed lines of the file:
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@@
-(kicad_pcb (version 20160815) (host pcbnew no-vcs-found-7452~57~ubuntu16.04.1)
+(kicad_pcb (version 4) (host pcbnew 4.0.4-stable)
   (general
     (links 339)
     (no_connects 0)
-    (area 129.424999 54.674999 225.575001 110.825001)
+    (area 122.624999 53.725 225.600001 111.616667)
     (thickness 1.6)
     (drawings 4)
-    (tracks 2351)
+    (tracks 2368)
     (zones 0)
     (modules 131)
@@
       (hpglpenspeed 20)
       (hpglpendiameter 15)
+      (hpglpenoverlay 2)
       (psnegative false)
       (psa4output false)
@@
     (descr "Through hole pin header")
     (tags "pin header")
-    (fp_text reference P3 (at -1 12.44 90) (layer F.SilkS)
+    (fp_text reference P3 (at -1 12.44 450) (layer F.SilkS)
       (effects (font (size 1 1) (thickness 0.15)))
     )
@@
       (effects (font (size 0.64 0.64) (thickness 0.05)))
     )
-    (fp_text value BSC016N06NS (at 3.5 -1.45 180) (layer F.SilkS) hide
+    (fp_text value BSC016N06NS (at 3.5 -1.45 540) (layer F.SilkS) hide
       (effects (font (size 0.64 0.64) (thickness 0.05)))
     )
@@
     (descr "SELF WE-PD3S")
     (attr smd)
-    (fp_text reference L2 (at -5 0.5) (layer F.SilkS)
+    (fp_text reference L2 (at -5 0.5 360) (layer F.SilkS)
       (effects (font (size 1 1) (thickness 0.15)))
     )
-    (fp_text value 47uH (at 0.889 -0.381) (layer F.Fab)
+    (fp_text value 47uH (at 0.889 -0.381 360) (layer F.Fab)
       (effects (font (size 1 1) (thickness 0.15)))
     )
@@
     (tags "resistor 0805")
     (attr smd)
-    (fp_text reference R11 (at -3.15 0.5) (layer F.SilkS)
+    (fp_text reference R11 (at -3.15 0.5 360) (layer F.SilkS)
       (effects (font (size 1 1) (thickness 0.15)))
     )
@@
     (tags "resistor 0805")
     (attr smd)
-    (fp_text reference R12 (at -3.15 0) (layer F.SilkS)
+    (fp_text reference R12 (at -3.15 0 360) (layer F.SilkS)
       (effects (font (size 1 1) (thickness 0.15)))
     )
@@
     (descr "Through hole pin header")
     (tags "pin header")
-    (fp_text reference P2 (at -2.5 5.33) (layer F.SilkS)
+    (fp_text reference P2 (at -2.5 5.33 360) (layer F.SilkS)
       (effects (font (size 1 1) (thickness 0.15)))
     )
@@
     (descr "Through hole pin header")
     (tags "pin header")
-    (fp_text reference P11 (at 2.6 3.24) (layer F.SilkS)
+    (fp_text reference P11 (at 2.6 3.24 360) (layer F.SilkS)
       (effects (font (size 1 1) (thickness 0.15)))
     )
@@
   )
   (module Measurement_Points:Measurement_Point_Round-SMD-Pad_Small (layer F.Cu)
-    (at 192.5 69.75)
+    (at 193 69.75)
     (descr "Mesurement Point, Round, SMD Pad, DM 1.5mm,")
     (tags "Mesurement Point, Round, SMD Pad, DM 1.5mm,")
@@
   (segment (start 148.049865 79.233119) (end 148.049865 77.618119) (width 0.5) (layer F.Cu) (net 1) (status 10))
   (segment (start 148.049865 77.618119) (end 147.564865 77.133119) (width 0.5) (layer F.Cu) (net 1) (status 20))
+  (via (at 143.4 109.6) (size 1) (drill 0.5) (layers F.Cu B.Cu) (net 2))
+  (via (at 133.2 56.2) (size 1) (drill 0.5) (layers F.Cu B.Cu) (net 2))
+  (via (at 188.2 69.6) (size 1) (drill 0.5) (layers F.Cu B.Cu) (net 2))
+  (via (at 191.2 69.6) (size 1) (drill 0.5) (layers F.Cu B.Cu) (net 2))
+  (via (at 190 82.8) (size 1) (drill 0.5) (layers F.Cu B.Cu) (net 2))
+  (via (at 156.6 71.4) (size 1) (drill 0.5) (layers F.Cu B.Cu) (net 2))
+  (via (at 169.4 59.4) (size 1) (drill 0.5) (layers F.Cu B.Cu) (net 2))
+  (via (at 188 65) (size 1) (drill 0.5) (layers F.Cu B.Cu) (net 2))
+  (via (at 132.4 109) (size 1) (drill 0.5) (layers F.Cu B.Cu) (net 2))
+  (via (at 140.4 57.2) (size 1) (drill 0.5) (layers F.Cu B.Cu) (net 2))
+  (via (at 203.788994 55.780601) (size 1) (drill 0.5) (layers F.Cu B.Cu) (net 2))
+  (via (at 153 109.5) (size 1) (drill 0.5) (layers F.Cu B.Cu) (net 2))
+  (via (at 192.5 109.5) (size 1) (drill 0.5) (layers F.Cu B.Cu) (net 2))
+  (segment (start 179.086114 65.604345) (end 179.086114 66.311451) (width 0.25) (layer B.Cu) (net 2))
+  (segment (start 179.086114 63.591847) (end 179.086114 65.604345) (width 0.25) (layer B.Cu) (net 2))
+  (segment (start 180.77594 61.902021) (end 179.086114 63.591847) (width 0.25) (layer B.Cu) (net 2))
+  (via (at 179.086114 66.311451) (size 1) (drill 0.5) (layers F.Cu B.Cu) (net 2))
+  (segment (start 181.077961 61.6) (end 180.77594 61.902021) (width 0.25) (layer B.Cu) (net 2))
+  (segment (start 193.8 61.6) (end 181.077961 61.6) (width 0.25) (layer B.Cu) (net 2))
+  (segment (start 186.077961 56.6) (end 180.77594 61.902021) (width 0.25) (layer B.Cu) (net 2))
+  (segment (start 192 56.6) (end 186.077961 56.6) (width 0.25) (layer B.Cu) (net 2))
   (segment (start 150.637755 98.101012) (end 151.344861 98.101012) (width 0.6) (layer B.Cu) (net 2))
   (segment (start 158 95) (end 158 96.65) (width 0.25) (layer F.Cu) (net 2))
@@
   (segment (start 138.05 84.25) (end 140.6 86.8) (width 0.25) (layer B.Cu) (net 2))
   (via (at 140.6 86.8) (size 1) (drill 0.5) (layers F.Cu B.Cu) (net 2))
-  (segment (start 182.4 61.4) (end 187.2 61.4) (width 0.25) (layer B.Cu) (net 2))
-  (segment (start 187.2 61.4) (end 192 56.6) (width 0.25) (layer B.Cu) (net 2))
   (via (at 192 56.6) (size 1) (drill 0.5) (layers F.Cu B.Cu) (net 2))
-  (segment (start 182.4 61.4) (end 193.6 61.4) (width 0.25) (layer B.Cu) (net 2))
-  (segment (start 193.6 61.4) (end 193.8 61.6) (width 0.25) (layer B.Cu) (net 2))
-  (via (at 182.4 61.4) (size 1) (drill 0.5) (layers F.Cu B.Cu) (net 2))
   (segment (start 194.968001 62.031999) (end 194.231999 62.031999) (width 0.6) (layer B.Cu) (net 2))
   (segment (start 197 60) (end 194.968001 62.031999) (width 0.6) (layer B.Cu) (net 2))
@@
   (segment (start 197.25 83.85) (end 199.4 83.85) (width 0.25) (layer F.Cu) (net 29) (status 30))
   (segment (start 199.4 83.85) (end 199.5 83.75) (width 0.25) (layer F.Cu) (net 29) (status 30))
-  (segment (start 187.615 59.5) (end 187.615 57.92) (width 1) (layer F.Cu) (net 30))
-  (segment (start 187.615 57.92) (end 189.035 56.5) (width 1) (layer F.Cu) (net 30))
+  (segment (start 187.615 59.5) (end 187.615 58.227595) (width 1) (layer F.Cu) (net 30))
+  (segment (start 187.615 58.227595) (end 189.035 56.807595) (width 1) (layer F.Cu) (net 30))
+  (segment (start 189.035 56.807595) (end 189.035 56.5) (width 1) (layer F.Cu) (net 30))
   (segment (start 187.25 63) (end 187.25 59.865) (width 1) (layer F.Cu) (net 30) (status 30))
   (segment (start 187.25 59.865) (end 187.615 59.5) (width 1) (layer F.Cu) (net 30) (status 30))
