File: MotorController2/Regulator.sch (KiCad schematic (older format))
At the start: 20 parts

Commit message: Initial schematic complete.
Parts:
- added W?: 5V, symbol TEST_1P
- added W?: 3V3, symbol TEST_1P
- added W?: DSUP, symbol TEST_1P
- added W?: GND, symbol TEST_1P
Connections:
- wire segments 54 -> 58
Changed lines of the file:
@@
 $EndDescr
 $Comp
-L GND #PWR?
+L GND #PWR063
 U 1 1 585F6F4B
 P 2850 3350
-F 0 "#PWR?" H 2850 3100 50  0001 C CNN
+F 0 "#PWR063" H 2850 3100 50  0001 C CNN
 F 1 "GND" H 2850 3200 50  0000 C CNN
 F 2 "" H 2850 3350 50  0000 C CNN
@@
 	2850 2650 3000 2650
 $Comp
-L +36V #PWR?
+L +36V #PWR064
 U 1 1 585F700E
 P 950 1450
-F 0 "#PWR?" H 950 1300 50  0001 C CNN
+F 0 "#PWR064" H 950 1300 50  0001 C CNN
 F 1 "+36V" H 950 1590 50  0000 C CNN
 F 2 "" H 950 1450 50  0000 C CNN
@@
 	4100 2800 4100 2450
 $Comp
-L GND #PWR?
+L GND #PWR065
 U 1 1 585F787D
 P 4350 2950
-F 0 "#PWR?" H 4350 2700 50  0001 C CNN
+F 0 "#PWR065" H 4350 2700 50  0001 C CNN
 F 1 "GND" H 4350 2800 50  0000 C CNN
 F 2 "" H 4350 2950 50  0000 C CNN
@@
 	4350 2950 4350 2850
 $Comp
-L GND #PWR?
+L GND #PWR066
 U 1 1 585F7983
 P 5450 2950
-F 0 "#PWR?" H 5450 2700 50  0001 C CNN
+F 0 "#PWR066" H 5450 2700 50  0001 C CNN
 F 1 "GND" H 5450 2800 50  0000 C CNN
 F 2 "" H 5450 2950 50  0000 C CNN
@@
 Connection ~ 2700 1600
 $Comp
-L GND #PWR?
+L GND #PWR067
 U 1 1 585F7C36
 P 1550 2050
-F 0 "#PWR?" H 1550 1800 50  0001 C CNN
+F 0 "#PWR067" H 1550 1800 50  0001 C CNN
 F 1 "GND" H 1550 1900 50  0000 C CNN
 F 2 "" H 1550 2050 50  0000 C CNN
@@
 $EndComp
 $Comp
-L GND #PWR?
+L GND #PWR068
 U 1 1 585F7C68
 P 2400 2050
-F 0 "#PWR?" H 2400 1800 50  0001 C CNN
+F 0 "#PWR068" H 2400 1800 50  0001 C CNN
 F 1 "GND" H 2400 1900 50  0000 C CNN
 F 2 "" H 2400 2050 50  0000 C CNN
@@
 $EndComp
 $Comp
-L GND #PWR?
+L GND #PWR069
 U 1 1 585F7C9A
 P 2700 2050
-F 0 "#PWR?" H 2700 1800 50  0001 C CNN
+F 0 "#PWR069" H 2700 1800 50  0001 C CNN
 F 1 "GND" H 2700 1900 50  0000 C CNN
 F 2 "" H 2700 2050 50  0000 C CNN
@@
 $EndComp
 $Comp
-L +5V #PWR?
+L +5V #PWR070
 U 1 1 586591BB
 P 5300 2050
-F 0 "#PWR?" H 5300 1900 50  0001 C CNN
+F 0 "#PWR070" H 5300 1900 50  0001 C CNN
 F 1 "+5V" H 5300 2190 50  0000 C CNN
 F 2 "" H 5300 2050 50  0000 C CNN
@@
 Connection ~ 1600 1600
 $Comp
-L +8V #PWR?
+L +8V #PWR071
 U 1 1 5865931B
 P 1600 1000
-F 0 "#PWR?" H 1600 850 50  0001 C CNN
+F 0 "#PWR071" H 1600 850 50  0001 C CNN
 F 1 "+8V" H 1600 1140 50  0000 C CNN
 F 2 "" H 1600 1000 50  0000 C CNN
@@
 	1600 1000 1600 1150
 $Comp
-L GND #PWR?
+L GND #PWR072
 U 1 1 586595C6
 P 6600 3150
-F 0 "#PWR?" H 6600 2900 50  0001 C CNN
+F 0 "#PWR072" H 6600 2900 50  0001 C CNN
 F 1 "GND" H 6600 3000 50  0000 C CNN
 F 2 "" H 6600 3150 50  0000 C CNN
@@
 	6600 3150 6600 2950
 $Comp
-L +3V3 #PWR?
+L +3V3 #PWR073
 U 1 1 58659680
 P 7300 2300
-F 0 "#PWR?" H 7300 2150 50  0001 C CNN
+F 0 "#PWR073" H 7300 2150 50  0001 C CNN
 F 1 "+3V3" H 7300 2440 50  0000 C CNN
 F 2 "" H 7300 2300 50  0000 C CNN
@@
 $EndComp
 $Comp
-L GND #PWR?
+L GND #PWR074
 U 1 1 586598C9
 P 7250 3000
-F 0 "#PWR?" H 7250 2750 50  0001 C CNN
+F 0 "#PWR074" H 7250 2750 50  0001 C CNN
 F 1 "GND" H 7250 2850 50  0000 C CNN
 F 2 "" H 7250 3000 50  0000 C CNN
@@
 $EndComp
 $Comp
-L GND #PWR?
+L GND #PWR075
 U 1 1 5865A3E7
 P 7900 3100
-F 0 "#PWR?" H 7900 2850 50  0001 C CNN
+F 0 "#PWR075" H 7900 2850 50  0001 C CNN
 F 1 "GND" H 7900 2950 50  0000 C CNN
 F 2 "" H 7900 3100 50  0000 C CNN
@@
 $EndComp
 $Comp
-L GND #PWR?
+L GND #PWR076
 U 1 1 5865A42E
 P 8550 3150
-F 0 "#PWR?" H 8550 2900 50  0001 C CNN
+F 0 "#PWR076" H 8550 2900 50  0001 C CNN
 F 1 "GND" H 8550 3000 50  0000 C CNN
 F 2 "" H 8550 3150 50  0000 C CNN
@@
 	7900 3000 7900 3100
 Wire Wire Line
-	6200 2450 5100 2450
+	5100 2450 6200 2450
+$Comp
+L TEST_1P W?
+U 1 1 586E8A7C
+P 5750 2200
+F 0 "W?" H 5750 2470 50  0000 C CNN
+F 1 "5V" H 5750 2400 50  0000 C CNN
+F 2 "" H 5950 2200 50  0000 C CNN
+F 3 "" H 5950 2200 50  0000 C CNN
+	1    5750 2200
+	1    0    0    -1
+$EndComp
+Wire Wire Line
+	5750 2200 5750 2450
+Connection ~ 5750 2450
+$Comp
+L TEST_1P W?
+U 1 1 586E8BDF
+P 8250 1950
+F 0 "W?" H 8250 2220 50  0000 C CNN
+F 1 "3V3" H 8250 2150 50  0000 C CNN
+F 2 "" H 8450 1950 50  0000 C CNN
+F 3 "" H 8450 1950 50  0000 C CNN
+	1    8250 1950
+	1    0    0    -1
+$EndComp
+Wire Wire Line
+	8250 1950 8250 2150
+Connection ~ 8250 2150
+$Comp
+L TEST_1P W?
+U 1 1 586EC5DC
+P 3000 1400
+F 0 "W?" H 3000 1670 50  0000 C CNN
+F 1 "DSUP" H 3000 1600 50  0000 C CNN
+F 2 "" H 3200 1400 50  0000 C CNN
+F 3 "" H 3200 1400 50  0000 C CNN
+	1    3000 1400
+	1    0    0    -1
+$EndComp
+Wire Wire Line
+	3000 1400 3000 1600
+Connection ~ 3000 1600
+$Comp
+L TEST_1P W?
+U 1 1 586ECE27
+P 4350 1450
+F 0 "W?" H 4350 1720 50  0000 C CNN
+F 1 "GND" H 4350 1650 50  0000 C CNN
+F 2 "" H 4550 1450 50  0000 C CNN
+F 3 "" H 4550 1450 50  0000 C CNN
+	1    4350 1450
+	1    0    0    -1
+$EndComp
+$Comp
+L GND #PWR077
+U 1 1 586ECEC7
+P 4350 1550
+F 0 "#PWR077" H 4350 1300 50  0001 C CNN
+F 1 "GND" H 4350 1400 50  0000 C CNN
+F 2 "" H 4350 1550 50  0000 C CNN
+F 3 "" H 4350 1550 50  0000 C CNN
+	1    4350 1550
+	1    0    0    -1
+$EndComp
+Wire Wire Line
+	4350 1550 4350 1450
 $EndSCHEMATC

Commit message: Component footprints.
Parts:
- C36, C39: renamed from C?; footprint (none) -> Capacitors_SMD:C_1206_HandSoldering
- C37: renamed from C?; footprint (none) -> Capacitors_SMD:c_elec_10x10.5
- C38, C40, C42, C43: renamed from C?; footprint (none) -> Capacitors_SMD:C_0805_HandSoldering
- C41: renamed from C?; footprint (none) -> Capacitors_SMD:c_elec_6.3x5.8
- D4, D5: renamed from D?; footprint (none) -> Diodes_SMD:DO-214AB_Handsoldering
- D6: renamed from D?; value D_Schottky -> 50V; footprint (none) -> Diodes_SMD:SOD-123
- D7, D8: renamed from D?; footprint (none) -> Diodes_SMD:SOD-123
- D9: renamed from D?; footprint (none) -> LEDs:LED_0805
- L2, L3: renamed from L?; footprint (none) -> Inductors:SELF-WE-PD3S
- R33, R34: renamed from R?; footprint (none) -> Resistors_SMD:R_0805_HandSoldering
- U4: renamed from U?; footprint (none) -> Housings_SOIC:SOIC-8-1EP_3.9x4.9mm_Pitch1.27mm
- U5: renamed from U?; footprint (none) -> TO_SOT_Packages_SMD:SOT-223; Order (none) -> http://uk.farnell.com/microchip/tc2117-3-3vdbtr/ic-cmso-ldo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
- W10, W11, W12, W13: renamed from W?; footprint (none) -> Measurement_Points:Measurement_Point_Round-SMD-Pad_Big
Connections:
- wire segments 58 -> 64

Commit message: Add local library.
Parts:
- L2: Order (none) -> http://uk.farnell.com/tdk/clf7045t-470m/inductor-47uh-1-3a-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
- L3: Order (none) -> http://uk.farnell.com/tdk/clf7045t-470m/inductor-47uh-1-3a-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; Order2 (none) -> https://www.digikey.co.uk/product-detail/en/tdk-corporation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
- U4: Order (none) -> https://www.digikey.co.uk/product-detail/en/infineon-techno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
Changed lines of the file:
@@
 $EndDescr
 $Comp
-L GND #PWR072
+L GND #PWR074
 U 1 1 585F6F4B
 P 2850 3350
-F 0 "#PWR072" H 2850 3100 50  0001 C CNN
+F 0 "#PWR074" H 2850 3100 50  0001 C CNN
 F 1 "GND" H 2850 3200 50  0000 C CNN
 F 2 "" H 2850 3350 50  0000 C CNN
@@
 	2850 2650 3000 2650
 $Comp
-L +36V #PWR073
+L +36V #PWR075
 U 1 1 585F700E
 P 950 1450
-F 0 "#PWR073" H 950 1300 50  0001 C CNN
+F 0 "#PWR075" H 950 1300 50  0001 C CNN
 F 1 "+36V" H 950 1590 50  0000 C CNN
 F 2 "" H 950 1450 50  0000 C CNN
@@
 F 2 "Inductors:SELF-WE-PD3S" H 2000 1600 50  0001 C CNN
 F 3 "" H 2000 1600 50  0000 C CNN
+F 4 "http://uk.farnell.com/tdk/clf7045t-470m/inductor-47uh-1-3a-20-smd/dp/2345091" V 2000 1600 60  0001 C CNN "Order"
 	1    2000 1600
 	0    1    1    0
@@
 F 2 "Inductors:SELF-WE-PD3S" H 4800 2450 50  0001 C CNN
 F 3 "" H 4800 2450 50  0000 C CNN
+F 4 "http://uk.farnell.com/tdk/clf7045t-470m/inductor-47uh-1-3a-20-smd/dp/2345091" V 4800 2450 60  0001 C CNN "Order"
+F 5 "https://www.digikey.co.uk/product-detail/en/tdk-corporation/CLF7045T-470M/445-9527-1-ND/3909700" V 4800 2450 60  0001 C CNN "Order2"
 	1    4800 2450
 	0    1    1    0
@@
 	4100 2800 4100 2450
 $Comp
-L GND #PWR074
+L GND #PWR076
 U 1 1 585F787D
 P 4350 2950
-F 0 "#PWR074" H 4350 2700 50  0001 C CNN
+F 0 "#PWR076" H 4350 2700 50  0001 C CNN
 F 1 "GND" H 4350 2800 50  0000 C CNN
 F 2 "" H 4350 2950 50  0000 C CNN
@@
 	4350 2950 4350 2850
 $Comp
-L GND #PWR075
+L GND #PWR077
 U 1 1 585F7983
 P 5450 2950
-F 0 "#PWR075" H 5450 2700 50  0001 C CNN
+F 0 "#PWR077" H 5450 2700 50  0001 C CNN
 F 1 "GND" H 5450 2800 50  0000 C CNN
 F 2 "" H 5450 2950 50  0000 C CNN
@@
 Connection ~ 2700 1600
 $Comp
-L GND #PWR076
+L GND #PWR078
 U 1 1 585F7C36
 P 1550 2050
-F 0 "#PWR076" H 1550 1800 50  0001 C CNN
+F 0 "#PWR078" H 1550 1800 50  0001 C CNN
 F 1 "GND" H 1550 1900 50  0000 C CNN
 F 2 "" H 1550 2050 50  0000 C CNN
@@
 $EndComp
 $Comp
-L GND #PWR077
+L GND #PWR079
 U 1 1 585F7C68
 P 2400 2050
-F 0 "#PWR077" H 2400 1800 50  0001 C CNN
+F 0 "#PWR079" H 2400 1800 50  0001 C CNN
 F 1 "GND" H 2400 1900 50  0000 C CNN
 F 2 "" H 2400 2050 50  0000 C CNN
@@
 $EndComp
 $Comp
-L GND #PWR078
+L GND #PWR080
 U 1 1 585F7C9A
 P 2700 2050
-F 0 "#PWR078" H 2700 1800 50  0001 C CNN
+F 0 "#PWR080" H 2700 1800 50  0001 C CNN
 F 1 "GND" H 2700 1900 50  0000 C CNN
 F 2 "" H 2700 2050 50  0000 C CNN
@@
 F 2 "Housings_SOIC:SOIC-8-1EP_3.9x4.9mm_Pitch1.27mm" H 3450 3100 60  0001 C CNN
 F 3 "http://www.infineon.com/dgdl/Infineon-IFX91041-DS-v01_01-en.pdf?fileId=db3a304320d39d59012153afb91a0548" H 3450 3100 60  0001 C CNN
+F 4 "https://www.digikey.co.uk/product-detail/en/infineon-technologies/IFX91041EJ-V50/IFX91041EJ-V50INCT-ND/3300395" H 3450 3100 60  0001 C CNN "Order"
 	1    3450 3100
 	1    0    0    -1
 $EndComp
 $Comp
-L +5V #PWR079
+L +5V #PWR081
 U 1 1 586591BB
 P 5300 2050
-F 0 "#PWR079" H 5300 1900 50  0001 C CNN
+F 0 "#PWR081" H 5300 1900 50  0001 C CNN
 F 1 "+5V" H 5300 2190 50  0000 C CNN
 F 2 "" H 5300 2050 50  0000 C CNN
@@
 Connection ~ 1600 1600
 $Comp
-L +8V #PWR080
+L +8V #PWR082
 U 1 1 5865931B
 P 1600 1000
-F 0 "#PWR080" H 1600 850 50  0001 C CNN
+F 0 "#PWR082" H 1600 850 50  0001 C CNN
 F 1 "+8V" H 1600 1140 50  0000 C CNN
 F 2 "" H 1600 1000 50  0000 C CNN
@@
 	1600 1000 1600 1150
 $Comp
-L GND #PWR081
+L GND #PWR083
 U 1 1 586595C6
 P 6600 3150
-F 0 "#PWR081" H 6600 2900 50  0001 C CNN
+F 0 "#PWR083" H 6600 2900 50  0001 C CNN
 F 1 "GND" H 6600 3000 50  0000 C CNN
 F 2 "" H 6600 3150 50  0000 C CNN
@@
 	6600 3150 6600 2950
 $Comp
-L +3V3 #PWR082
+L +3V3 #PWR084
 U 1 1 58659680
 P 7300 2300
-F 0 "#PWR082" H 7300 2150 50  0001 C CNN
+F 0 "#PWR084" H 7300 2150 50  0001 C CNN
 F 1 "+3V3" H 7300 2440 50  0000 C CNN
 F 2 "" H 7300 2300 50  0000 C CNN
@@
 $EndComp
 $Comp
-L GND #PWR083
+L GND #PWR085
 U 1 1 586598C9
 P 7250 3000
-F 0 "#PWR083" H 7250 2750 50  0001 C CNN
+F 0 "#PWR085" H 7250 2750 50  0001 C CNN
 F 1 "GND" H 7250 2850 50  0000 C CNN
 F 2 "" H 7250 3000 50  0000 C CNN
@@
 $EndComp
 $Comp
-L GND #PWR084
+L GND #PWR086
 U 1 1 5865A3E7
 P 7900 3100
-F 0 "#PWR084" H 7900 2850 50  0001 C CNN
+F 0 "#PWR086" H 7900 2850 50  0001 C CNN
 F 1 "GND" H 7900 2950 50  0000 C CNN
 F 2 "" H 7900 3100 50  0000 C CNN
@@
 $EndComp
 $Comp
-L GND #PWR085
+L GND #PWR087
 U 1 1 5865A42E
 P 8550 3150
-F 0 "#PWR085" H 8550 2900 50  0001 C CNN
+F 0 "#PWR087" H 8550 2900 50  0001 C CNN
 F 1 "GND" H 8550 3000 50  0000 C CNN
 F 2 "" H 8550 3150 50  0000 C CNN
@@
 $EndComp
 $Comp
-L GND #PWR086
+L GND #PWR088
 U 1 1 586ECEC7
 P 4350 1550
-F 0 "#PWR086" H 4350 1300 50  0001 C CNN
+F 0 "#PWR088" H 4350 1300 50  0001 C CNN
 F 1 "GND" H 4350 1400 50  0000 C CNN
 F 2 "" H 4350 1550 50  0000 C CNN
@@
 	4350 1550 4350 1450
 $Comp
-L PWR_FLAG #FLG087
+L PWR_FLAG #FLG089
 U 1 1 5874647E
 P 6000 2250
-F 0 "#FLG087" H 6000 2345 50  0001 C CNN
+F 0 "#FLG089" H 6000 2345 50  0001 C CNN
 F 1 "PWR_FLAG" H 6000 2430 50  0000 C CNN
 F 2 "" H 6000 2250 50  0000 C CNN
@@
 Connection ~ 6000 2450
 $Comp
-L PWR_FLAG #FLG088
+L PWR_FLAG #FLG090
 U 1 1 58746589
 P 7950 2050
-F 0 "#FLG088" H 7950 2145 50  0001 C CNN
+F 0 "#FLG090" H 7950 2145 50  0001 C CNN
 F 1 "PWR_FLAG" H 7950 2230 50  0000 C CNN
 F 2 "" H 7950 2050 50  0000 C CNN
@@
 Connection ~ 7950 2150
 $Comp
-L PWR_FLAG #FLG089
+L PWR_FLAG #FLG091
 U 1 1 58746947
 P 1900 1050
-F 0 "#FLG089" H 1900 1145 50  0001 C CNN
+F 0 "#FLG091" H 1900 1145 50  0001 C CNN
 F 1 "PWR_FLAG" H 1900 1230 50  0000 C CNN
 F 2 "" H 1900 1050 50  0000 C CNN
@@
 	1900 1150 1600 1150
 $Comp
-L PWR_FLAG #FLG090
+L PWR_FLAG #FLG092
 U 1 1 58746A06
 P 900 2000
-F 0 "#FLG090" H 900 2095 50  0001 C CNN
+F 0 "#FLG092" H 900 2095 50  0001 C CNN
 F 1 "PWR_FLAG" H 900 2180 50  0000 C CNN
 F 2 "" H 900 2000 50  0000 C CNN
@@
 Connection ~ 1100 1600
 $Comp
-L PWR_FLAG #FLG091
+L PWR_FLAG #FLG093
 U 1 1 58764812
 P 3350 1450
-F 0 "#FLG091" H 3350 1545 50  0001 C CNN
+F 0 "#FLG093" H 3350 1545 50  0001 C CNN
 F 1 "PWR_FLAG" H 3350 1630 50  0000 C CNN
 F 2 "" H 3350 1450 50  0000 C CNN

Commit message: Laying out power section.
Parts:
- D4: value D -> 60V 2A; footprint Diodes_SMD:DO-214AB_Handsoldering -> Diodes_SMD:SOD-123; Order (none) -> http://uk.farnell.com/panasonic-electronic-components/db2w6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
- D5: value D -> 60V 2A; footprint Diodes_SMD:DO-214AB_Handsoldering -> Diodes_SMD:SOD-123; Order (none) -> http://uk.farnell.com/panasonic-electronic-components/db2w6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; Type (none) -> DB2W60400L
- D9: symbol LED -> LED-RESCUE-BMC2
- W10, W12, W13: footprint Measurement_Points:Measurement_Point_Round-SMD-Pad_Big -> Measurement_Points:Measurement_Point_Round-SMD-Pad_Small
Changed lines of the file:
@@
 EESchema Schematic File Version 2
+LIBS:BMC2-rescue
 LIBS:power
 LIBS:device
@@
 LIBS:IFX91041EJV33
 LIBS:BMC2-cache
-EELAYER 25 0
+EELAYER 26 0
 EELAYER END
 $Descr A4 11693 8268
@@
 P 1300 1600
 F 0 "D4" H 1300 1700 50  0000 C CNN
-F 1 "D" H 1300 1500 50  0000 C CNN
-F 2 "Diodes_SMD:DO-214AB_Handsoldering" H 1300 1600 50  0001 C CNN
+F 1 "60V 2A" H 1300 1500 50  0000 C CNN
+F 2 "Diodes_SMD:SOD-123" H 1300 1600 50  0001 C CNN
 F 3 "" H 1300 1600 50  0000 C CNN
+F 4 "http://uk.farnell.com/panasonic-electronic-components/db2w60400l/diode-schottky-60v-mini2-f3-b/dp/2284958" H 1300 1600 60  0001 C CNN "Order"
 	1    1300 1600
 	-1   0    0    1
@@
 Connection ~ 5550 2450
 $Comp
-L LED D9
+L LED-RESCUE-BMC2 D9
 U 1 1 585F871A
 P 8550 2850
+AR Path="/585F871A" Ref="D9"  Part="1"
+AR Path="/585F64FD/585F871A" Ref="D9"  Part="1"
 F 0 "D9" H 8550 2950 50  0000 C CNN
 F 1 "LED" H 8550 2750 50  0000 C CNN
@@
 P 1600 1300
 F 0 "D5" H 1600 1400 50  0000 C CNN
-F 1 "D" H 1600 1200 50  0000 C CNN
-F 2 "Diodes_SMD:DO-214AB_Handsoldering" H 1600 1300 50  0001 C CNN
-F 3 "" H 1600 1300 50  0000 C CNN
+F 1 "60V 2A " H 1600 1200 50  0000 C CNN
+F 2 "Diodes_SMD:SOD-123" H 1600 1300 50  0001 C CNN
+F 3 "http://www.farnell.com/datasheets/1912070.pdf?_ga=1.4639027.1808009743.1471515981" H 1600 1300 50  0001 C CNN
+F 4 "http://uk.farnell.com/panasonic-electronic-components/db2w60400l/diode-schottky-60v-mini2-f3-b/dp/2284958" H 1600 1300 60  0001 C CNN "Order"
+F 5 "DB2W60400L" H 1600 1300 60  0001 C CNN "Type"
 	1    1600 1300
 	0    -1   -1   0
@@
 F 0 "W12" H 5750 2470 50  0000 C CNN
 F 1 "5V" H 5750 2400 50  0000 C CNN
-F 2 "Measurement_Points:Measurement_Point_Round-SMD-Pad_Big" H 5950 2200 50  0001 C CNN
+F 2 "Measurement_Points:Measurement_Point_Round-SMD-Pad_Small" H 5950 2200 50  0001 C CNN
 F 3 "" H 5950 2200 50  0000 C CNN
 	1    5750 2200
@@
 F 0 "W13" H 8250 2220 50  0000 C CNN
 F 1 "3V3" H 8250 2150 50  0000 C CNN
-F 2 "Measurement_Points:Measurement_Point_Round-SMD-Pad_Big" H 8450 1950 50  0001 C CNN
+F 2 "Measurement_Points:Measurement_Point_Round-SMD-Pad_Small" H 8450 1950 50  0001 C CNN
 F 3 "" H 8450 1950 50  0000 C CNN
 	1    8250 1950
@@
 F 0 "W10" H 3000 1670 50  0000 C CNN
 F 1 "DSUP" H 3000 1600 50  0000 C CNN
-F 2 "Measurement_Points:Measurement_Point_Round-SMD-Pad_Big" H 3200 1400 50  0001 C CNN
+F 2 "Measurement_Points:Measurement_Point_Round-SMD-Pad_Small" H 3200 1400 50  0001 C CNN
 F 3 "" H 3200 1400 50  0000 C CNN
 	1    3000 1400

Commit message: Layout nearly complete.
Connections:
- net +3V3: now also U5.4 (Vout)
- net GND: now also U4.9 (GND)
Changed lines of the file:
@@
 LIBS:IFX91041EJV33
 LIBS:BMC2-cache
-EELAYER 26 0
+EELAYER 25 0
 EELAYER END
 $Descr A4 11693 8268
@@
 $EndDescr
 $Comp
-L GND #PWR074
+L GND #PWR076
 U 1 1 585F6F4B
 P 2850 3350
-F 0 "#PWR074" H 2850 3100 50  0001 C CNN
+F 0 "#PWR076" H 2850 3100 50  0001 C CNN
 F 1 "GND" H 2850 3200 50  0000 C CNN
 F 2 "" H 2850 3350 50  0000 C CNN
@@
 $EndComp
 Wire Wire Line
-	2850 3250 2500 3250
+	2500 3250 3500 3250
 Wire Wire Line
 	2500 3250 2500 3200
@@
 	2850 2650 3000 2650
 $Comp
-L +36V #PWR075
+L +36V #PWR077
 U 1 1 585F700E
 P 950 1450
-F 0 "#PWR075" H 950 1300 50  0001 C CNN
+F 0 "#PWR077" H 950 1300 50  0001 C CNN
 F 1 "+36V" H 950 1590 50  0000 C CNN
 F 2 "" H 950 1450 50  0000 C CNN
@@
 	4100 2800 4100 2450
 $Comp
-L GND #PWR076
+L GND #PWR078
 U 1 1 585F787D
 P 4350 2950
-F 0 "#PWR076" H 4350 2700 50  0001 C CNN
+F 0 "#PWR078" H 4350 2700 50  0001 C CNN
 F 1 "GND" H 4350 2800 50  0000 C CNN
 F 2 "" H 4350 2950 50  0000 C CNN
@@
 	4350 2950 4350 2850
 $Comp
-L GND #PWR077
+L GND #PWR079
 U 1 1 585F7983
 P 5450 2950
-F 0 "#PWR077" H 5450 2700 50  0001 C CNN
+F 0 "#PWR079" H 5450 2700 50  0001 C CNN
 F 1 "GND" H 5450 2800 50  0000 C CNN
 F 2 "" H 5450 2950 50  0000 C CNN
@@
 Connection ~ 2700 1600
 $Comp
-L GND #PWR078
+L GND #PWR080
 U 1 1 585F7C36
 P 1550 2050
-F 0 "#PWR078" H 1550 1800 50  0001 C CNN
+F 0 "#PWR080" H 1550 1800 50  0001 C CNN
 F 1 "GND" H 1550 1900 50  0000 C CNN
 F 2 "" H 1550 2050 50  0000 C CNN
@@
 $EndComp
 $Comp
-L GND #PWR079
+L GND #PWR081
 U 1 1 585F7C68
 P 2400 2050
-F 0 "#PWR079" H 2400 1800 50  0001 C CNN
+F 0 "#PWR081" H 2400 1800 50  0001 C CNN
 F 1 "GND" H 2400 1900 50  0000 C CNN
 F 2 "" H 2400 2050 50  0000 C CNN
@@
 $EndComp
 $Comp
-L GND #PWR080
+L GND #PWR082
 U 1 1 585F7C9A
 P 2700 2050
-F 0 "#PWR080" H 2700 1800 50  0001 C CNN
+F 0 "#PWR082" H 2700 1800 50  0001 C CNN
 F 1 "GND" H 2700 1900 50  0000 C CNN
 F 2 "" H 2700 2050 50  0000 C CNN
@@
 $EndComp
 $Comp
-L +5V #PWR081
+L +5V #PWR083
 U 1 1 586591BB
 P 5300 2050
-F 0 "#PWR081" H 5300 1900 50  0001 C CNN
+F 0 "#PWR083" H 5300 1900 50  0001 C CNN
 F 1 "+5V" H 5300 2190 50  0000 C CNN
 F 2 "" H 5300 2050 50  0000 C CNN
@@
 Connection ~ 1600 1600
 $Comp
-L +8V #PWR082
+L +8V #PWR084
 U 1 1 5865931B
 P 1600 1000
-F 0 "#PWR082" H 1600 850 50  0001 C CNN
+F 0 "#PWR084" H 1600 850 50  0001 C CNN
 F 1 "+8V" H 1600 1140 50  0000 C CNN
 F 2 "" H 1600 1000 50  0000 C CNN
@@
 	1600 1000 1600 1150
 $Comp
-L GND #PWR083
+L GND #PWR085
 U 1 1 586595C6
 P 6600 3150
-F 0 "#PWR083" H 6600 2900 50  0001 C CNN
+F 0 "#PWR085" H 6600 2900 50  0001 C CNN
 F 1 "GND" H 6600 3000 50  0000 C CNN
 F 2 "" H 6600 3150 50  0000 C CNN
@@
 	6600 3150 6600 2950
 $Comp
-L +3V3 #PWR084
+L +3V3 #PWR086
 U 1 1 58659680
 P 7300 2300
-F 0 "#PWR084" H 7300 2150 50  0001 C CNN
+F 0 "#PWR086" H 7300 2150 50  0001 C CNN
 F 1 "+3V3" H 7300 2440 50  0000 C CNN
 F 2 "" H 7300 2300 50  0000 C CNN
@@
 $EndComp
 $Comp
-L GND #PWR085
+L GND #PWR087
 U 1 1 586598C9
 P 7250 3000
-F 0 "#PWR085" H 7250 2750 50  0001 C CNN
+F 0 "#PWR087" H 7250 2750 50  0001 C CNN
 F 1 "GND" H 7250 2850 50  0000 C CNN
 F 2 "" H 7250 3000 50  0000 C CNN
@@
 $EndComp
 $Comp
-L GND #PWR086
+L GND #PWR088
 U 1 1 5865A3E7
 P 7900 3100
-F 0 "#PWR086" H 7900 2850 50  0001 C CNN
+F 0 "#PWR088" H 7900 2850 50  0001 C CNN
 F 1 "GND" H 7900 2950 50  0000 C CNN
 F 2 "" H 7900 3100 50  0000 C CNN
@@
 $EndComp
 $Comp
-L GND #PWR087
+L GND #PWR089
 U 1 1 5865A42E
 P 8550 3150
-F 0 "#PWR087" H 8550 2900 50  0001 C CNN
+F 0 "#PWR089" H 8550 2900 50  0001 C CNN
 F 1 "GND" H 8550 3000 50  0000 C CNN
 F 2 "" H 8550 3150 50  0000 C CNN
@@
 $EndComp
 $Comp
-L GND #PWR088
+L GND #PWR090
 U 1 1 586ECEC7
 P 4350 1550
-F 0 "#PWR088" H 4350 1300 50  0001 C CNN
+F 0 "#PWR090" H 4350 1300 50  0001 C CNN
 F 1 "GND" H 4350 1400 50  0000 C CNN
 F 2 "" H 4350 1550 50  0000 C CNN
@@
 	4350 1550 4350 1450
 $Comp
-L PWR_FLAG #FLG089
+L PWR_FLAG #FLG091
 U 1 1 5874647E
 P 6000 2250
-F 0 "#FLG089" H 6000 2345 50  0001 C CNN
+F 0 "#FLG091" H 6000 2345 50  0001 C CNN
 F 1 "PWR_FLAG" H 6000 2430 50  0000 C CNN
 F 2 "" H 6000 2250 50  0000 C CNN
@@
 Connection ~ 6000 2450
 $Comp
-L PWR_FLAG #FLG090
+L PWR_FLAG #FLG092
 U 1 1 58746589
 P 7950 2050
-F 0 "#FLG090" H 7950 2145 50  0001 C CNN
+F 0 "#FLG092" H 7950 2145 50  0001 C CNN
 F 1 "PWR_FLAG" H 7950 2230 50  0000 C CNN
 F 2 "" H 7950 2050 50  0000 C CNN
@@
 Connection ~ 7950 2150
 $Comp
-L PWR_FLAG #FLG091
+L PWR_FLAG #FLG093
 U 1 1 58746947
 P 1900 1050
-F 0 "#FLG091" H 1900 1145 50  0001 C CNN
+F 0 "#FLG093" H 1900 1145 50  0001 C CNN
 F 1 "PWR_FLAG" H 1900 1230 50  0000 C CNN
 F 2 "" H 1900 1050 50  0000 C CNN
@@
 	1900 1150 1600 1150
 $Comp
-L PWR_FLAG #FLG092
+L PWR_FLAG #FLG094
 U 1 1 58746A06
 P 900 2000
-F 0 "#FLG092" H 900 2095 50  0001 C CNN
+F 0 "#FLG094" H 900 2095 50  0001 C CNN
 F 1 "PWR_FLAG" H 900 2180 50  0000 C CNN
 F 2 "" H 900 2000 50  0000 C CNN
@@
 Connection ~ 1100 1600
 $Comp
-L PWR_FLAG #FLG093
+L PWR_FLAG #FLG095
 U 1 1 58764812
 P 3350 1450
-F 0 "#FLG093" H 3350 1545 50  0001 C CNN
+F 0 "#FLG095" H 3350 1545 50  0001 C CNN
 F 1 "PWR_FLAG" H 3350 1630 50  0000 C CNN
 F 2 "" H 3350 1450 50  0000 C CNN
@@
 	1    0    0    -1
 $EndComp
+Wire Wire Line
+	7050 2550 7250 2550
+Connection ~ 7250 2550
 $EndSCHEMATC
