File: MotorController2/Regulator.sch (KiCad schematic (older format))
At the start: 24 parts, among them U4 IFX91041EJV50, U5 TC2117-3.3V

Commit message: Work on BOM.
Parts:
- C36: value 220nF 60V -> 220nF 100V; Farnell (none) -> 1856615
- C37: value 100uF 60V -> 100uF 63V; Farnell (none) -> 9696040
- C38: value 22nF 6V -> 22nF 50V; Farnell (none) -> 2581093; Notes (none) -> 6V
- C39: value 220nF 60V -> 220nF 100V; Farnell (none) -> 1856615; Note (none) -> 60V
- C40, C42: value 220nF 6V -> 220nF 100V; Farnell (none) -> 1856615; Notes (none) -> 6V
- C41: value 100uF 6V -> 100uF 6.3V; Farnell (none) -> 2611349
- C43: value 1uF 4V min -> 1uF 50V; Notes (none) -> 4V
- D5: value 60V 2A -> 60V 2A; Farnell (none) -> 2284958
- D6: value 50V -> 60V 2A; Farnell (none) -> 2284958
- D7: value 5.4V -> 5.6V; Farnell (none) -> 1431292; Order (none) -> http://uk.farnell.com/on-semiconductor/mmsz5v6t1g/diode-zen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; Part (none) -> MMSZ5V6T1G
- D8: Farnell (none) -> 1651592; Order (none) -> http://uk.farnell.com/on-semiconductor/mmsz4685t1g/diode-ze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; Part (none) -> MMSZ4685T1G
- D9: value LED -> RED; Farnell (none) -> 1581239
Changed lines of the file:
@@
 LIBS:IFX91041EJV33
 LIBS:BMC2-cache
-EELAYER 25 0
+EELAYER 26 0
 EELAYER END
 $Descr A4 11693 8268
@@
 $EndDescr
 $Comp
-L GND #PWR076
+L GND #PWR077
 U 1 1 585F6F4B
 P 2850 3350
-F 0 "#PWR076" H 2850 3100 50  0001 C CNN
+F 0 "#PWR077" H 2850 3100 50  0001 C CNN
 F 1 "GND" H 2850 3200 50  0000 C CNN
 F 2 "" H 2850 3350 50  0000 C CNN
@@
 P 2500 2700
 F 0 "C38" H 2525 2800 50  0000 L CNN
-F 1 "22nF 6V" H 2525 2600 50  0000 L CNN
+F 1 "22nF 50V" H 2525 2600 50  0000 L CNN
 F 2 "Capacitors_SMD:C_0805_HandSoldering" H 2538 2550 50  0001 C CNN
 F 3 "" H 2500 2700 50  0000 C CNN
+F 4 "2581093" H 2500 2700 60  0001 C CNN "Farnell"
+F 5 "6V" H 2500 2700 60  0001 C CNN "Notes"
 	1    2500 2700
 	1    0    0    -1
@@
 	2850 2650 3000 2650
 $Comp
-L +36V #PWR077
+L +36V #PWR078
 U 1 1 585F700E
 P 950 1450
-F 0 "#PWR077" H 950 1300 50  0001 C CNN
+F 0 "#PWR078" H 950 1300 50  0001 C CNN
 F 1 "+36V" H 950 1590 50  0000 C CNN
 F 2 "" H 950 1450 50  0000 C CNN
@@
 P 1550 1800
 F 0 "C36" H 1575 1900 50  0000 L CNN
-F 1 "220nF 60V" H 1575 1700 50  0000 L CNN
+F 1 "220nF 100V" H 1300 1700 50  0000 L CNN
 F 2 "Capacitors_SMD:C_1206_HandSoldering" H 1588 1650 50  0001 C CNN
 F 3 "" H 1550 1800 50  0000 C CNN
+F 4 "1856615" H 1550 1800 60  0001 C CNN "Farnell"
 	1    1550 1800
 	1    0    0    -1
@@
 P 2700 1850
 F 0 "C39" H 2725 1950 50  0000 L CNN
-F 1 "220nF 60V" H 2725 1750 50  0000 L CNN
+F 1 "220nF 100V" H 2725 1750 50  0000 L CNN
 F 2 "Capacitors_SMD:C_1206_HandSoldering" H 2738 1700 50  0001 C CNN
 F 3 "" H 2700 1850 50  0000 C CNN
+F 4 "60V" H 2700 1850 60  0001 C CNN "Note"
+F 5 "1856615" H 2700 1850 60  0001 C CNN "Farnell"
 	1    2700 1850
 	1    0    0    -1
@@
 P 2400 1850
 F 0 "C37" H 2425 1950 50  0000 L CNN
-F 1 "100uF 60V" H 1900 1750 50  0000 L CNN
+F 1 "100uF 63V" H 2150 1750 50  0000 L CNN
 F 2 "Capacitors_SMD:c_elec_10x10.5" H 2438 1700 50  0001 C CNN
 F 3 "" H 2400 1850 50  0000 C CNN
+F 4 "9696040" H 2400 1850 60  0001 C CNN "Farnell"
 	1    2400 1850
 	1    0    0    -1
@@
 P 4350 2250
 F 0 "C40" H 4375 2350 50  0000 L CNN
-F 1 "220nF 6V" H 4375 2150 50  0000 L CNN
+F 1 "220nF 100V" H 4375 2150 50  0000 L CNN
 F 2 "Capacitors_SMD:C_0805_HandSoldering" H 4388 2100 50  0001 C CNN
 F 3 "" H 4350 2250 50  0000 C CNN
+F 4 "6V" H 4350 2250 60  0001 C CNN "Notes"
+F 5 "1856615" H 4350 2250 60  0001 C CNN "Farnell"
 	1    4350 2250
 	1    0    0    -1
@@
 P 4350 2700
 F 0 "D6" H 4350 2800 50  0000 C CNN
-F 1 "50V" H 4350 2600 50  0000 C CNN
+F 1 "60V 2A" H 4350 2600 50  0000 C CNN
 F 2 "Diodes_SMD:SOD-123" H 4350 2700 50  0001 C CNN
 F 3 "" H 4350 2700 50  0000 C CNN
+F 4 "2284958" H 4350 2700 60  0001 C CNN "Farnell"
 	1    4350 2700
 	0    1    1    0
@@
 P 5300 2700
 F 0 "C41" H 5325 2800 50  0000 L CNN
-F 1 "100uF 6V" H 4900 2600 50  0000 L CNN
+F 1 "100uF 6.3V" H 4900 2600 50  0000 L CNN
 F 2 "Capacitors_SMD:c_elec_6.3x5.8" H 5338 2550 50  0001 C CNN
 F 3 "" H 5300 2700 50  0000 C CNN
+F 4 "2611349" H 5300 2700 60  0001 C CNN "Farnell"
 	1    5300 2700
 	1    0    0    -1
@@
 P 5550 2700
 F 0 "C42" H 5575 2800 50  0000 L CNN
-F 1 "220nF 6V" H 5400 2600 50  0000 L CNN
+F 1 "220nF 100V" H 5400 2600 50  0000 L CNN
 F 2 "Capacitors_SMD:C_0805_HandSoldering" H 5588 2550 50  0001 C CNN
 F 3 "" H 5550 2700 50  0000 C CNN
+F 4 "6V" H 5550 2700 60  0001 C CNN "Notes"
+F 5 "1856615" H 5550 2700 60  0001 C CNN "Farnell"
 	1    5550 2700
 	1    0    0    -1
@@
 	4100 2800 4100 2450
 $Comp
-L GND #PWR078
+L GND #PWR079
 U 1 1 585F787D
 P 4350 2950
-F 0 "#PWR078" H 4350 2700 50  0001 C CNN
+F 0 "#PWR079" H 4350 2700 50  0001 C CNN
 F 1 "GND" H 4350 2800 50  0000 C CNN
 F 2 "" H 4350 2950 50  0000 C CNN
@@
 	4350 2950 4350 2850
 $Comp
-L GND #PWR079
+L GND #PWR080
 U 1 1 585F7983
 P 5450 2950
-F 0 "#PWR079" H 5450 2700 50  0001 C CNN
+F 0 "#PWR080" H 5450 2700 50  0001 C CNN
 F 1 "GND" H 5450 2800 50  0000 C CNN
 F 2 "" H 5450 2950 50  0000 C CNN
@@
 Connection ~ 2700 1600
 $Comp
-L GND #PWR080
+L GND #PWR081
 U 1 1 585F7C36
 P 1550 2050
-F 0 "#PWR080" H 1550 1800 50  0001 C CNN
+F 0 "#PWR081" H 1550 1800 50  0001 C CNN
 F 1 "GND" H 1550 1900 50  0000 C CNN
 F 2 "" H 1550 2050 50  0000 C CNN
@@
 $EndComp
 $Comp
-L GND #PWR081
+L GND #PWR082
 U 1 1 585F7C68
 P 2400 2050
-F 0 "#PWR081" H 2400 1800 50  0001 C CNN
+F 0 "#PWR082" H 2400 1800 50  0001 C CNN
 F 1 "GND" H 2400 1900 50  0000 C CNN
 F 2 "" H 2400 2050 50  0000 C CNN
@@
 $EndComp
 $Comp
-L GND #PWR082
+L GND #PWR083
 U 1 1 585F7C9A
 P 2700 2050
-F 0 "#PWR082" H 2700 1800 50  0001 C CNN
+F 0 "#PWR083" H 2700 1800 50  0001 C CNN
 F 1 "GND" H 2700 1900 50  0000 C CNN
 F 2 "" H 2700 2050 50  0000 C CNN
@@
 P 5900 2700
 F 0 "D7" H 5900 2800 50  0000 C CNN
-F 1 "5.4V" H 5900 2600 50  0000 C CNN
+F 1 "5.6V" H 5900 2600 50  0000 C CNN
 F 2 "Diodes_SMD:SOD-123" H 5900 2700 50  0001 C CNN
 F 3 "" H 5900 2700 50  0000 C CNN
+F 4 "MMSZ5V6T1G" H 5900 2700 60  0001 C CNN "Part"
+F 5 "http://uk.farnell.com/on-semiconductor/mmsz5v6t1g/diode-zener-5-6v-0-5w/dp/1431292" H 5900 2700 60  0001 C CNN "Order"
+F 6 "1431292" H 5900 2700 60  0001 C CNN "Farnell"
 	1    5900 2700
 	0    1    1    0
@@
 AR Path="/585F64FD/585F871A" Ref="D9"  Part="1"
 F 0 "D9" H 8550 2950 50  0000 C CNN
-F 1 "LED" H 8550 2750 50  0000 C CNN
+F 1 "RED" H 8550 2750 50  0000 C CNN
 F 2 "LEDs:LED_0805" H 8550 2850 50  0001 C CNN
 F 3 "" H 8550 2850 50  0000 C CNN
+F 4 "1581239" H 8550 2850 60  0001 C CNN "Farnell"
 	1    8550 2850
 	0    -1   -1   0
@@
 $EndComp
 $Comp
-L +5V #PWR083
+L +5V #PWR084
 U 1 1 586591BB
 P 5300 2050
-F 0 "#PWR083" H 5300 1900 50  0001 C CNN
+F 0 "#PWR084" H 5300 1900 50  0001 C CNN
 F 1 "+5V" H 5300 2190 50  0000 C CNN
 F 2 "" H 5300 2050 50  0000 C CNN
@@
 P 1600 1300
 F 0 "D5" H 1600 1400 50  0000 C CNN
-F 1 "60V 2A " H 1600 1200 50  0000 C CNN
+F 1 "60V 2A" H 1600 1200 50  0000 C CNN
 F 2 "Diodes_SMD:SOD-123" H 1600 1300 50  0001 C CNN
 F 3 "http://www.farnell.com/datasheets/1912070.pdf?_ga=1.4639027.1808009743.1471515981" H 1600 1300 50  0001 C CNN
 F 4 "http://uk.farnell.com/panasonic-electronic-components/db2w60400l/diode-schottky-60v-mini2-f3-b/dp/2284958" H 1600 1300 60  0001 C CNN "Order"
 F 5 "DB2W60400L" H 1600 1300 60  0001 C CNN "Type"
+F 6 "2284958" H 1600 1300 60  0001 C CNN "Farnell"
 	1    1600 1300
 	0    -1   -1   0
@@
 Connection ~ 1600 1600
 $Comp
-L +8V #PWR084
+L +8V #PWR085
 U 1 1 5865931B
 P 1600 1000
-F 0 "#PWR084" H 1600 850 50  0001 C CNN
+F 0 "#PWR085" H 1600 850 50  0001 C CNN
 F 1 "+8V" H 1600 1140 50  0000 C CNN
 F 2 "" H 1600 1000 50  0000 C CNN
@@
 	1600 1000 1600 1150
 $Comp
-L GND #PWR085
+L GND #PWR086
 U 1 1 586595C6
 P 6600 3150
-F 0 "#PWR085" H 6600 2900 50  0001 C CNN
+F 0 "#PWR086" H 6600 2900 50  0001 C CNN
 F 1 "GND" H 6600 3000 50  0000 C CNN
 F 2 "" H 6600 3150 50  0000 C CNN
@@
 	6600 3150 6600 2950
 $Comp
-L +3V3 #PWR086
+L +3V3 #PWR087
 U 1 1 58659680
 P 7300 2300
-F 0 "#PWR086" H 7300 2150 50  0001 C CNN
+F 0 "#PWR087" H 7300 2150 50  0001 C CNN
 F 1 "+3V3" H 7300 2440 50  0000 C CNN
 F 2 "" H 7300 2300 50  0000 C CNN
@@
 P 7250 2750
 F 0 "C43" H 7275 2850 50  0000 L CNN
-F 1 "1uF 4V min" H 7275 2650 50  0000 L CNN
+F 1 "1uF 50V" H 7275 2650 50  0000 L CNN
 F 2 "Capacitors_SMD:C_0805_HandSoldering" H 7288 2600 50  0001 C CNN
 F 3 "" H 7250 2750 50  0000 C CNN
+F 4 "4V" H 7250 2750 60  0001 C CNN "Notes"
 	1    7250 2750
 	1    0    0    -1
 $EndComp
 $Comp
-L GND #PWR087
+L GND #PWR088
 U 1 1 586598C9
 P 7250 3000
-F 0 "#PWR087" H 7250 2750 50  0001 C CNN
+F 0 "#PWR088" H 7250 2750 50  0001 C CNN
 F 1 "GND" H 7250 2850 50  0000 C CNN
 F 2 "" H 7250 3000 50  0000 C CNN
@@
 F 2 "Diodes_SMD:SOD-123" H 7900 2800 50  0001 C CNN
 F 3 "" H 7900 2800 50  0000 C CNN
+F 4 "http://uk.farnell.com/on-semiconductor/mmsz4685t1g/diode-zener-vz-3-6v/dp/1651592" H 7900 2800 60  0001 C CNN "Order"
+F 5 "MMSZ4685T1G" H 7900 2800 60  0001 C CNN "Part"
+F 6 "1651592" H 7900 2800 60  0001 C CNN "Farnell"
 	1    7900 2800
 	0    1    1    0
@@
 $EndComp
 $Comp
-L GND #PWR088
+L GND #PWR089
 U 1 1 5865A3E7
 P 7900 3100
-F 0 "#PWR088" H 7900 2850 50  0001 C CNN
+F 0 "#PWR089" H 7900 2850 50  0001 C CNN
 F 1 "GND" H 7900 2950 50  0000 C CNN
 F 2 "" H 7900 3100 50  0000 C CNN
@@
 $EndComp
 $Comp
-L GND #PWR089
+L GND #PWR090
 U 1 1 5865A42E
 P 8550 3150
-F 0 "#PWR089" H 8550 2900 50  0001 C CNN
+F 0 "#PWR090" H 8550 2900 50  0001 C CNN
 F 1 "GND" H 8550 3000 50  0000 C CNN
 F 2 "" H 8550 3150 50  0000 C CNN
@@
 $EndComp
 $Comp
-L GND #PWR090
+L GND #PWR091
 U 1 1 586ECEC7
 P 4350 1550
-F 0 "#PWR090" H 4350 1300 50  0001 C CNN
+F 0 "#PWR091" H 4350 1300 50  0001 C CNN
 F 1 "GND" H 4350 1400 50  0000 C CNN
 F 2 "" H 4350 1550 50  0000 C CNN
@@
 	4350 1550 4350 1450
 $Comp
-L PWR_FLAG #FLG091
+L PWR_FLAG #FLG092
 U 1 1 5874647E
 P 6000 2250
-F 0 "#FLG091" H 6000 2345 50  0001 C CNN
+F 0 "#FLG092" H 6000 2345 50  0001 C CNN
 F 1 "PWR_FLAG" H 6000 2430 50  0000 C CNN
 F 2 "" H 6000 2250 50  0000 C CNN
@@
 Connection ~ 6000 2450
 $Comp
-L PWR_FLAG #FLG092
+L PWR_FLAG #FLG093
 U 1 1 58746589
 P 7950 2050
-F 0 "#FLG092" H 7950 2145 50  0001 C CNN
+F 0 "#FLG093" H 7950 2145 50  0001 C CNN
 F 1 "PWR_FLAG" H 7950 2230 50  0000 C CNN
 F 2 "" H 7950 2050 50  0000 C CNN
@@
 Connection ~ 7950 2150
 $Comp
-L PWR_FLAG #FLG093
+L PWR_FLAG #FLG094
 U 1 1 58746947
 P 1900 1050
-F 0 "#FLG093" H 1900 1145 50  0001 C CNN
+F 0 "#FLG094" H 1900 1145 50  0001 C CNN
 F 1 "PWR_FLAG" H 1900 1230 50  0000 C CNN
 F 2 "" H 1900 1050 50  0000 C CNN
@@
 	1900 1150 1600 1150
 $Comp
-L PWR_FLAG #FLG094
+L PWR_FLAG #FLG095
 U 1 1 58746A06
 P 900 2000
-F 0 "#FLG094" H 900 2095 50  0001 C CNN
+F 0 "#FLG095" H 900 2095 50  0001 C CNN
 F 1 "PWR_FLAG" H 900 2180 50  0000 C CNN
 F 2 "" H 900 2000 50  0000 C CNN
@@
 Connection ~ 1100 1600
 $Comp
-L PWR_FLAG #FLG095
+L PWR_FLAG #FLG096
 U 1 1 58764812
 P 3350 1450
-F 0 "#FLG095" H 3350 1545 50  0001 C CNN
+F 0 "#FLG096" H 3350 1545 50  0001 C CNN
 F 1 "PWR_FLAG" H 3350 1630 50  0000 C CNN
 F 2 "" H 3350 1450 50  0000 C CNN

Commit message: Tweaks to PCB.
Parts:
- C40: value 220nF 100V -> 220nF 25V
Changed lines of the file:
@@
 LIBS:IFX91041EJV33
 LIBS:BMC2-cache
-EELAYER 26 0
+EELAYER 25 0
 EELAYER END
 $Descr A4 11693 8268
@@
 P 4350 2250
 F 0 "C40" H 4375 2350 50  0000 L CNN
-F 1 "220nF 100V" H 4375 2150 50  0000 L CNN
+F 1 "220nF 25V" H 4375 2150 50  0000 L CNN
 F 2 "Capacitors_SMD:C_0805_HandSoldering" H 4388 2100 50  0001 C CNN
 F 3 "" H 4350 2250 50  0000 C CNN

Commit message: BMCV2.1 updates.
Parts:
- removed D9: RED, LEDs:LED_0805, symbol LED-RESCUE-BMC2
- removed R34: 100R, Resistors_SMD:R_0805_HandSoldering, symbol R
- removed W11: GND, Measurement_Points:Measurement_Point_Round-SMD-Pad_Big, symbol TEST_1P
Changed lines of the file:
@@
-EESchema Schematic File Version 2
+EESchema Schematic File Version 3
 LIBS:BMC2-rescue
 LIBS:power
@@
 LIBS:dc-dc
 LIBS:IFX91041EJV33
+LIBS:MIC2009A-1YM6TR
 LIBS:BMC2-cache
-EELAYER 25 0
+EELAYER 26 0
 EELAYER END
 $Descr A4 11693 8268
 encoding utf-8
-Sheet 4 4
+Sheet 3 4
 Title ""
 Date ""
@@
 	5900 2450 5900 2500
 Connection ~ 5550 2450
-$Comp
-L LED-RESCUE-BMC2 D9
-U 1 1 585F871A
-P 8550 2850
-AR Path="/585F871A" Ref="D9"  Part="1"
-AR Path="/585F64FD/585F871A" Ref="D9"  Part="1"
-F 0 "D9" H 8550 2950 50  0000 C CNN
-F 1 "RED" H 8550 2750 50  0000 C CNN
-F 2 "LEDs:LED_0805" H 8550 2850 50  0001 C CNN
-F 3 "" H 8550 2850 50  0000 C CNN
-F 4 "1581239" H 8550 2850 60  0001 C CNN "Farnell"
-	1    8550 2850
-	0    -1   -1   0
-$EndComp
-$Comp
-L R R34
-U 1 1 585F876D
-P 8550 2400
-F 0 "R34" V 8630 2400 50  0000 C CNN
-F 1 "100R" V 8550 2400 50  0000 C CNN
-F 2 "Resistors_SMD:R_0805_HandSoldering" V 8480 2400 50  0001 C CNN
-F 3 "" H 8550 2400 50  0000 C CNN
-	1    8550 2400
-	1    0    0    -1
-$EndComp
 Connection ~ 5900 2950
 Connection ~ 5900 2450
@@
 	7900 2150 7900 2600
 Connection ~ 7300 2450
-Wire Wire Line
-	8550 2550 8550 2650
-Wire Wire Line
-	7900 2150 8550 2150
-Wire Wire Line
-	8550 2150 8550 2250
 Connection ~ 7900 2450
 Wire Wire Line
 	5300 2950 5900 2950
+$Comp
+L GND #PWR089
+U 1 1 5865A3E7
+P 7900 3100
+F 0 "#PWR089" H 7900 2850 50  0001 C CNN
+F 1 "GND" H 7900 2950 50  0000 C CNN
+F 2 "" H 7900 3100 50  0000 C CNN
+F 3 "" H 7900 3100 50  0000 C CNN
+	1    7900 3100
+	1    0    0    -1
+$EndComp
+Wire Wire Line
+	7900 3000 7900 3100
+Wire Wire Line
+	5100 2450 6200 2450
+$Comp
+L TEST_1P W12
+U 1 1 586E8A7C
+P 5750 2200
+F 0 "W12" H 5750 2470 50  0000 C CNN
+F 1 "5V" H 5750 2400 50  0000 C CNN
+F 2 "Measurement_Points:Measurement_Point_Round-SMD-Pad_Small" H 5950 2200 50  0001 C CNN
+F 3 "" H 5950 2200 50  0000 C CNN
+	1    5750 2200
+	1    0    0    -1
+$EndComp
+Wire Wire Line
+	5750 2200 5750 2450
+Connection ~ 5750 2450
+$Comp
+L TEST_1P W13
+U 1 1 586E8BDF
+P 8250 1950
+F 0 "W13" H 8250 2220 50  0000 C CNN
+F 1 "3V3" H 8250 2150 50  0000 C CNN
+F 2 "Measurement_Points:Measurement_Point_Round-SMD-Pad_Small" H 8450 1950 50  0001 C CNN
+F 3 "" H 8450 1950 50  0000 C CNN
+	1    8250 1950
+	1    0    0    -1
+$EndComp
+Wire Wire Line
+	8250 2150 8250 1950
+$Comp
+L TEST_1P W10
+U 1 1 586EC5DC
+P 3000 1400
+F 0 "W10" H 3000 1670 50  0000 C CNN
+F 1 "DSUP" H 3000 1600 50  0000 C CNN
+F 2 "Measurement_Points:Measurement_Point_Round-SMD-Pad_Small" H 3200 1400 50  0001 C CNN
+F 3 "" H 3200 1400 50  0000 C CNN
+	1    3000 1400
+	1    0    0    -1
+$EndComp
+Wire Wire Line
+	3000 1400 3000 1600
+Connection ~ 3000 1600
+$Comp
+L PWR_FLAG #FLG092
+U 1 1 5874647E
+P 6000 2250
+F 0 "#FLG092" H 6000 2345 50  0001 C CNN
+F 1 "PWR_FLAG" H 6000 2430 50  0000 C CNN
+F 2 "" H 6000 2250 50  0000 C CNN
+F 3 "" H 6000 2250 50  0000 C CNN
+	1    6000 2250
+	1    0    0    -1
+$EndComp
+Wire Wire Line
+	6000 2250 6000 2450
+Connection ~ 6000 2450
+$Comp
+L PWR_FLAG #FLG093
+U 1 1 58746589
+P 7950 2050
+F 0 "#FLG093" H 7950 2145 50  0001 C CNN
+F 1 "PWR_FLAG" H 7950 2230 50  0000 C CNN
+F 2 "" H 7950 2050 50  0000 C CNN
+F 3 "" H 7950 2050 50  0000 C CNN
+	1    7950 2050
+	1    0    0    -1
+$EndComp
+Wire Wire Line
+	7950 2050 7950 2150
+Connection ~ 7950 2150
+$Comp
+L PWR_FLAG #FLG094
+U 1 1 58746947
+P 1900 1050
+F 0 "#FLG094" H 1900 1145 50  0001 C CNN
+F 1 "PWR_FLAG" H 1900 1230 50  0000 C CNN
+F 2 "" H 1900 1050 50  0000 C CNN
+F 3 "" H 1900 1050 50  0000 C CNN
+	1    1900 1050
+	1    0    0    -1
+$EndComp
+Wire Wire Line
+	1900 1050 1900 1150
+Wire Wire Line
+	1900 1150 1600 1150
+$Comp
+L PWR_FLAG #FLG095
+U 1 1 58746A06
+P 900 2000
+F 0 "#FLG095" H 900 2095 50  0001 C CNN
+F 1 "PWR_FLAG" H 900 2180 50  0000 C CNN
+F 2 "" H 900 2000 50  0000 C CNN
+F 3 "" H 900 2000 50  0000 C CNN
+	1    900  2000
+	1    0    0    -1
+$EndComp
+Wire Wire Line
+	900  2000 1100 2000
+Wire Wire Line
+	1100 2000 1100 1600
+Connection ~ 1100 1600
+$Comp
+L PWR_FLAG #FLG096
+U 1 1 58764812
+P 3350 1450
+F 0 "#FLG096" H 3350 1545 50  0001 C CNN
+F 1 "PWR_FLAG" H 3350 1630 50  0000 C CNN
+F 2 "" H 3350 1450 50  0000 C CNN
+F 3 "" H 3350 1450 50  0000 C CNN
+	1    3350 1450
+	1    0    0    -1
+$EndComp
+Connection ~ 7250 2550
+Wire Wire Line
+	7900 2150 8250 2150
 $Comp
 L TC2117-3.3V U5
@@
 	1    0    0    -1
 $EndComp
-$Comp
-L GND #PWR089
-U 1 1 5865A3E7
-P 7900 3100
-F 0 "#PWR089" H 7900 2850 50  0001 C CNN
-F 1 "GND" H 7900 2950 50  0000 C CNN
-F 2 "" H 7900 3100 50  0000 C CNN
-F 3 "" H 7900 3100 50  0000 C CNN
-	1    7900 3100
-	1    0    0    -1
-$EndComp
-$Comp
-L GND #PWR090
-U 1 1 5865A42E
-P 8550 3150
-F 0 "#PWR090" H 8550 2900 50  0001 C CNN
-F 1 "GND" H 8550 3000 50  0000 C CNN
-F 2 "" H 8550 3150 50  0000 C CNN
-F 3 "" H 8550 3150 50  0000 C CNN
-	1    8550 3150
-	1    0    0    -1
-$EndComp
-Wire Wire Line
-	8550 3050 8550 3150
-Wire Wire Line
-	7900 3000 7900 3100
-Wire Wire Line
-	5100 2450 6200 2450
-$Comp
-L TEST_1P W12
-U 1 1 586E8A7C
-P 5750 2200
-F 0 "W12" H 5750 2470 50  0000 C CNN
-F 1 "5V" H 5750 2400 50  0000 C CNN
-F 2 "Measurement_Points:Measurement_Point_Round-SMD-Pad_Small" H 5950 2200 50  0001 C CNN
-F 3 "" H 5950 2200 50  0000 C CNN
-	1    5750 2200
-	1    0    0    -1
-$EndComp
-Wire Wire Line
-	5750 2200 5750 2450
-Connection ~ 5750 2450
-$Comp
-L TEST_1P W13
-U 1 1 586E8BDF
-P 8250 1950
-F 0 "W13" H 8250 2220 50  0000 C CNN
-F 1 "3V3" H 8250 2150 50  0000 C CNN
-F 2 "Measurement_Points:Measurement_Point_Round-SMD-Pad_Small" H 8450 1950 50  0001 C CNN
-F 3 "" H 8450 1950 50  0000 C CNN
-	1    8250 1950
-	1    0    0    -1
-$EndComp
-Wire Wire Line
-	8250 1950 8250 2150
-Connection ~ 8250 2150
-$Comp
-L TEST_1P W10
-U 1 1 586EC5DC
-P 3000 1400
-F 0 "W10" H 3000 1670 50  0000 C CNN
-F 1 "DSUP" H 3000 1600 50  0000 C CNN
-F 2 "Measurement_Points:Measurement_Point_Round-SMD-Pad_Small" H 3200 1400 50  0001 C CNN
-F 3 "" H 3200 1400 50  0000 C CNN
-	1    3000 1400
-	1    0    0    -1
-$EndComp
-Wire Wire Line
-	3000 1400 3000 1600
-Connection ~ 3000 1600
-$Comp
-L TEST_1P W11
-U 1 1 586ECE27
-P 4350 1450
-F 0 "W11" H 4350 1720 50  0000 C CNN
-F 1 "GND" H 4350 1650 50  0000 C CNN
-F 2 "Measurement_Points:Measurement_Point_Round-SMD-Pad_Big" H 4550 1450 50  0001 C CNN
-F 3 "" H 4550 1450 50  0000 C CNN
-	1    4350 1450
-	1    0    0    -1
-$EndComp
-$Comp
-L GND #PWR091
-U 1 1 586ECEC7
-P 4350 1550
-F 0 "#PWR091" H 4350 1300 50  0001 C CNN
-F 1 "GND" H 4350 1400 50  0000 C CNN
-F 2 "" H 4350 1550 50  0000 C CNN
-F 3 "" H 4350 1550 50  0000 C CNN
-	1    4350 1550
-	1    0    0    -1
-$EndComp
-Wire Wire Line
-	4350 1550 4350 1450
-$Comp
-L PWR_FLAG #FLG092
-U 1 1 5874647E
-P 6000 2250
-F 0 "#FLG092" H 6000 2345 50  0001 C CNN
-F 1 "PWR_FLAG" H 6000 2430 50  0000 C CNN
-F 2 "" H 6000 2250 50  0000 C CNN
-F 3 "" H 6000 2250 50  0000 C CNN
-	1    6000 2250
-	1    0    0    -1
-$EndComp
-Wire Wire Line
-	6000 2250 6000 2450
-Connection ~ 6000 2450
-$Comp
-L PWR_FLAG #FLG093
-U 1 1 58746589
-P 7950 2050
-F 0 "#FLG093" H 7950 2145 50  0001 C CNN
-F 1 "PWR_FLAG" H 7950 2230 50  0000 C CNN
-F 2 "" H 7950 2050 50  0000 C CNN
-F 3 "" H 7950 2050 50  0000 C CNN
-	1    7950 2050
-	1    0    0    -1
-$EndComp
-Wire Wire Line
-	7950 2050 7950 2150
-Connection ~ 7950 2150
-$Comp
-L PWR_FLAG #FLG094
-U 1 1 58746947
-P 1900 1050
-F 0 "#FLG094" H 1900 1145 50  0001 C CNN
-F 1 "PWR_FLAG" H 1900 1230 50  0000 C CNN
-F 2 "" H 1900 1050 50  0000 C CNN
-F 3 "" H 1900 1050 50  0000 C CNN
-	1    1900 1050
-	1    0    0    -1
-$EndComp
-Wire Wire Line
-	1900 1050 1900 1150
-Wire Wire Line
-	1900 1150 1600 1150
-$Comp
-L PWR_FLAG #FLG095
-U 1 1 58746A06
-P 900 2000
-F 0 "#FLG095" H 900 2095 50  0001 C CNN
-F 1 "PWR_FLAG" H 900 2180 50  0000 C CNN
-F 2 "" H 900 2000 50  0000 C CNN
-F 3 "" H 900 2000 50  0000 C CNN
-	1    900  2000
-	1    0    0    -1
-$EndComp
-Wire Wire Line
-	900  2000 1100 2000
-Wire Wire Line
-	1100 2000 1100 1600
-Connection ~ 1100 1600
-$Comp
-L PWR_FLAG #FLG096
-U 1 1 58764812
-P 3350 1450
-F 0 "#FLG096" H 3350 1545 50  0001 C CNN
-F 1 "PWR_FLAG" H 3350 1630 50  0000 C CNN
-F 2 "" H 3350 1450 50  0000 C CNN
-F 3 "" H 3350 1450 50  0000 C CNN
-	1    3350 1450
-	1    0    0    -1
-$EndComp
 Wire Wire Line
 	7050 2550 7250 2550
-Connection ~ 7250 2550
 $EndSCHEMATC
