File: MotorController2/Controller.sch (KiCad schematic (older format))
At the start: 32 parts, among them P8 CONN_02X05, SW1 RESET, SW2 CAL, U2 STM32F205RBTx, X1 8MHz

Commit message: More updates.
Parts:
- R13: Farnell (none) -> 2447556
Changed lines of the file:
@@
 F 2 "Resistors_SMD:R_0805_HandSoldering" V 9630 2500 50  0001 C CNN
 F 3 "" H 9700 2500 50  0000 C CNN
+F 4 "2447556" V 9700 2500 60  0001 C CNN "Farnell"
 	1    9700 2500
 	0    1    1    0

Commit message: BMCV2.1 updates.
Parts:
- removed R14, R15: 10K, Resistors_SMD:R_0805_HandSoldering, symbol R
- removed W14: PB12, Measurement_Points:Measurement_Point_Round-SMD-Pad_Small, symbol TEST_1P
Connections:
- net CAN_RX: now also U2.61 (CAN1_RX/I2C1_SCL/SDIO_D4/TIM10_CH1/TIM4_CH3/PB8); no longer U2.62 (CAN1_TX/DAC_EXTI9/I2C1_SDA/I2S2_WS/SDIO_D5/SPI2_NSS/TIM11_CH1/TIM4_CH4/PB9)
- net CAN_TX: now also U2.62 (CAN1_TX/DAC_EXTI9/I2C1_SDA/I2S2_WS/SDIO_D5/SPI2_NSS/TIM11_CH1/TIM4_CH4/PB9); no longer U2.61 (CAN1_RX/I2C1_SCL/SDIO_D4/TIM10_CH1/TIM4_CH3/PB8)
- net FanCtrl: now reaches U2.23 (ADC1_IN7/ADC2_IN7/SPI1_MOSI/TIM14_CH1/TIM1_CH1N/TIM3_CH2/TIM8_CH1N/PA7)
- net SensorPwrCtrl: now reaches U2.33 (CAN2_RX/I2C2_SMBA/I2S2_WS/SPI2_NSS/TIM1_BKIN/USART3_CK/USB_OTG_HS_ID/USB_OTG_HS_ULPI_D5/PB12)
- net I2C_SCL renamed SENSOR_PWR_FAULT
- net I2C_SDA renamed FAN_FAULT
- no-connect marks 2 -> 1
Changed lines of the file:
@@
-EESchema Schematic File Version 2
+EESchema Schematic File Version 3
 LIBS:BMC2-rescue
 LIBS:power
@@
 LIBS:dc-dc
 LIBS:IFX91041EJV33
+LIBS:MIC2009A-1YM6TR
 LIBS:BMC2-cache
-EELAYER 25 0
+EELAYER 26 0
 EELAYER END
 $Descr A3 16535 11693
@@
 Text Notes 14350 5700 0    60   ~ 0
 RST
-Text HLabel 13100 6750 2    60   Output ~ 0
+Text HLabel 13100 6850 2    60   Output ~ 0
 CAN_TX
-Text HLabel 13100 6850 2    60   Input ~ 0
+Text HLabel 13100 6750 2    60   Input ~ 0
 CAN_RX
 Text HLabel 13250 5250 2    60   Output ~ 0
@@
 	14550 5700 14550 6350
 Wire Wire Line
-	12800 6750 13100 6750
-Wire Wire Line
-	12800 6850 13100 6850
-Wire Wire Line
 	4350 5950 4600 5950
 Wire Wire Line
@@
 Wire Wire Line
 	12800 5450 13150 5450
-Text HLabel 13100 6950 2    60   BiDi ~ 0
-I2C_SCL
-Text HLabel 13100 7050 2    60   BiDi ~ 0
-I2C_SDA
+Text HLabel 13100 6950 2    60   Input ~ 0
+SENSOR_PWR_FAULT
+Text HLabel 13100 7050 2    60   Input ~ 0
+FAN_FAULT
 Wire Wire Line
 	12800 6950 13100 6950
@@
 Wire Wire Line
 	15050 7050 15050 7100
-$Comp
-L R R15
-U 1 1 586FC3AC
-P 14350 6650
-F 0 "R15" V 14430 6650 50  0000 C CNN
-F 1 "10K" V 14350 6650 50  0000 C CNN
-F 2 "Resistors_SMD:R_0805_HandSoldering" V 14280 6650 50  0001 C CNN
-F 3 "" H 14350 6650 50  0000 C CNN
-	1    14350 6650
-	1    0    0    -1
-$EndComp
-Wire Wire Line
-	14350 6500 14250 6500
-Wire Wire Line
-	14250 6500 14250 6350
 Connection ~ 14250 6350
-$Comp
-L +3V3 #PWR044
-U 1 1 586FC541
-P 14500 6950
-F 0 "#PWR044" H 14500 6800 50  0001 C CNN
-F 1 "+3V3" H 14500 7090 50  0000 C CNN
-F 2 "" H 14500 6950 50  0000 C CNN
-F 3 "" H 14500 6950 50  0000 C CNN
-	1    14500 6950
-	1    0    0    -1
-$EndComp
-Wire Wire Line
-	14500 6950 14350 6950
-Wire Wire Line
-	14350 6950 14350 6800
 $Comp
 L SW_PUSH SW2
@@
 	0    1    1    0
 $EndComp
-$Comp
-L R R14
-U 1 1 586FE4BF
-P 14100 7500
-F 0 "R14" V 14180 7500 50  0000 C CNN
-F 1 "10K" V 14100 7500 50  0000 C CNN
-F 2 "Resistors_SMD:R_0805_HandSoldering" V 14030 7500 50  0001 C CNN
-F 3 "" H 14100 7500 50  0000 C CNN
-	1    14100 7500
-	1    0    0    -1
-$EndComp
-$Comp
-L +3V3 #PWR045
-U 1 1 586FE559
-P 14100 7250
-F 0 "#PWR045" H 14100 7100 50  0001 C CNN
-F 1 "+3V3" H 14100 7390 50  0000 C CNN
-F 2 "" H 14100 7250 50  0000 C CNN
-F 3 "" H 14100 7250 50  0000 C CNN
-	1    14100 7250
-	1    0    0    -1
-$EndComp
-Wire Wire Line
-	14100 7250 14100 7350
-Wire Wire Line
-	14100 7650 14100 7750
+Wire Wire Line
+	14100 7700 14100 7750
 $Comp
 L GND #PWR046
@@
 	13800 6150 12800 6150
 $Comp
-L TEST_1P W14
-U 1 1 58716B1C
-P 13650 7150
-F 0 "W14" H 13650 7420 50  0000 C CNN
-F 1 "PB12" H 13650 7350 50  0000 C CNN
-F 2 "Measurement_Points:Measurement_Point_Round-SMD-Pad_Small" H 13850 7150 50  0001 C CNN
-F 3 "" H 13850 7150 50  0000 C CNN
-	1    13650 7150
-	1    0    0    -1
-$EndComp
-Wire Wire Line
-	12800 7150 13650 7150
-$Comp
 L +3.3VADC #PWR047
 U 1 1 585F9182
@@
 	3500 5550 3350 5550
 Connection ~ 3350 5550
-NoConn ~ 12800 4950
 $Comp
 L PWR_FLAG #FLG049
@@
 Wire Wire Line
 	12800 7450 13100 7450
+Wire Wire Line
+	12800 6750 13100 6750
+Wire Wire Line
+	12800 6850 13100 6850
+Text HLabel 13250 4950 2    60   Output ~ 0
+FanCtrl
+Wire Wire Line
+	12800 4950 13250 4950
+Text HLabel 13100 7150 2    60   Output ~ 0
+SensorPwrCtrl
+Wire Wire Line
+	12800 7150 13100 7150
 $EndSCHEMATC

Commit message: Updates for parts list.
Parts:
- C3: Price (none) -> 0.0897
- C5: Price (none) -> .0303
- C8: Farnell 1828835 -> 9227938; Price (none) -> 0.306
- D2: value GREEN LED -> Green LED; Price (none) -> 0.249
- D3: value YELLOW -> Yellow LED; Price (none) -> 0.171
- JP2: Farnell (none) -> 9333681; Price (none) -> 0.0097
- L1: Price (none) -> 0.0944
- P8: Price (none) -> 1.63; RSStockNo (none) -> 451-732; Supplier (none) -> RS
- R13: Price (none) -> 0.0062
- SW1: Farnell 42468741 -> 2468741; Price (none) -> 0.192
- U2: value STM32F205RBTx -> STM32F405RGT6V; Farnell (none) -> 2333282; Price (none) -> 8.38; RSStockNo (none) -> 810-7673; Supplier (none) -> RS
- X1: MF (none) -> ABRACON; MP (none) -> ABM3-8.000MHZ-B4Y-T; Mouser (none) -> 815-ABM38000B4YT; Supplier (none) -> Mouser
Changed lines of the file:
@@
-EESchema Schematic File Version 2
+EESchema Schematic File Version 3
 LIBS:BMC2-rescue
 LIBS:power
 LIBS:device
-LIBS:transistors
-LIBS:conn
 LIBS:linear
 LIBS:regul
-LIBS:74xx
-LIBS:cmos4000
 LIBS:adc-dac
 LIBS:memory
@@
 LIBS:digital-audio
 LIBS:philips
-LIBS:display
 LIBS:cypress
 LIBS:siliconi
@@
 LIBS:atmel
 LIBS:contrib
-LIBS:valves
-LIBS:stm32
 LIBS:Power_Management
 LIBS:motor_drivers
@@
 LIBS:MIC2009A-1YM6TR
 LIBS:BMC2-cache
-EELAYER 25 0
+EELAYER 26 0
 EELAYER END
 $Descr A3 16535 11693
@@
 F 3 "" H 3650 5100 50  0000 C CNN
 F 4 "2497014" H 3650 5100 60  0001 C CNN "Farnell"
+F 5 ".0303" H 3650 5100 60  0001 C CNN "Price"
 	1    3650 5100
 	0    1    1    0
@@
 F 3 "" H 14800 4300 50  0000 C CNN
 F 4 "http://uk.rs-online.com/web/p/pcb-headers/0451732/?searchTerm=FTSH-105-01-F-DV-K&autocorrected=y&relevancy-data=636F3D3526696E3D4931384E4D616E506172744E756D626572266C753D656E266D6D3D6D61746368616C6C7061727469616C26706D3D5E5B5C707B4C7D5C707B4E647D2D2C2F255C2E5D2B2426706F3D3226736E3D592673723D4175746F636F727265637465642673613D6674736831303530316664762673743D4B4559574F52445F53494E474C455F414C5048415F4E554D455249432673633D592677633D4E4F4E45267573743D465453482D3130352D30312D462D44562D4B267374613D4654534831303530314644564B26" H 14800 5500 60  0001 C CNN "Order"
+F 5 "451-732" H 14800 5500 60  0001 C CNN "RSStockNo"
+F 6 "RS" H 14800 5500 60  0001 C CNN "Supplier"
+F 7 "1.63" H 14800 5500 60  0001 C CNN "Price"
 	1    14800 5500
 	-1   0    0    -1
@@
 F 2 "Capacitors_SMD:C_1206_HandSoldering" H 7238 2900 50  0001 C CNN
 F 3 "" H 7200 3050 50  0000 C CNN
-F 4 "1828835" H 7200 3050 60  0001 C CNN "Farnell"
+F 4 "9227938" H 7200 3050 60  0001 C CNN "Farnell"
+F 5 "0.306" H 7200 3050 60  0001 C CNN "Price"
 	1    7200 3050
 	1    0    0    -1
@@
 F 3 "" H 9700 2500 50  0000 C CNN
 F 4 "2447556" V 9700 2500 60  0001 C CNN "Farnell"
+F 5 "0.0062" V 9700 2500 60  0001 C CNN "Price"
 	1    9700 2500
 	0    1    1    0
@@
 F 3 "" H 9200 2500 50  0000 C CNN
 F 4 "2215650" V 9200 2500 60  0001 C CNN "Farnell"
+F 5 "0.0944" V 9200 2500 60  0001 C CNN "Price"
 	1    9200 2500
 	0    -1   -1   0
@@
 F 2 "Buttons_Switches_SMD:SW_SPST_FSMSM" H 3600 3550 50  0001 C CNN
 F 3 "" H 3600 3550 50  0000 C CNN
-F 4 "42468741" H 3600 3550 60  0001 C CNN "Farnell"
+F 4 "2468741" H 3600 3550 60  0001 C CNN "Farnell"
+F 5 "0.192" H 3600 3550 60  0001 C CNN "Price"
 	1    3600 3550
 	1    0    0    -1
@@
 F 2 "Resistors_SMD:R_0805_HandSoldering" H 14750 6350 50  0001 C CNN
 F 3 "" H 14750 6350 50  0000 C CNN
+F 4 "9333681" H 14750 6350 60  0001 C CNN "Farnell"
+F 5 "0.0097" H 14750 6350 60  0001 C CNN "Price"
 	1    14750 6350
 	1    0    0    -1
@@
 F 3 "" H 2750 4900 50  0000 C CNN
 F 4 "2611933" H 2750 4900 60  0001 C CNN "Farnell"
+F 5 "0.0897" H 2750 4900 60  0001 C CNN "Price"
 	1    2750 4900
 	1    0    0    -1
@@
 P 8700 5850
 F 0 "U2" H 4700 7775 50  0000 L BNN
-F 1 "STM32F205RBTx" H 12700 7775 50  0000 R BNN
+F 1 "STM32F405RGT6V" H 12700 7775 50  0000 R BNN
 F 2 "Housings_QFP:LQFP-64_10x10mm_Pitch0.5mm" H 12700 7725 50  0000 R TNN
 F 3 "http://www.st.com/content/ccc/resource/technical/document/datasheet/bc/21/42/43/b0/f3/4d/d3/CD00237391.pdf/files/CD00237391.pdf/jcr:content/translations/en.CD00237391.pdf" H 8700 5850 50  0001 C CNN
+F 4 "2333282" H 8700 5850 60  0001 C CNN "Farnell"
+F 5 "8.38" H 8700 5850 60  0001 C CNN "Price"
+F 6 "RS" H 8700 5850 60  0001 C CNN "Supplier"
+F 7 "810-7673" H 8700 5850 60  0001 C CNN "RSStockNo"
 	1    8700 5850
 	1    0    0    -1
@@
 P 3000 7050
 F 0 "D2" H 3000 7150 50  0000 C CNN
-F 1 "GREEN LED" H 3000 6950 50  0000 C CNN
+F 1 "Green LED" H 3000 6950 50  0000 C CNN
 F 2 "LEDs:LED_0805" H 3000 7050 50  0001 C CNN
 F 3 "" H 3000 7050 50  0000 C CNN
 F 4 "1465996" H 3000 7050 60  0001 C CNN "Farnell"
 F 5 "2V" H 3000 7050 60  0001 C CNN "Notes"
+F 6 "0.249" H 3000 7050 60  0001 C CNN "Price"
 	1    3000 7050
 	0    -1   -1   0
@@
 P 3250 7050
 F 0 "D3" H 3250 7150 50  0000 C CNN
-F 1 "YELLOW" H 3250 6950 50  0000 C CNN
+F 1 "Yellow LED" H 3250 6950 50  0000 C CNN
 F 2 "LEDs:LED_0805" H 3250 7050 50  0001 C CNN
 F 3 "" H 3250 7050 50  0000 C CNN
 F 4 "1581241" H 3250 7050 60  0001 C CNN "Farnell"
+F 5 "0.171" H 3250 7050 60  0001 C CNN "Price"
 	1    3250 7050
 	0    -1   -1   0
@@
 F 4 "http://uk.farnell.com/abracon/abm3-8-000mhz-d2y-t/crystal-8mhz-18pf-smd/dp/2101329" H 4000 5300 60  0001 C CNN "Order"
 F 5 "2101329" H 4000 5300 60  0001 C CNN "Farnell"
+F 6 "Mouser" H 4000 5300 60  0001 C CNN "Supplier"
+F 7 "815-ABM38000B4YT " H 4000 5300 60  0001 C CNN "Mouser"
+F 8 "ABM3-8.000MHZ-B4Y-T" H 4000 5300 60  0001 C CNN "MP"
+F 9 "ABRACON" H 4000 5300 60  0001 C CNN "MF"
 	1    4000 5300
 	0    1    1    0

Commit message: Add some annotations.
Other:
- note added: "L1 and R13 are intended to help keep some \nnoise out of the Analog supply. It isn't clear \nthey are needed."
Changed lines of the file:
@@
-EESchema Schematic File Version 3
+EESchema Schematic File Version 2
 LIBS:BMC2-rescue
 LIBS:power
 LIBS:device
+LIBS:transistors
+LIBS:conn
 LIBS:linear
 LIBS:regul
+LIBS:74xx
+LIBS:cmos4000
 LIBS:adc-dac
 LIBS:memory
@@
 LIBS:digital-audio
 LIBS:philips
+LIBS:display
 LIBS:cypress
 LIBS:siliconi
@@
 LIBS:atmel
 LIBS:contrib
+LIBS:valves
+LIBS:stm32
 LIBS:Power_Management
 LIBS:motor_drivers
@@
 LIBS:MIC2009A-1YM6TR
 LIBS:BMC2-cache
-EELAYER 26 0
+EELAYER 25 0
 EELAYER END
 $Descr A3 16535 11693
@@
 Wire Wire Line
 	12800 7150 13100 7150
+Text Notes 8400 2250 0    60   ~ 0
+L1 and R13 are intended to help keep some \nnoise out of the Analog supply.  It isn't clear \nthey are needed.
 $EndSCHEMATC
