File: MotorController2/HallSensorBoard/HallSensorBoard.sch (KiCad schematic (older format))
At the start: 6 parts, among them J1 Conn_01x07, J2 Conn_01x02, U1 S49E, U2 S49E, U3 S49E

Commit message: Updates for parts list.
Parts:
- C1: Farnell (none) -> 1759265
- J1: Farnell (none) -> Socket 588763 , Plug 1098693
Changed lines of the file:
@@
 LIBS:valves
 LIBS:s49e
+LIBS:HallSensorBoard-cache
 EELAYER 26 0
 EELAYER END
@@
 F 2 "Capacitors_SMD:C_0805_HandSoldering" H 2488 1950 50  0001 C CNN
 F 3 "" H 2450 2100 50  0001 C CNN
+F 4 "1759265" H 2450 2100 60  0001 C CNN "Farnell"
 	1    2450 2100
 	1    0    0    -1
@@
 F 2 "Pin_Headers:Pin_Header_Angled_1x07_Pitch2.54mm" H 3000 3300 50  0001 C CNN
 F 3 "" H 3000 3300 50  0001 C CNN
+F 4 "Socket  588763 ,  Plug 1098693" H 3000 3300 60  0001 C CNN "Farnell"
 	1    3000 3300
 	-1   0    0    -1

Commit message: Add index sensor plug.
Parts:
- added P1: CONN_01X03, Pin_Headers:Pin_Header_Straight_1x03_Pitch2.54mm, symbol CONN_01X03
- J1: symbol Conn_01x07 -> CONN_01X07
Connections:
- net +3V3: now also P1.1 (P1)
- net GND: now also J2.2 (Pin_2), P1.2 (P2)
- net at J1.7 (P7): now also P1.3 (P3); no longer J2.2 (Pin_2)
Changed lines of the file:
@@
-EESchema Schematic File Version 3
+EESchema Schematic File Version 2
+LIBS:HallSensorBoard-rescue
 LIBS:power
 LIBS:device
@@
 LIBS:contrib
 LIBS:valves
-LIBS:s49e
 LIBS:HallSensorBoard-cache
-EELAYER 26 0
+EELAYER 25 0
 EELAYER END
 $Descr A4 11693 8268
@@
 	5150 2300 5200 2300
 $Comp
-L Conn_01x07 J1
+L CONN_01X07 J1
 U 1 1 59C4E97F
 P 3000 3300
@@
 	3750 3500 3750 3550
 Wire Wire Line
-	3200 3600 3600 3600
-Wire Wire Line
-	3600 3600 3600 3650
-Wire Wire Line
-	3600 3650 3750 3650
+	3650 3650 3750 3650
 $Comp
 L S49E U1
@@
 $EndComp
 $Comp
-L PWR_FLAG #FLG01
+L PWR_FLAG #FLG09
 U 1 1 59C4F0CE
 P 1750 3000
-F 0 "#FLG01" H 1750 3075 50  0001 C CNN
+F 0 "#FLG09" H 1750 3075 50  0001 C CNN
 F 1 "PWR_FLAG" H 1750 3174 50  0000 C CNN
 F 2 "" H 1750 3000 50  0001 C CNN
@@
 $EndComp
 $Comp
-L PWR_FLAG #FLG02
+L PWR_FLAG #FLG010
 U 1 1 59C4F13C
 P 2150 3000
-F 0 "#FLG02" H 2150 3075 50  0001 C CNN
+F 0 "#FLG010" H 2150 3075 50  0001 C CNN
 F 1 "PWR_FLAG" H 2150 3174 50  0000 C CNN
 F 2 "" H 2150 3000 50  0001 C CNN
@@
 $EndComp
 $Comp
-L GND #PWR010
+L GND #PWR011
 U 1 1 59C4F15A
 P 2150 3150
-F 0 "#PWR010" H 2150 2900 50  0001 C CNN
+F 0 "#PWR011" H 2150 2900 50  0001 C CNN
 F 1 "GND" H 2155 2977 50  0000 C CNN
 F 2 "" H 2150 3150 50  0001 C CNN
@@
 	2150 3000 2150 3150
 $Comp
-L +3V3 #PWR09
+L +3V3 #PWR012
 U 1 1 59C4F1D6
 P 1750 3150
-F 0 "#PWR09" H 1750 3000 50  0001 C CNN
+F 0 "#PWR012" H 1750 3000 50  0001 C CNN
 F 1 "+3V3" H 1765 3323 50  0000 C CNN
 F 2 "" H 1750 3150 50  0001 C CNN
@@
 	3050 2050 3100 2050
 $Comp
-L +3V3 #PWR011
+L +3V3 #PWR013
 U 1 1 59C4F296
 P 2450 1900
-F 0 "#PWR011" H 2450 1750 50  0001 C CNN
+F 0 "#PWR013" H 2450 1750 50  0001 C CNN
 F 1 "+3V3" H 2465 2073 50  0000 C CNN
 F 2 "" H 2450 1900 50  0001 C CNN
@@
 $EndComp
 $Comp
-L GND #PWR012
+L GND #PWR014
 U 1 1 59C4F2AD
 P 2450 2300
-F 0 "#PWR012" H 2450 2050 50  0001 C CNN
+F 0 "#PWR014" H 2450 2050 50  0001 C CNN
 F 1 "GND" H 2455 2127 50  0000 C CNN
 F 2 "" H 2450 2300 50  0001 C CNN
@@
 Wire Wire Line
 	2450 1950 2450 1900
+$Comp
+L GND #PWR015
+U 1 1 5A1E9D59
+P 3650 3800
+F 0 "#PWR015" H 3650 3550 50  0001 C CNN
+F 1 "GND" H 3655 3627 50  0000 C CNN
+F 2 "" H 3650 3800 50  0001 C CNN
+F 3 "" H 3650 3800 50  0001 C CNN
+	1    3650 3800
+	1    0    0    -1
+$EndComp
+Wire Wire Line
+	3650 3800 3650 3650
+$Comp
+L CONN_01X03 P1
+U 1 1 5A1E9DB1
+P 3950 4250
+F 0 "P1" H 3950 4450 50  0000 C CNN
+F 1 "CONN_01X03" V 4050 4250 50  0000 C CNN
+F 2 "Pin_Headers:Pin_Header_Straight_1x03_Pitch2.54mm" H 3950 4250 50  0001 C CNN
+F 3 "" H 3950 4250 50  0000 C CNN
+	1    3950 4250
+	1    0    0    -1
+$EndComp
+$Comp
+L GND #PWR016
+U 1 1 5A1E9DF2
+P 3500 4350
+F 0 "#PWR016" H 3500 4100 50  0001 C CNN
+F 1 "GND" H 3505 4177 50  0000 C CNN
+F 2 "" H 3500 4350 50  0001 C CNN
+F 3 "" H 3500 4350 50  0001 C CNN
+	1    3500 4350
+	1    0    0    -1
+$EndComp
+Wire Wire Line
+	3500 4350 3500 4250
+Wire Wire Line
+	3500 4250 3750 4250
+$Comp
+L +3V3 #PWR017
+U 1 1 5A1E9E3A
+P 3500 4100
+F 0 "#PWR017" H 3500 3950 50  0001 C CNN
+F 1 "+3V3" H 3515 4273 50  0000 C CNN
+F 2 "" H 3500 4100 50  0001 C CNN
+F 3 "" H 3500 4100 50  0001 C CNN
+	1    3500 4100
+	1    0    0    -1
+$EndComp
+Wire Wire Line
+	3500 4100 3500 4150
+Wire Wire Line
+	3500 4150 3750 4150
+Wire Wire Line
+	3750 4350 3650 4350
+Wire Wire Line
+	3650 4350 3650 4550
+Wire Wire Line
+	3650 4550 3300 4550
+Wire Wire Line
+	3300 4550 3300 3600
+Wire Wire Line
+	3300 3600 3200 3600
 $EndSCHEMATC
